File: electronics/stage4/controller-carrier/controller_carrier.kicad_sch (KiCad schematic)
At the start: 1 part, among them J1 HOST POWER

Commit message: Rename project to Project SCCI RH across research and engineering
Parts:
- J1: footprint ato_controller:PinHeader_1x02_P2.54mm_Vertical -> scci_rh_controller:PinHeader_1x02_P2.54mm_Vertical; symbol ATO_CONTROLLER:J1 -> SCCI_RH_CONTROLLER:J1
Other:
- company: Project ATO -> Project SCCI RH
- title: ATO S4 / Controller carrier / interface index -> Project SCCI RH S4 / Controller carrier / interface index
