File: electronics/stage4/controller-carrier/sideband.kicad_sch (KiCad schematic)
At the start: 8 parts, among them U10 SN74LVC165APWR, U11 SN74LVC165APWR, U12 SN74LVC165APWR, U13 SN74LVC165APWR

Commit message: Rename project to Project SCCI RH across research and engineering
Parts:
- C10: footprint ato_controller:C_1206_3216Metric -> scci_rh_controller:C_1206_3216Metric; symbol ATO_CONTROLLER:C10 -> SCCI_RH_CONTROLLER:C10
- C11: footprint ato_controller:C_1206_3216Metric -> scci_rh_controller:C_1206_3216Metric; symbol ATO_CONTROLLER:C11 -> SCCI_RH_CONTROLLER:C11
- C12: footprint ato_controller:C_1206_3216Metric -> scci_rh_controller:C_1206_3216Metric; symbol ATO_CONTROLLER:C12 -> SCCI_RH_CONTROLLER:C12
- C13: footprint ato_controller:C_1206_3216Metric -> scci_rh_controller:C_1206_3216Metric; symbol ATO_CONTROLLER:C13 -> SCCI_RH_CONTROLLER:C13
- U10: footprint ato_controller:TSSOP-16_4.4x5mm_P0.65mm -> scci_rh_controller:TSSOP-16_4.4x5mm_P0.65mm; symbol ATO_CONTROLLER:U10 -> SCCI_RH_CONTROLLER:U10
- U11: footprint ato_controller:TSSOP-16_4.4x5mm_P0.65mm -> scci_rh_controller:TSSOP-16_4.4x5mm_P0.65mm; symbol ATO_CONTROLLER:U11 -> SCCI_RH_CONTROLLER:U11
- U12: footprint ato_controller:TSSOP-16_4.4x5mm_P0.65mm -> scci_rh_controller:TSSOP-16_4.4x5mm_P0.65mm; symbol ATO_CONTROLLER:U12 -> SCCI_RH_CONTROLLER:U12
- U13: footprint ato_controller:TSSOP-16_4.4x5mm_P0.65mm -> scci_rh_controller:TSSOP-16_4.4x5mm_P0.65mm; symbol ATO_CONTROLLER:U13 -> SCCI_RH_CONTROLLER:U13
Other:
- company: Project ATO -> Project SCCI RH
- title: ATO S4 / Four physical 165 devices / parallel observations -> Project SCCI RH S4 / Four physical 165 devices / parallel observations
