File: electronics/stage4/current-driver/permission0.kicad_sch (KiCad schematic)
At the start: 53 parts, among them U300 LTC6993HS6-1#TRPBF, U301 SN74LVC1G86DBVR, U302 SN74LVC1G11DBVR, U303 SN74LVC1G11DBVR, U304 SN74LVC1G08DBVR, U305 SN74LVC1G04DBVR, U306 SN74LVC1G04DBVR, U307 SN74LVC1G08DBVR, U308 SN74LVC1G04DBVR, U309 SN74LVC1G08DBVR, U310 SN74LVC1G11DBVR, U311 SN74LVC1G11DBVR, U312 SN74LVC1G04DBVR, U313 SN74LVC1G74DCUR, U314 SN74LVC1G32DBVR, U315 SN74LVC1G74DCUR, U316 SN74LVC1G74DCUR, U317 SN74LVC1G11DBVR, U318 SN74LVC1G11DBVR, U319 SN74LVC1G08DBVR, U320 SN74LVC1G08DBVR

Commit message: Rename project to Project SCCI RH across research and engineering
Parts:
- C300: footprint ato_drv:C_0805_2012Metric -> scci_rh_drv:C_0805_2012Metric; symbol ATO_DRV:C300 -> SCCI_RH_DRV:C300
- C301: footprint ato_drv:C_0805_2012Metric -> scci_rh_drv:C_0805_2012Metric; symbol ATO_DRV:C301 -> SCCI_RH_DRV:C301
- C302: footprint ato_drv:C_0805_2012Metric -> scci_rh_drv:C_0805_2012Metric; symbol ATO_DRV:C302 -> SCCI_RH_DRV:C302
- C303: footprint ato_drv:C_0805_2012Metric -> scci_rh_drv:C_0805_2012Metric; symbol ATO_DRV:C303 -> SCCI_RH_DRV:C303
- C304: footprint ato_drv:C_0805_2012Metric -> scci_rh_drv:C_0805_2012Metric; symbol ATO_DRV:C304 -> SCCI_RH_DRV:C304
- C305: footprint ato_drv:C_0805_2012Metric -> scci_rh_drv:C_0805_2012Metric; symbol ATO_DRV:C305 -> SCCI_RH_DRV:C305
- C306: footprint ato_drv:C_0805_2012Metric -> scci_rh_drv:C_0805_2012Metric; symbol ATO_DRV:C306 -> SCCI_RH_DRV:C306
- C307: footprint ato_drv:C_0805_2012Metric -> scci_rh_drv:C_0805_2012Metric; symbol ATO_DRV:C307 -> SCCI_RH_DRV:C307
- C308: footprint ato_drv:C_0805_2012Metric -> scci_rh_drv:C_0805_2012Metric; symbol ATO_DRV:C308 -> SCCI_RH_DRV:C308
- C309: footprint ato_drv:C_0805_2012Metric -> scci_rh_drv:C_0805_2012Metric; symbol ATO_DRV:C309 -> SCCI_RH_DRV:C309
- C310: footprint ato_drv:C_0805_2012Metric -> scci_rh_drv:C_0805_2012Metric; symbol ATO_DRV:C310 -> SCCI_RH_DRV:C310
- C311: footprint ato_drv:C_0805_2012Metric -> scci_rh_drv:C_0805_2012Metric; symbol ATO_DRV:C311 -> SCCI_RH_DRV:C311
- C312: footprint ato_drv:C_0805_2012Metric -> scci_rh_drv:C_0805_2012Metric; symbol ATO_DRV:C312 -> SCCI_RH_DRV:C312
- C313: footprint ato_drv:C_0805_2012Metric -> scci_rh_drv:C_0805_2012Metric; symbol ATO_DRV:C313 -> SCCI_RH_DRV:C313
- C314: footprint ato_drv:C_0805_2012Metric -> scci_rh_drv:C_0805_2012Metric; symbol ATO_DRV:C314 -> SCCI_RH_DRV:C314
- C315: footprint ato_drv:C_0805_2012Metric -> scci_rh_drv:C_0805_2012Metric; symbol ATO_DRV:C315 -> SCCI_RH_DRV:C315
- C316: footprint ato_drv:C_0805_2012Metric -> scci_rh_drv:C_0805_2012Metric; symbol ATO_DRV:C316 -> SCCI_RH_DRV:C316
- C317: footprint ato_drv:C_0805_2012Metric -> scci_rh_drv:C_0805_2012Metric; symbol ATO_DRV:C317 -> SCCI_RH_DRV:C317
- C318: footprint ato_drv:C_0805_2012Metric -> scci_rh_drv:C_0805_2012Metric; symbol ATO_DRV:C318 -> SCCI_RH_DRV:C318
- C319: footprint ato_drv:C_0805_2012Metric -> scci_rh_drv:C_0805_2012Metric; symbol ATO_DRV:C319 -> SCCI_RH_DRV:C319
- C320: footprint ato_drv:C_0805_2012Metric -> scci_rh_drv:C_0805_2012Metric; symbol ATO_DRV:C320 -> SCCI_RH_DRV:C320
- R300: footprint ato_drv:R_0805_2012Metric -> scci_rh_drv:R_0805_2012Metric; symbol ATO_DRV:R300 -> SCCI_RH_DRV:R300
- R301: footprint ato_drv:R_0805_2012Metric -> scci_rh_drv:R_0805_2012Metric; symbol ATO_DRV:R301 -> SCCI_RH_DRV:R301
- R302: footprint ato_drv:R_0805_2012Metric -> scci_rh_drv:R_0805_2012Metric; symbol ATO_DRV:R302 -> SCCI_RH_DRV:R302
- R303: footprint ato_drv:R_0805_2012Metric -> scci_rh_drv:R_0805_2012Metric; symbol ATO_DRV:R303 -> SCCI_RH_DRV:R303
- R304: footprint ato_drv:R_0805_2012Metric -> scci_rh_drv:R_0805_2012Metric; symbol ATO_DRV:R304 -> SCCI_RH_DRV:R304
- R305: footprint ato_drv:R_0805_2012Metric -> scci_rh_drv:R_0805_2012Metric; symbol ATO_DRV:R305 -> SCCI_RH_DRV:R305
- R306: footprint ato_drv:R_0805_2012Metric -> scci_rh_drv:R_0805_2012Metric; symbol ATO_DRV:R306 -> SCCI_RH_DRV:R306
- R307: footprint ato_drv:R_0805_2012Metric -> scci_rh_drv:R_0805_2012Metric; symbol ATO_DRV:R307 -> SCCI_RH_DRV:R307
- R308: footprint ato_drv:R_0805_2012Metric -> scci_rh_drv:R_0805_2012Metric; symbol ATO_DRV:R308 -> SCCI_RH_DRV:R308
- R309: footprint ato_drv:R_0805_2012Metric -> scci_rh_drv:R_0805_2012Metric; symbol ATO_DRV:R309 -> SCCI_RH_DRV:R309
- R310: footprint ato_drv:R_0805_2012Metric -> scci_rh_drv:R_0805_2012Metric; symbol ATO_DRV:R310 -> SCCI_RH_DRV:R310
- U300: footprint ato_drv:TSOT-23-6 -> scci_rh_drv:TSOT-23-6; symbol ATO_DRV:U300 -> SCCI_RH_DRV:U300
- U301: footprint ato_drv:SOT-23-5 -> scci_rh_drv:SOT-23-5; symbol ATO_DRV:U301 -> SCCI_RH_DRV:U301
- U302: footprint ato_drv:SOT-23-6 -> scci_rh_drv:SOT-23-6; symbol ATO_DRV:U302 -> SCCI_RH_DRV:U302
- U303: footprint ato_drv:SOT-23-6 -> scci_rh_drv:SOT-23-6; symbol ATO_DRV:U303 -> SCCI_RH_DRV:U303
- U304: footprint ato_drv:SOT-23-5 -> scci_rh_drv:SOT-23-5; symbol ATO_DRV:U304 -> SCCI_RH_DRV:U304
- U305: footprint ato_drv:SOT-23-5 -> scci_rh_drv:SOT-23-5; symbol ATO_DRV:U305 -> SCCI_RH_DRV:U305
- U306: footprint ato_drv:SOT-23-5 -> scci_rh_drv:SOT-23-5; symbol ATO_DRV:U306 -> SCCI_RH_DRV:U306
- U307: footprint ato_drv:SOT-23-5 -> scci_rh_drv:SOT-23-5; symbol ATO_DRV:U307 -> SCCI_RH_DRV:U307
- U308: footprint ato_drv:SOT-23-5 -> scci_rh_drv:SOT-23-5; symbol ATO_DRV:U308 -> SCCI_RH_DRV:U308
- U309: footprint ato_drv:SOT-23-5 -> scci_rh_drv:SOT-23-5; symbol ATO_DRV:U309 -> SCCI_RH_DRV:U309
- U310: footprint ato_drv:SOT-23-6 -> scci_rh_drv:SOT-23-6; symbol ATO_DRV:U310 -> SCCI_RH_DRV:U310
- U311: footprint ato_drv:SOT-23-6 -> scci_rh_drv:SOT-23-6; symbol ATO_DRV:U311 -> SCCI_RH_DRV:U311
- U312: footprint ato_drv:SOT-23-5 -> scci_rh_drv:SOT-23-5; symbol ATO_DRV:U312 -> SCCI_RH_DRV:U312
- U313: footprint ato_drv:VSSOP-8_2.3x2mm_P0.5mm -> scci_rh_drv:VSSOP-8_2.3x2mm_P0.5mm; symbol ATO_DRV:U313 -> SCCI_RH_DRV:U313
- U314: footprint ato_drv:SOT-23-5 -> scci_rh_drv:SOT-23-5; symbol ATO_DRV:U314 -> SCCI_RH_DRV:U314
- U315: footprint ato_drv:VSSOP-8_2.3x2mm_P0.5mm -> scci_rh_drv:VSSOP-8_2.3x2mm_P0.5mm; symbol ATO_DRV:U315 -> SCCI_RH_DRV:U315
- U316: footprint ato_drv:VSSOP-8_2.3x2mm_P0.5mm -> scci_rh_drv:VSSOP-8_2.3x2mm_P0.5mm; symbol ATO_DRV:U316 -> SCCI_RH_DRV:U316
- U317: footprint ato_drv:SOT-23-6 -> scci_rh_drv:SOT-23-6; symbol ATO_DRV:U317 -> SCCI_RH_DRV:U317
- U318: footprint ato_drv:SOT-23-6 -> scci_rh_drv:SOT-23-6; symbol ATO_DRV:U318 -> SCCI_RH_DRV:U318
- U319: footprint ato_drv:SOT-23-5 -> scci_rh_drv:SOT-23-5; symbol ATO_DRV:U319 -> SCCI_RH_DRV:U319
- U320: footprint ato_drv:SOT-23-5 -> scci_rh_drv:SOT-23-5; symbol ATO_DRV:U320 -> SCCI_RH_DRV:U320
Other:
- company: Project ATO -> Project SCCI RH
- title: ATO S4 / Source 0: independent duration and sticky admission -> Project SCCI RH S4 / Source 0: independent duration and sticky admission
