File: electronics/stage4/current-driver/permission1.kicad_sch (KiCad schematic)
At the start: 53 parts, among them U400 LTC6993HS6-1#TRPBF, U401 SN74LVC1G86DBVR, U402 SN74LVC1G11DBVR, U403 SN74LVC1G11DBVR, U404 SN74LVC1G08DBVR, U405 SN74LVC1G04DBVR, U406 SN74LVC1G04DBVR, U407 SN74LVC1G08DBVR, U408 SN74LVC1G04DBVR, U409 SN74LVC1G08DBVR, U410 SN74LVC1G11DBVR, U411 SN74LVC1G11DBVR, U412 SN74LVC1G04DBVR, U413 SN74LVC1G74DCUR, U414 SN74LVC1G32DBVR, U415 SN74LVC1G74DCUR, U416 SN74LVC1G74DCUR, U417 SN74LVC1G11DBVR, U418 SN74LVC1G11DBVR, U419 SN74LVC1G08DBVR, U420 SN74LVC1G08DBVR

Commit message: Rename project to Project SCCI RH across research and engineering
Parts:
- C400: footprint ato_drv:C_0805_2012Metric -> scci_rh_drv:C_0805_2012Metric; symbol ATO_DRV:C400 -> SCCI_RH_DRV:C400
- C401: footprint ato_drv:C_0805_2012Metric -> scci_rh_drv:C_0805_2012Metric; symbol ATO_DRV:C401 -> SCCI_RH_DRV:C401
- C402: footprint ato_drv:C_0805_2012Metric -> scci_rh_drv:C_0805_2012Metric; symbol ATO_DRV:C402 -> SCCI_RH_DRV:C402
- C403: footprint ato_drv:C_0805_2012Metric -> scci_rh_drv:C_0805_2012Metric; symbol ATO_DRV:C403 -> SCCI_RH_DRV:C403
- C404: footprint ato_drv:C_0805_2012Metric -> scci_rh_drv:C_0805_2012Metric; symbol ATO_DRV:C404 -> SCCI_RH_DRV:C404
- C405: footprint ato_drv:C_0805_2012Metric -> scci_rh_drv:C_0805_2012Metric; symbol ATO_DRV:C405 -> SCCI_RH_DRV:C405
- C406: footprint ato_drv:C_0805_2012Metric -> scci_rh_drv:C_0805_2012Metric; symbol ATO_DRV:C406 -> SCCI_RH_DRV:C406
- C407: footprint ato_drv:C_0805_2012Metric -> scci_rh_drv:C_0805_2012Metric; symbol ATO_DRV:C407 -> SCCI_RH_DRV:C407
- C408: footprint ato_drv:C_0805_2012Metric -> scci_rh_drv:C_0805_2012Metric; symbol ATO_DRV:C408 -> SCCI_RH_DRV:C408
- C409: footprint ato_drv:C_0805_2012Metric -> scci_rh_drv:C_0805_2012Metric; symbol ATO_DRV:C409 -> SCCI_RH_DRV:C409
- C410: footprint ato_drv:C_0805_2012Metric -> scci_rh_drv:C_0805_2012Metric; symbol ATO_DRV:C410 -> SCCI_RH_DRV:C410
- C411: footprint ato_drv:C_0805_2012Metric -> scci_rh_drv:C_0805_2012Metric; symbol ATO_DRV:C411 -> SCCI_RH_DRV:C411
- C412: footprint ato_drv:C_0805_2012Metric -> scci_rh_drv:C_0805_2012Metric; symbol ATO_DRV:C412 -> SCCI_RH_DRV:C412
- C413: footprint ato_drv:C_0805_2012Metric -> scci_rh_drv:C_0805_2012Metric; symbol ATO_DRV:C413 -> SCCI_RH_DRV:C413
- C414: footprint ato_drv:C_0805_2012Metric -> scci_rh_drv:C_0805_2012Metric; symbol ATO_DRV:C414 -> SCCI_RH_DRV:C414
- C415: footprint ato_drv:C_0805_2012Metric -> scci_rh_drv:C_0805_2012Metric; symbol ATO_DRV:C415 -> SCCI_RH_DRV:C415
- C416: footprint ato_drv:C_0805_2012Metric -> scci_rh_drv:C_0805_2012Metric; symbol ATO_DRV:C416 -> SCCI_RH_DRV:C416
- C417: footprint ato_drv:C_0805_2012Metric -> scci_rh_drv:C_0805_2012Metric; symbol ATO_DRV:C417 -> SCCI_RH_DRV:C417
- C418: footprint ato_drv:C_0805_2012Metric -> scci_rh_drv:C_0805_2012Metric; symbol ATO_DRV:C418 -> SCCI_RH_DRV:C418
- C419: footprint ato_drv:C_0805_2012Metric -> scci_rh_drv:C_0805_2012Metric; symbol ATO_DRV:C419 -> SCCI_RH_DRV:C419
- C420: footprint ato_drv:C_0805_2012Metric -> scci_rh_drv:C_0805_2012Metric; symbol ATO_DRV:C420 -> SCCI_RH_DRV:C420
- R400: footprint ato_drv:R_0805_2012Metric -> scci_rh_drv:R_0805_2012Metric; symbol ATO_DRV:R400 -> SCCI_RH_DRV:R400
- R401: footprint ato_drv:R_0805_2012Metric -> scci_rh_drv:R_0805_2012Metric; symbol ATO_DRV:R401 -> SCCI_RH_DRV:R401
- R402: footprint ato_drv:R_0805_2012Metric -> scci_rh_drv:R_0805_2012Metric; symbol ATO_DRV:R402 -> SCCI_RH_DRV:R402
- R403: footprint ato_drv:R_0805_2012Metric -> scci_rh_drv:R_0805_2012Metric; symbol ATO_DRV:R403 -> SCCI_RH_DRV:R403
- R404: footprint ato_drv:R_0805_2012Metric -> scci_rh_drv:R_0805_2012Metric; symbol ATO_DRV:R404 -> SCCI_RH_DRV:R404
- R405: footprint ato_drv:R_0805_2012Metric -> scci_rh_drv:R_0805_2012Metric; symbol ATO_DRV:R405 -> SCCI_RH_DRV:R405
- R406: footprint ato_drv:R_0805_2012Metric -> scci_rh_drv:R_0805_2012Metric; symbol ATO_DRV:R406 -> SCCI_RH_DRV:R406
- R407: footprint ato_drv:R_0805_2012Metric -> scci_rh_drv:R_0805_2012Metric; symbol ATO_DRV:R407 -> SCCI_RH_DRV:R407
- R408: footprint ato_drv:R_0805_2012Metric -> scci_rh_drv:R_0805_2012Metric; symbol ATO_DRV:R408 -> SCCI_RH_DRV:R408
- R409: footprint ato_drv:R_0805_2012Metric -> scci_rh_drv:R_0805_2012Metric; symbol ATO_DRV:R409 -> SCCI_RH_DRV:R409
- R410: footprint ato_drv:R_0805_2012Metric -> scci_rh_drv:R_0805_2012Metric; symbol ATO_DRV:R410 -> SCCI_RH_DRV:R410
- U400: footprint ato_drv:TSOT-23-6 -> scci_rh_drv:TSOT-23-6; symbol ATO_DRV:U400 -> SCCI_RH_DRV:U400
- U401: footprint ato_drv:SOT-23-5 -> scci_rh_drv:SOT-23-5; symbol ATO_DRV:U401 -> SCCI_RH_DRV:U401
- U402: footprint ato_drv:SOT-23-6 -> scci_rh_drv:SOT-23-6; symbol ATO_DRV:U402 -> SCCI_RH_DRV:U402
- U403: footprint ato_drv:SOT-23-6 -> scci_rh_drv:SOT-23-6; symbol ATO_DRV:U403 -> SCCI_RH_DRV:U403
- U404: footprint ato_drv:SOT-23-5 -> scci_rh_drv:SOT-23-5; symbol ATO_DRV:U404 -> SCCI_RH_DRV:U404
- U405: footprint ato_drv:SOT-23-5 -> scci_rh_drv:SOT-23-5; symbol ATO_DRV:U405 -> SCCI_RH_DRV:U405
- U406: footprint ato_drv:SOT-23-5 -> scci_rh_drv:SOT-23-5; symbol ATO_DRV:U406 -> SCCI_RH_DRV:U406
- U407: footprint ato_drv:SOT-23-5 -> scci_rh_drv:SOT-23-5; symbol ATO_DRV:U407 -> SCCI_RH_DRV:U407
- U408: footprint ato_drv:SOT-23-5 -> scci_rh_drv:SOT-23-5; symbol ATO_DRV:U408 -> SCCI_RH_DRV:U408
- U409: footprint ato_drv:SOT-23-5 -> scci_rh_drv:SOT-23-5; symbol ATO_DRV:U409 -> SCCI_RH_DRV:U409
- U410: footprint ato_drv:SOT-23-6 -> scci_rh_drv:SOT-23-6; symbol ATO_DRV:U410 -> SCCI_RH_DRV:U410
- U411: footprint ato_drv:SOT-23-6 -> scci_rh_drv:SOT-23-6; symbol ATO_DRV:U411 -> SCCI_RH_DRV:U411
- U412: footprint ato_drv:SOT-23-5 -> scci_rh_drv:SOT-23-5; symbol ATO_DRV:U412 -> SCCI_RH_DRV:U412
- U413: footprint ato_drv:VSSOP-8_2.3x2mm_P0.5mm -> scci_rh_drv:VSSOP-8_2.3x2mm_P0.5mm; symbol ATO_DRV:U413 -> SCCI_RH_DRV:U413
- U414: footprint ato_drv:SOT-23-5 -> scci_rh_drv:SOT-23-5; symbol ATO_DRV:U414 -> SCCI_RH_DRV:U414
- U415: footprint ato_drv:VSSOP-8_2.3x2mm_P0.5mm -> scci_rh_drv:VSSOP-8_2.3x2mm_P0.5mm; symbol ATO_DRV:U415 -> SCCI_RH_DRV:U415
- U416: footprint ato_drv:VSSOP-8_2.3x2mm_P0.5mm -> scci_rh_drv:VSSOP-8_2.3x2mm_P0.5mm; symbol ATO_DRV:U416 -> SCCI_RH_DRV:U416
- U417: footprint ato_drv:SOT-23-6 -> scci_rh_drv:SOT-23-6; symbol ATO_DRV:U417 -> SCCI_RH_DRV:U417
- U418: footprint ato_drv:SOT-23-6 -> scci_rh_drv:SOT-23-6; symbol ATO_DRV:U418 -> SCCI_RH_DRV:U418
- U419: footprint ato_drv:SOT-23-5 -> scci_rh_drv:SOT-23-5; symbol ATO_DRV:U419 -> SCCI_RH_DRV:U419
- U420: footprint ato_drv:SOT-23-5 -> scci_rh_drv:SOT-23-5; symbol ATO_DRV:U420 -> SCCI_RH_DRV:U420
Other:
- company: Project ATO -> Project SCCI RH
- title: ATO S4 / Source 1: independent duration and sticky admission -> Project SCCI RH S4 / Source 1: independent duration and sticky admission
