File: electronics/stage4/integrated-pcb/boards/contact-router/source1.kicad_sch (KiCad schematic)
At the start: 12 parts, among them J40200 DRIVER A / MONITORED RETURN, U40200 TMUX6208PWR, U40201 TMUX6208PWR

Commit message: Rename project to Project SCCI RH across research and engineering
Parts:
- C40200: footprint ato_rte:C_0805_2012Metric -> scci_rh_rte:C_0805_2012Metric; symbol ATO_RTE:C200 -> SCCI_RH_RTE:C200
- C40201: footprint ato_rte:C_0805_2012Metric -> scci_rh_rte:C_0805_2012Metric; symbol ATO_RTE:C201 -> SCCI_RH_RTE:C201
- C40202: footprint ato_rte:C_0805_2012Metric -> scci_rh_rte:C_0805_2012Metric; symbol ATO_RTE:C202 -> SCCI_RH_RTE:C202
- C40203: footprint ato_rte:C_0805_2012Metric -> scci_rh_rte:C_0805_2012Metric; symbol ATO_RTE:C203 -> SCCI_RH_RTE:C203
- J40200: footprint ato_rte:PinHeader_1x03_P2.54mm_Vertical -> scci_rh_rte:PinHeader_1x03_P2.54mm_Vertical; symbol ATO_RTE:J200 -> SCCI_RH_RTE:J200
- R40200: footprint ato_rte:R_0805_2012Metric -> scci_rh_rte:R_0805_2012Metric; symbol ATO_RTE:R200 -> SCCI_RH_RTE:R200
- R40201: footprint ato_rte:R_0805_2012Metric -> scci_rh_rte:R_0805_2012Metric; symbol ATO_RTE:R201 -> SCCI_RH_RTE:R201
- R40202: footprint ato_rte:R_0805_2012Metric -> scci_rh_rte:R_0805_2012Metric; symbol ATO_RTE:R202 -> SCCI_RH_RTE:R202
- R40203: footprint ato_rte:R_0805_2012Metric -> scci_rh_rte:R_0805_2012Metric; symbol ATO_RTE:R203 -> SCCI_RH_RTE:R203
- R40204: footprint ato_rte:R_0805_2012Metric -> scci_rh_rte:R_0805_2012Metric; symbol ATO_RTE:R204 -> SCCI_RH_RTE:R204
- U40200: footprint ato_rte:TSSOP-16_4.4x5mm_P0.65mm -> scci_rh_rte:TSSOP-16_4.4x5mm_P0.65mm; symbol ATO_RTE:U200 -> SCCI_RH_RTE:U200
- U40201: footprint ato_rte:TSSOP-16_4.4x5mm_P0.65mm -> scci_rh_rte:TSSOP-16_4.4x5mm_P0.65mm; symbol ATO_RTE:U201 -> SCCI_RH_RTE:U201
Other:
- company: Project ATO -> Project SCCI RH
- title: ATO S4 / Source 1 / sixteen-contact output -> Project SCCI RH S4 / Source 1 / sixteen-contact output
