File: electronics/stage4/integrated-pcb/boards/controller-carrier/defaults_3.kicad_sch (KiCad schematic)
At the start: 12 parts

Commit message: Rename project to Project SCCI RH across research and engineering
Parts:
- R80128: footprint ato_controller:R_0805_2012Metric -> scci_rh_controller:R_0805_2012Metric; symbol ATO_CONTROLLER:R128 -> SCCI_RH_CONTROLLER:R128
- R80129: footprint ato_controller:R_0805_2012Metric -> scci_rh_controller:R_0805_2012Metric; symbol ATO_CONTROLLER:R129 -> SCCI_RH_CONTROLLER:R129
- R80130: footprint ato_controller:R_0805_2012Metric -> scci_rh_controller:R_0805_2012Metric; symbol ATO_CONTROLLER:R130 -> SCCI_RH_CONTROLLER:R130
- R80131: footprint ato_controller:R_0805_2012Metric -> scci_rh_controller:R_0805_2012Metric; symbol ATO_CONTROLLER:R131 -> SCCI_RH_CONTROLLER:R131
- R80132: footprint ato_controller:R_0805_2012Metric -> scci_rh_controller:R_0805_2012Metric; symbol ATO_CONTROLLER:R132 -> SCCI_RH_CONTROLLER:R132
- R80133: footprint ato_controller:R_0805_2012Metric -> scci_rh_controller:R_0805_2012Metric; symbol ATO_CONTROLLER:R133 -> SCCI_RH_CONTROLLER:R133
- R80134: footprint ato_controller:R_0805_2012Metric -> scci_rh_controller:R_0805_2012Metric; symbol ATO_CONTROLLER:R134 -> SCCI_RH_CONTROLLER:R134
- R80135: footprint ato_controller:R_0805_2012Metric -> scci_rh_controller:R_0805_2012Metric; symbol ATO_CONTROLLER:R135 -> SCCI_RH_CONTROLLER:R135
- R80136: footprint ato_controller:R_0805_2012Metric -> scci_rh_controller:R_0805_2012Metric; symbol ATO_CONTROLLER:R136 -> SCCI_RH_CONTROLLER:R136
- R80137: footprint ato_controller:R_0805_2012Metric -> scci_rh_controller:R_0805_2012Metric; symbol ATO_CONTROLLER:R137 -> SCCI_RH_CONTROLLER:R137
- R80138: footprint ato_controller:R_0805_2012Metric -> scci_rh_controller:R_0805_2012Metric; symbol ATO_CONTROLLER:R138 -> SCCI_RH_CONTROLLER:R138
- R80139: footprint ato_controller:R_0805_2012Metric -> scci_rh_controller:R_0805_2012Metric; symbol ATO_CONTROLLER:R139 -> SCCI_RH_CONTROLLER:R139
Other:
- company: Project ATO -> Project SCCI RH
- title: ATO S4 / Passive reset defaults / explicit recovery / 3 -> Project SCCI RH S4 / Passive reset defaults / explicit recovery / 3
