File: electronics/stage4/integrated-pcb/boards/controller-carrier/handoff.kicad_sch (KiCad schematic)
At the start: 4 parts, among them J80010 RAW MONITOR, J80011 ISOLATED RECORDING HOST, J80012 SHARED CHARGE ENDPOINT SPI, J80013 DOSE / MONITOR REARM

Commit message: Rename project to Project SCCI RH across research and engineering
Parts:
- J80010: footprint ato_controller:PinHeader_1x06_P2.54mm_Vertical -> scci_rh_controller:PinHeader_1x06_P2.54mm_Vertical; symbol ATO_CONTROLLER:J10 -> SCCI_RH_CONTROLLER:J10
- J80011: footprint ato_controller:PinHeader_1x10_P2.54mm_Vertical -> scci_rh_controller:PinHeader_1x10_P2.54mm_Vertical; symbol ATO_CONTROLLER:J11 -> SCCI_RH_CONTROLLER:J11
- J80012: footprint ato_controller:PinHeader_1x07_P2.54mm_Vertical -> scci_rh_controller:PinHeader_1x07_P2.54mm_Vertical; symbol ATO_CONTROLLER:J12 -> SCCI_RH_CONTROLLER:J12
- J80013: footprint ato_controller:PinHeader_1x05_P2.54mm_Vertical -> scci_rh_controller:PinHeader_1x05_P2.54mm_Vertical; symbol ATO_CONTROLLER:J13 -> SCCI_RH_CONTROLLER:J13
Other:
- company: Project ATO -> Project SCCI RH
- title: ATO S4 / Matched peripheral handoff connectors -> Project SCCI RH S4 / Matched peripheral handoff connectors
