File: electronics/stage4/integrated-pcb/boards/controller-carrier/power.kicad_sch (KiCad schematic)
At the start: 7 parts, among them J80002 SWD / TARGET VREF, J80003 RESET SHORTING HEADER

Commit message: Rename project to Project SCCI RH across research and engineering
Parts:
- C80001: footprint ato_controller:C_1206_3216Metric -> scci_rh_controller:C_1206_3216Metric; symbol ATO_CONTROLLER:C1 -> SCCI_RH_CONTROLLER:C1
- C80002: footprint ato_controller:C_1206_3216Metric -> scci_rh_controller:C_1206_3216Metric; symbol ATO_CONTROLLER:C2 -> SCCI_RH_CONTROLLER:C2
- C80003: footprint ato_controller:C_1206_3216Metric -> scci_rh_controller:C_1206_3216Metric; symbol ATO_CONTROLLER:C3 -> SCCI_RH_CONTROLLER:C3
- J80002: footprint ato_controller:PinHeader_1x06_P2.54mm_Vertical -> scci_rh_controller:PinHeader_1x06_P2.54mm_Vertical; symbol ATO_CONTROLLER:J2 -> SCCI_RH_CONTROLLER:J2
- J80003: footprint ato_controller:PinHeader_1x02_P2.54mm_Vertical -> scci_rh_controller:PinHeader_1x02_P2.54mm_Vertical; symbol ATO_CONTROLLER:J3 -> SCCI_RH_CONTROLLER:J3
- R80001: footprint ato_controller:R_0805_2012Metric -> scci_rh_controller:R_0805_2012Metric; symbol ATO_CONTROLLER:R1 -> SCCI_RH_CONTROLLER:R1
- R80002: footprint ato_controller:R_0805_2012Metric -> scci_rh_controller:R_0805_2012Metric; symbol ATO_CONTROLLER:R2 -> SCCI_RH_CONTROLLER:R2
Other:
- company: Project ATO -> Project SCCI RH
- title: ATO S4 / Module normal-voltage supply and SWD -> Project SCCI RH S4 / Module normal-voltage supply and SWD
