File: electronics/stage4/integrated-pcb/boards/controller-carrier/processor.kicad_sch (KiCad schematic)
At the start: 1 part, among them U80001 FANSTEL BT40F / nRF5340

Commit message: Rename project to Project SCCI RH across research and engineering
Parts:
- U80001: footprint ato_controller:BT40F_Manufacturer_66Pad -> scci_rh_controller:BT40F_Manufacturer_66Pad; symbol ATO_CONTROLLER:U1 -> SCCI_RH_CONTROLLER:U1
Other:
- company: Project ATO -> Project SCCI RH
- title: ATO S4 / BT40F / actual nRF5340 physical pads -> Project SCCI RH S4 / BT40F / actual nRF5340 physical pads
