File: electronics/stage4/integrated-pcb/boards/current-driver/current_driver.kicad_pcb (KiCad board)
At the start: 4 copper layers, 175 x 155 mm, 160 parts, among them J20001 QUALIFIED EXTERNAL RAILS, J20002 MCU SPI / PRELOAD INHIBITED, J20003 MCU PHASE / EXPLICIT REARM, J20004 EXTERNAL HEALTH CONTRACTS, J20005 STATUS ONLY / NOT DELIVERY EV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, J20100 EXTERNAL ROUTER / MONITOR, J20200 EXTERNAL ROUTER / MONITOR, Q20100 BSP89H6327XTSA1, Q20200 BSP89H6327XTSA1, U20001 DAC80502DRXR, U20100 OPA192IDBVR, U20101 TMUX7212PWR, U20102 TMUX6219DGKR, U20103 TMUX6219DGKR, U20200 OPA192IDBVR, U20201 TMUX7212PWR, U20202 TMUX6219DGKR, U20203 TMUX6219DGKR, U20300 LTC6993HS6-1#TRPBF, U20301 SN74LVC1G86DBVR, U20302 SN74LVC1G11DBVR, U20303 SN74LVC1G11DBVR, U20304 SN74LVC1G08DBVR, U20305 SN74LVC1G04DBVR, U20306 SN74LVC1G04DBVR, U20307 SN74LVC1G08DBVR, U20308 SN74LVC1G04DBVR, U20309 SN74LVC1G08DBVR, U20310 SN74LVC1G11DBVR, U20311 SN74LVC1G11DBVR, U20312 SN74LVC1G04DBVR, U20313 SN74LVC1G74DCUR, U20314 SN74LVC1G32DBVR, U20315 SN74LVC1G74DCUR, U20316 SN74LVC1G74DCUR, U20317 SN74LVC1G11DBVR, U20318 SN74LVC1G11DBVR, U20319 SN74LVC1G08DBVR, U20320 SN74LVC1G08DBVR, U20400 LTC6993HS6-1#TRPBF, U20401 SN74LVC1G86DBVR, U20402 SN74LVC1G11DBVR, U20403 SN74LVC1G11DBVR, U20404 SN74LVC1G08DBVR, U20405 SN74LVC1G04DBVR, U20406 SN74LVC1G04DBVR, U20407 SN74LVC1G08DBVR, U20408 SN74LVC1G04DBVR, U20409 SN74LVC1G08DBVR, U20410 SN74LVC1G11DBVR, U20411 SN74LVC1G11DBVR, U20412 SN74LVC1G04DBVR, U20413 SN74LVC1G74DCUR, U20414 SN74LVC1G32DBVR, U20415 SN74LVC1G74DCUR, U20416 SN74LVC1G74DCUR, U20417 SN74LVC1G11DBVR, U20418 SN74LVC1G11DBVR, U20419 SN74LVC1G08DBVR, U20420 SN74LVC1G08DBVR

Commit message: Rename project to Project SCCI RH across research and engineering
Parts:
- C20001, C20002, C20003, C20100, C20101, C20102, C20103, C20104, C20105, C20200, C20201, C20202, C20203, C20204, C20205, C20300, C20301, C20302, C20303, C20304, C20305, C20306, C20307, C20308, C20309, C20310, C20311, C20312, C20313, C20314, C20315, C20316, C20317, C20318, C20319, C20320, C20400, C20401, C20402, C20403, C20404, C20405, C20406, C20407, C20408, C20409, C20410, C20411, C20412, C20413, C20414, C20415, C20416, C20417, C20418, C20419, C20420: footprint ato_drv:C_0805_2012Metric -> scci_rh_drv:C_0805_2012Metric
- J20001: footprint ato_drv:PinHeader_1x05_P2.54mm_Vertical -> scci_rh_drv:PinHeader_1x05_P2.54mm_Vertical
- J20002, J20100, J20200: footprint ato_drv:PinHeader_1x04_P2.54mm_Vertical -> scci_rh_drv:PinHeader_1x04_P2.54mm_Vertical
- J20003, J20005: footprint ato_drv:PinHeader_1x09_P2.54mm_Vertical -> scci_rh_drv:PinHeader_1x09_P2.54mm_Vertical
- J20004: footprint ato_drv:PinHeader_1x11_P2.54mm_Vertical -> scci_rh_drv:PinHeader_1x11_P2.54mm_Vertical
- Q20100, Q20200: footprint ato_drv:BSP89_PG-SOT223-4_DrainTab -> scci_rh_drv:BSP89_PG-SOT223-4_DrainTab
- R20001, R20002, R20003, R20004, R20005, R20100, R20101, R20102, R20103, R20104, R20105, R20200, R20201, R20202, R20203, R20204, R20205, R20300, R20301, R20302, R20303, R20304, R20305, R20306, R20307, R20308, R20309, R20310, R20400, R20401, R20402, R20403, R20404, R20405, R20406, R20407, R20408, R20409, R20410: footprint ato_drv:R_0805_2012Metric -> scci_rh_drv:R_0805_2012Metric
- U20001: footprint ato_drv:Texas_DRX_WSON-10_2.5x2.5mm_P0.5mm -> scci_rh_drv:Texas_DRX_WSON-10_2.5x2.5mm_P0.5mm
- U20100, U20200, U20301, U20304, U20305, U20306, U20307, U20308, U20309, U20312, U20314, U20319, U20320, U20401, U20404, U20405, U20406, U20407, U20408, U20409, U20412, U20414, U20419, U20420: footprint ato_drv:SOT-23-5 -> scci_rh_drv:SOT-23-5
- U20101, U20201: footprint ato_drv:TSSOP-16_4.4x5mm_P0.65mm -> scci_rh_drv:TSSOP-16_4.4x5mm_P0.65mm
- U20102, U20103, U20202, U20203, U20313, U20315, U20316, U20413, U20415, U20416: footprint ato_drv:VSSOP-8_2.3x2mm_P0.5mm -> scci_rh_drv:VSSOP-8_2.3x2mm_P0.5mm
- U20300, U20400: footprint ato_drv:TSOT-23-6 -> scci_rh_drv:TSOT-23-6
- U20302, U20303, U20310, U20311, U20317, U20318, U20402, U20403, U20410, U20411, U20417, U20418: footprint ato_drv:SOT-23-6 -> scci_rh_drv:SOT-23-6
Other:
- board text added: "SCCI_RH / CURRENT DRIVER"
- board text removed: "ATO / CURRENT DRIVER"
