File: electronics/stage4/integrated-pcb/boards/current-driver/current_driver.kicad_sch (KiCad schematic)
At the start: 14 parts, among them J20001 QUALIFIED EXTERNAL RAILS, J20002 MCU SPI / PRELOAD INHIBITED, J20003 MCU PHASE / EXPLICIT REARM, J20004 EXTERNAL HEALTH CONTRACTS, J20005 STATUS ONLY / NOT DELIVERY EV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, U20001 DAC80502DRXR

Commit message: Rename project to Project SCCI RH across research and engineering
Parts:
- C20001: footprint ato_drv:C_0805_2012Metric -> scci_rh_drv:C_0805_2012Metric; symbol ATO_DRV:C1 -> SCCI_RH_DRV:C1
- C20002: footprint ato_drv:C_0805_2012Metric -> scci_rh_drv:C_0805_2012Metric; symbol ATO_DRV:C2 -> SCCI_RH_DRV:C2
- C20003: footprint ato_drv:C_0805_2012Metric -> scci_rh_drv:C_0805_2012Metric; symbol ATO_DRV:C3 -> SCCI_RH_DRV:C3
- J20001: footprint ato_drv:PinHeader_1x05_P2.54mm_Vertical -> scci_rh_drv:PinHeader_1x05_P2.54mm_Vertical; symbol ATO_DRV:J1 -> SCCI_RH_DRV:J1
- J20002: footprint ato_drv:PinHeader_1x04_P2.54mm_Vertical -> scci_rh_drv:PinHeader_1x04_P2.54mm_Vertical; symbol ATO_DRV:J2 -> SCCI_RH_DRV:J2
- J20003: footprint ato_drv:PinHeader_1x09_P2.54mm_Vertical -> scci_rh_drv:PinHeader_1x09_P2.54mm_Vertical; symbol ATO_DRV:J3 -> SCCI_RH_DRV:J3
- J20004: footprint ato_drv:PinHeader_1x11_P2.54mm_Vertical -> scci_rh_drv:PinHeader_1x11_P2.54mm_Vertical; symbol ATO_DRV:J4 -> SCCI_RH_DRV:J4
- J20005: footprint ato_drv:PinHeader_1x09_P2.54mm_Vertical -> scci_rh_drv:PinHeader_1x09_P2.54mm_Vertical; symbol ATO_DRV:J5 -> SCCI_RH_DRV:J5
- R20001: footprint ato_drv:R_0805_2012Metric -> scci_rh_drv:R_0805_2012Metric; symbol ATO_DRV:R1 -> SCCI_RH_DRV:R1
- R20002: footprint ato_drv:R_0805_2012Metric -> scci_rh_drv:R_0805_2012Metric; symbol ATO_DRV:R2 -> SCCI_RH_DRV:R2
- R20003: footprint ato_drv:R_0805_2012Metric -> scci_rh_drv:R_0805_2012Metric; symbol ATO_DRV:R3 -> SCCI_RH_DRV:R3
- R20004: footprint ato_drv:R_0805_2012Metric -> scci_rh_drv:R_0805_2012Metric; symbol ATO_DRV:R4 -> SCCI_RH_DRV:R4
- R20005: footprint ato_drv:R_0805_2012Metric -> scci_rh_drv:R_0805_2012Metric; symbol ATO_DRV:R5 -> SCCI_RH_DRV:R5
- U20001: footprint ato_drv:Texas_DRX_WSON-10_2.5x2.5mm_P0.5mm -> scci_rh_drv:Texas_DRX_WSON-10_2.5x2.5mm_P0.5mm; symbol ATO_DRV:U1 -> SCCI_RH_DRV:U1
Other:
- company: Project ATO -> Project SCCI RH
- title: ATO S4 / Dual setpoint and external contracts -> Project SCCI RH S4 / Dual setpoint and external contracts
