File: electronics/stage4/integrated-pcb/boards/monitoring-transport/health.kicad_sch (KiCad schematic)
At the start: 4 parts

Commit message: Rename project to Project SCCI RH across research and engineering
Parts:
- R70120: footprint ato_transport:R_0805_2012Metric -> scci_rh_transport:R_0805_2012Metric; symbol ATO_TRANSPORT:R120 -> SCCI_RH_TRANSPORT:R120
- R70121: footprint ato_transport:R_0805_2012Metric -> scci_rh_transport:R_0805_2012Metric; symbol ATO_TRANSPORT:R121 -> SCCI_RH_TRANSPORT:R121
- R70122: footprint ato_transport:R_0805_2012Metric -> scci_rh_transport:R_0805_2012Metric; symbol ATO_TRANSPORT:R122 -> SCCI_RH_TRANSPORT:R122
- R70123: footprint ato_transport:R_0805_2012Metric -> scci_rh_transport:R_0805_2012Metric; symbol ATO_TRANSPORT:R123 -> SCCI_RH_TRANSPORT:R123
Other:
- company: Project ATO -> Project SCCI RH
- title: ATO S4 / Divided power observations -> Project SCCI RH S4 / Divided power observations
