File: electronics/stage4/integrated-pcb/boards/power/enable.kicad_sch (KiCad schematic)
At the start: 20 parts, among them U60200 TPS3700DDCR, U60201 TPS3700DDCR, U60202 TPS3700DDCR

Commit message: Rename project to Project SCCI RH across research and engineering
Parts:
- C60200: footprint ato_power:C_1206_3216Metric -> scci_rh_power:C_1206_3216Metric; symbol ATO_POWER:C200 -> SCCI_RH_POWER:C200
- C60201: footprint ato_power:C_1206_3216Metric -> scci_rh_power:C_1206_3216Metric; symbol ATO_POWER:C201 -> SCCI_RH_POWER:C201
- R62000: footprint ato_power:R_0805_2012Metric -> scci_rh_power:R_0805_2012Metric; symbol ATO_POWER:R2000 -> SCCI_RH_POWER:R2000
- R62001: footprint ato_power:R_0805_2012Metric -> scci_rh_power:R_0805_2012Metric; symbol ATO_POWER:R2001 -> SCCI_RH_POWER:R2001
- R62002: footprint ato_power:R_0805_2012Metric -> scci_rh_power:R_0805_2012Metric; symbol ATO_POWER:R2002 -> SCCI_RH_POWER:R2002
- R62003: footprint ato_power:R_0805_2012Metric -> scci_rh_power:R_0805_2012Metric; symbol ATO_POWER:R2003 -> SCCI_RH_POWER:R2003
- R62004: footprint ato_power:R_0805_2012Metric -> scci_rh_power:R_0805_2012Metric; symbol ATO_POWER:R2004 -> SCCI_RH_POWER:R2004
- R62010: footprint ato_power:R_0805_2012Metric -> scci_rh_power:R_0805_2012Metric; symbol ATO_POWER:R2010 -> SCCI_RH_POWER:R2010
- R62011: footprint ato_power:R_0805_2012Metric -> scci_rh_power:R_0805_2012Metric; symbol ATO_POWER:R2011 -> SCCI_RH_POWER:R2011
- R62012: footprint ato_power:R_0805_2012Metric -> scci_rh_power:R_0805_2012Metric; symbol ATO_POWER:R2012 -> SCCI_RH_POWER:R2012
- R62013: footprint ato_power:R_0805_2012Metric -> scci_rh_power:R_0805_2012Metric; symbol ATO_POWER:R2013 -> SCCI_RH_POWER:R2013
- R62014: footprint ato_power:R_0805_2012Metric -> scci_rh_power:R_0805_2012Metric; symbol ATO_POWER:R2014 -> SCCI_RH_POWER:R2014
- R62020: footprint ato_power:R_0805_2012Metric -> scci_rh_power:R_0805_2012Metric; symbol ATO_POWER:R2020 -> SCCI_RH_POWER:R2020
- R62021: footprint ato_power:R_0805_2012Metric -> scci_rh_power:R_0805_2012Metric; symbol ATO_POWER:R2021 -> SCCI_RH_POWER:R2021
- R62022: footprint ato_power:R_0805_2012Metric -> scci_rh_power:R_0805_2012Metric; symbol ATO_POWER:R2022 -> SCCI_RH_POWER:R2022
- R62023: footprint ato_power:R_0805_2012Metric -> scci_rh_power:R_0805_2012Metric; symbol ATO_POWER:R2023 -> SCCI_RH_POWER:R2023
- R62024: footprint ato_power:R_0805_2012Metric -> scci_rh_power:R_0805_2012Metric; symbol ATO_POWER:R2024 -> SCCI_RH_POWER:R2024
- U60200: footprint ato_power:SOT-23-6 -> scci_rh_power:SOT-23-6; symbol ATO_POWER:U200 -> SCCI_RH_POWER:U200
- U60201: footprint ato_power:SOT-23-6 -> scci_rh_power:SOT-23-6; symbol ATO_POWER:U201 -> SCCI_RH_POWER:U201
- U60202: footprint ato_power:SOT-23-6 -> scci_rh_power:SOT-23-6; symbol ATO_POWER:U202 -> SCCI_RH_POWER:U202
Other:
- company: Project ATO -> Project SCCI RH
- title: ATO S4 / Native battery and startup qualification -> Project SCCI RH S4 / Native battery and startup qualification
