File: electronics/stage4/integrated-pcb/boards/recording-front-end/bank0.kicad_sch (KiCad schematic)
At the start: 27 parts, among them U30020 TMUX7412FRRPR, U30100 TMUX6219DGKR, U30101 TMUX6219DGKR, U30102 TMUX6219DGKR, U30103 TMUX6219DGKR

Commit message: Rename project to Project SCCI RH across research and engineering
Parts:
- C30020: footprint ato_afe:C_0805_2012Metric -> scci_rh_afe:C_0805_2012Metric; symbol ATO_AFE:C20 -> SCCI_RH_AFE:C20
- C30030: footprint ato_afe:C_0805_2012Metric -> scci_rh_afe:C_0805_2012Metric; symbol ATO_AFE:C30 -> SCCI_RH_AFE:C30
- C30100: footprint ato_afe:C_0805_2012Metric -> scci_rh_afe:C_0805_2012Metric; symbol ATO_AFE:C100 -> SCCI_RH_AFE:C100
- C30101: footprint ato_afe:C_0805_2012Metric -> scci_rh_afe:C_0805_2012Metric; symbol ATO_AFE:C101 -> SCCI_RH_AFE:C101
- C30102: footprint ato_afe:C_0805_2012Metric -> scci_rh_afe:C_0805_2012Metric; symbol ATO_AFE:C102 -> SCCI_RH_AFE:C102
- C30103: footprint ato_afe:C_0805_2012Metric -> scci_rh_afe:C_0805_2012Metric; symbol ATO_AFE:C103 -> SCCI_RH_AFE:C103
- C30200: footprint ato_afe:C_0805_2012Metric -> scci_rh_afe:C_0805_2012Metric; symbol ATO_AFE:C200 -> SCCI_RH_AFE:C200
- C30201: footprint ato_afe:C_0805_2012Metric -> scci_rh_afe:C_0805_2012Metric; symbol ATO_AFE:C201 -> SCCI_RH_AFE:C201
- C30202: footprint ato_afe:C_0805_2012Metric -> scci_rh_afe:C_0805_2012Metric; symbol ATO_AFE:C202 -> SCCI_RH_AFE:C202
- C30203: footprint ato_afe:C_0805_2012Metric -> scci_rh_afe:C_0805_2012Metric; symbol ATO_AFE:C203 -> SCCI_RH_AFE:C203
- C30300: footprint ato_afe:C_0805_2012Metric -> scci_rh_afe:C_0805_2012Metric; symbol ATO_AFE:C300 -> SCCI_RH_AFE:C300
- C30301: footprint ato_afe:C_0805_2012Metric -> scci_rh_afe:C_0805_2012Metric; symbol ATO_AFE:C301 -> SCCI_RH_AFE:C301
- C30302: footprint ato_afe:C_0805_2012Metric -> scci_rh_afe:C_0805_2012Metric; symbol ATO_AFE:C302 -> SCCI_RH_AFE:C302
- C30303: footprint ato_afe:C_0805_2012Metric -> scci_rh_afe:C_0805_2012Metric; symbol ATO_AFE:C303 -> SCCI_RH_AFE:C303
- R30100: footprint ato_afe:R_0805_2012Metric -> scci_rh_afe:R_0805_2012Metric; symbol ATO_AFE:R100 -> SCCI_RH_AFE:R100
- R30101: footprint ato_afe:R_0805_2012Metric -> scci_rh_afe:R_0805_2012Metric; symbol ATO_AFE:R101 -> SCCI_RH_AFE:R101
- R30102: footprint ato_afe:R_0805_2012Metric -> scci_rh_afe:R_0805_2012Metric; symbol ATO_AFE:R102 -> SCCI_RH_AFE:R102
- R30103: footprint ato_afe:R_0805_2012Metric -> scci_rh_afe:R_0805_2012Metric; symbol ATO_AFE:R103 -> SCCI_RH_AFE:R103
- R30200: footprint ato_afe:R_0805_2012Metric -> scci_rh_afe:R_0805_2012Metric; symbol ATO_AFE:R200 -> SCCI_RH_AFE:R200
- R30201: footprint ato_afe:R_0805_2012Metric -> scci_rh_afe:R_0805_2012Metric; symbol ATO_AFE:R201 -> SCCI_RH_AFE:R201
- R30202: footprint ato_afe:R_0805_2012Metric -> scci_rh_afe:R_0805_2012Metric; symbol ATO_AFE:R202 -> SCCI_RH_AFE:R202
- R30203: footprint ato_afe:R_0805_2012Metric -> scci_rh_afe:R_0805_2012Metric; symbol ATO_AFE:R203 -> SCCI_RH_AFE:R203
- U30020: footprint ato_afe:Texas_RRP0016A_WQFN16_4x4_P0.65_EP2.6 -> scci_rh_afe:Texas_RRP0016A_WQFN16_4x4_P0.65_EP2.6; symbol ATO_AFE:U20 -> SCCI_RH_AFE:U20
- U30100: footprint ato_afe:VSSOP-8_2.3x2mm_P0.5mm -> scci_rh_afe:VSSOP-8_2.3x2mm_P0.5mm; symbol ATO_AFE:U100 -> SCCI_RH_AFE:U100
- U30101: footprint ato_afe:VSSOP-8_2.3x2mm_P0.5mm -> scci_rh_afe:VSSOP-8_2.3x2mm_P0.5mm; symbol ATO_AFE:U101 -> SCCI_RH_AFE:U101
- U30102: footprint ato_afe:VSSOP-8_2.3x2mm_P0.5mm -> scci_rh_afe:VSSOP-8_2.3x2mm_P0.5mm; symbol ATO_AFE:U102 -> SCCI_RH_AFE:U102
- U30103: footprint ato_afe:VSSOP-8_2.3x2mm_P0.5mm -> scci_rh_afe:VSSOP-8_2.3x2mm_P0.5mm; symbol ATO_AFE:U103 -> SCCI_RH_AFE:U103
Other:
- company: Project ATO -> Project SCCI RH
- title: ATO S4 / Inputs 00-03 / protected recording -> Project SCCI RH S4 / Inputs 00-03 / protected recording
