File: electronics/stage4/integrated-pcb/boards/recording-front-end/bank2.kicad_sch (KiCad schematic)
At the start: 27 parts, among them U30022 TMUX7412FRRPR, U30108 TMUX6219DGKR, U30109 TMUX6219DGKR, U30110 TMUX6219DGKR, U30111 TMUX6219DGKR

Commit message: Rename project to Project SCCI RH across research and engineering
Parts:
- C30022: footprint ato_afe:C_0805_2012Metric -> scci_rh_afe:C_0805_2012Metric; symbol ATO_AFE:C22 -> SCCI_RH_AFE:C22
- C30032: footprint ato_afe:C_0805_2012Metric -> scci_rh_afe:C_0805_2012Metric; symbol ATO_AFE:C32 -> SCCI_RH_AFE:C32
- C30108: footprint ato_afe:C_0805_2012Metric -> scci_rh_afe:C_0805_2012Metric; symbol ATO_AFE:C108 -> SCCI_RH_AFE:C108
- C30109: footprint ato_afe:C_0805_2012Metric -> scci_rh_afe:C_0805_2012Metric; symbol ATO_AFE:C109 -> SCCI_RH_AFE:C109
- C30110: footprint ato_afe:C_0805_2012Metric -> scci_rh_afe:C_0805_2012Metric; symbol ATO_AFE:C110 -> SCCI_RH_AFE:C110
- C30111: footprint ato_afe:C_0805_2012Metric -> scci_rh_afe:C_0805_2012Metric; symbol ATO_AFE:C111 -> SCCI_RH_AFE:C111
- C30208: footprint ato_afe:C_0805_2012Metric -> scci_rh_afe:C_0805_2012Metric; symbol ATO_AFE:C208 -> SCCI_RH_AFE:C208
- C30209: footprint ato_afe:C_0805_2012Metric -> scci_rh_afe:C_0805_2012Metric; symbol ATO_AFE:C209 -> SCCI_RH_AFE:C209
- C30210: footprint ato_afe:C_0805_2012Metric -> scci_rh_afe:C_0805_2012Metric; symbol ATO_AFE:C210 -> SCCI_RH_AFE:C210
- C30211: footprint ato_afe:C_0805_2012Metric -> scci_rh_afe:C_0805_2012Metric; symbol ATO_AFE:C211 -> SCCI_RH_AFE:C211
- C30308: footprint ato_afe:C_0805_2012Metric -> scci_rh_afe:C_0805_2012Metric; symbol ATO_AFE:C308 -> SCCI_RH_AFE:C308
- C30309: footprint ato_afe:C_0805_2012Metric -> scci_rh_afe:C_0805_2012Metric; symbol ATO_AFE:C309 -> SCCI_RH_AFE:C309
- C30310: footprint ato_afe:C_0805_2012Metric -> scci_rh_afe:C_0805_2012Metric; symbol ATO_AFE:C310 -> SCCI_RH_AFE:C310
- C30311: footprint ato_afe:C_0805_2012Metric -> scci_rh_afe:C_0805_2012Metric; symbol ATO_AFE:C311 -> SCCI_RH_AFE:C311
- R30108: footprint ato_afe:R_0805_2012Metric -> scci_rh_afe:R_0805_2012Metric; symbol ATO_AFE:R108 -> SCCI_RH_AFE:R108
- R30109: footprint ato_afe:R_0805_2012Metric -> scci_rh_afe:R_0805_2012Metric; symbol ATO_AFE:R109 -> SCCI_RH_AFE:R109
- R30110: footprint ato_afe:R_0805_2012Metric -> scci_rh_afe:R_0805_2012Metric; symbol ATO_AFE:R110 -> SCCI_RH_AFE:R110
- R30111: footprint ato_afe:R_0805_2012Metric -> scci_rh_afe:R_0805_2012Metric; symbol ATO_AFE:R111 -> SCCI_RH_AFE:R111
- R30208: footprint ato_afe:R_0805_2012Metric -> scci_rh_afe:R_0805_2012Metric; symbol ATO_AFE:R208 -> SCCI_RH_AFE:R208
- R30209: footprint ato_afe:R_0805_2012Metric -> scci_rh_afe:R_0805_2012Metric; symbol ATO_AFE:R209 -> SCCI_RH_AFE:R209
- R30210: footprint ato_afe:R_0805_2012Metric -> scci_rh_afe:R_0805_2012Metric; symbol ATO_AFE:R210 -> SCCI_RH_AFE:R210
- R30211: footprint ato_afe:R_0805_2012Metric -> scci_rh_afe:R_0805_2012Metric; symbol ATO_AFE:R211 -> SCCI_RH_AFE:R211
- U30022: footprint ato_afe:Texas_RRP0016A_WQFN16_4x4_P0.65_EP2.6 -> scci_rh_afe:Texas_RRP0016A_WQFN16_4x4_P0.65_EP2.6; symbol ATO_AFE:U22 -> SCCI_RH_AFE:U22
- U30108: footprint ato_afe:VSSOP-8_2.3x2mm_P0.5mm -> scci_rh_afe:VSSOP-8_2.3x2mm_P0.5mm; symbol ATO_AFE:U108 -> SCCI_RH_AFE:U108
- U30109: footprint ato_afe:VSSOP-8_2.3x2mm_P0.5mm -> scci_rh_afe:VSSOP-8_2.3x2mm_P0.5mm; symbol ATO_AFE:U109 -> SCCI_RH_AFE:U109
- U30110: footprint ato_afe:VSSOP-8_2.3x2mm_P0.5mm -> scci_rh_afe:VSSOP-8_2.3x2mm_P0.5mm; symbol ATO_AFE:U110 -> SCCI_RH_AFE:U110
- U30111: footprint ato_afe:VSSOP-8_2.3x2mm_P0.5mm -> scci_rh_afe:VSSOP-8_2.3x2mm_P0.5mm; symbol ATO_AFE:U111 -> SCCI_RH_AFE:U111
Other:
- company: Project ATO -> Project SCCI RH
- title: ATO S4 / Inputs 08-11 / protected recording -> Project SCCI RH S4 / Inputs 08-11 / protected recording
