File: electronics/stage4/integrated-pcb/boards/recording-front-end/recording_front_end.kicad_pcb (KiCad board)
At the start: 4 copper layers, 155 x 190 mm, 157 parts, among them J30001 EXTERNAL ISOLATED AFE RAILS, J30002 HOST SPI / SUPERVISOR, J30003 18 RECORDING FUNCTIONAL PORTS, J39901 AFE TAP HARNESS, J39902 AFE TAP HARNESS, U30001 ISO6741FDWR, U30002 ISO6741FDWR, U30003 SN74LVC1G04DBVR, U30004 SN74LVC1G08DBVR, U30010 RHD2216, U30020 TMUX7412FRRPR, U30021 TMUX7412FRRPR, U30022 TMUX7412FRRPR, U30023 TMUX7412FRRPR, U30024 TMUX7412FRRPR, U30100 TMUX6219DGKR, U30101 TMUX6219DGKR, U30102 TMUX6219DGKR, U30103 TMUX6219DGKR, U30104 TMUX6219DGKR, U30105 TMUX6219DGKR, U30106 TMUX6219DGKR, U30107 TMUX6219DGKR, U30108 TMUX6219DGKR, U30109 TMUX6219DGKR, U30110 TMUX6219DGKR, U30111 TMUX6219DGKR, U30112 TMUX6219DGKR, U30113 TMUX6219DGKR, U30114 TMUX6219DGKR, U30115 TMUX6219DGKR, U30500 TMUX6219DGKR

Commit message: Rename project to Project SCCI RH across research and engineering
Parts:
- C30001, C30002, C30003, C30004, C30005, C30006, C30010, C30011, C30012, C30013, C30020, C30021, C30022, C30023, C30030, C30031, C30032, C30033, C30100, C30101, C30102, C30103, C30104, C30105, C30106, C30107, C30108, C30109, C30110, C30111, C30112, C30113, C30114, C30115, C30200, C30201, C30202, C30203, C30204, C30205, C30206, C30207, C30208, C30209, C30210, C30211, C30212, C30213, C30214, C30215, C30300, C30301, C30302, C30303, C30304, C30305, C30306, C30307, C30308, C30309, C30310, C30311, C30312, C30313, C30314, C30315, C30500, C30510, C30511, C30512, C30513: footprint ato_afe:C_0805_2012Metric -> scci_rh_afe:C_0805_2012Metric
- J30001: footprint ato_afe:PinHeader_1x04_P2.54mm_Vertical -> scci_rh_afe:PinHeader_1x04_P2.54mm_Vertical
- J30002: footprint ato_afe:PinHeader_1x10_P2.54mm_Vertical -> scci_rh_afe:PinHeader_1x10_P2.54mm_Vertical
- J30003: footprint ato_afe:PinHeader_1x18_P2.54mm_Vertical -> scci_rh_afe:PinHeader_1x18_P2.54mm_Vertical
- R30001, R30002, R30003, R30004, R30005, R30006, R30007, R30008, R30009, R30010, R30011, R30012, R30013, R30014, R30100, R30101, R30102, R30103, R30104, R30105, R30106, R30107, R30108, R30109, R30110, R30111, R30112, R30113, R30114, R30115, R30200, R30201, R30202, R30203, R30204, R30205, R30206, R30207, R30208, R30209, R30210, R30211, R30212, R30213, R30214, R30215, R30500, R30501, R30502, R30503: footprint ato_afe:R_0805_2012Metric -> scci_rh_afe:R_0805_2012Metric
- U30001, U30002: footprint ato_afe:SOIC-16W_7.5x10.3mm_P1.27mm -> scci_rh_afe:SOIC-16W_7.5x10.3mm_P1.27mm
- U30003, U30004: footprint ato_afe:SOT-23-5 -> scci_rh_afe:SOT-23-5
- U30010: footprint ato_afe:RHD2216_QFN56_8x8_P0.5_EP6.1 -> scci_rh_afe:RHD2216_QFN56_8x8_P0.5_EP6.1
- U30020, U30021, U30022, U30023, U30024: footprint ato_afe:Texas_RRP0016A_WQFN16_4x4_P0.65_EP2.6 -> scci_rh_afe:Texas_RRP0016A_WQFN16_4x4_P0.65_EP2.6
- U30100, U30101, U30102, U30103, U30104, U30105, U30106, U30107, U30108, U30109, U30110, U30111, U30112, U30113, U30114, U30115, U30500: footprint ato_afe:VSSOP-8_2.3x2mm_P0.5mm -> scci_rh_afe:VSSOP-8_2.3x2mm_P0.5mm
Other:
- board text added: "SCCI_RH / RECORDING FRONT END"
- board text removed: "ATO / RECORDING FRONT END"
