File: electronics/stage4/integrated-pcb/boards/supervision/admission_2.kicad_sch (KiCad schematic)
At the start: 27 parts, among them U50900 SN74LVC1G74DCUR, U51060 SN74LVC1G04DBVR, U51061 SN74LVC1G11DBVR, U51062 SN74LVC1G11DBVR, U51063 SN74LVC1G08DBVR, U51064 SN74LVC1G11DBVR, U51065 SN74LVC1G08DBVR, U51066 SN74LVC1G08DBVR, U51067 SN74LVC1G04DBVR, U51068 SN74LVC1G04DBVR, U51069 SN74LVC1G04DBVR, U51070 SN74LVC1G11DBVR, U51097 SN74LVC1G32DBVR

Commit message: Rename project to Project SCCI RH across research and engineering
Parts:
- C50900: footprint ato_sup:C_0805_2012Metric -> scci_rh_sup:C_0805_2012Metric; symbol ATO_SUP:C900 -> SCCI_RH_SUP:C900
- C51059: footprint ato_sup:C_0805_2012Metric -> scci_rh_sup:C_0805_2012Metric; symbol ATO_SUP:C1059 -> SCCI_RH_SUP:C1059
- C51060: footprint ato_sup:C_0805_2012Metric -> scci_rh_sup:C_0805_2012Metric; symbol ATO_SUP:C1060 -> SCCI_RH_SUP:C1060
- C51061: footprint ato_sup:C_0805_2012Metric -> scci_rh_sup:C_0805_2012Metric; symbol ATO_SUP:C1061 -> SCCI_RH_SUP:C1061
- C51062: footprint ato_sup:C_0805_2012Metric -> scci_rh_sup:C_0805_2012Metric; symbol ATO_SUP:C1062 -> SCCI_RH_SUP:C1062
- C51063: footprint ato_sup:C_0805_2012Metric -> scci_rh_sup:C_0805_2012Metric; symbol ATO_SUP:C1063 -> SCCI_RH_SUP:C1063
- C51064: footprint ato_sup:C_0805_2012Metric -> scci_rh_sup:C_0805_2012Metric; symbol ATO_SUP:C1064 -> SCCI_RH_SUP:C1064
- C51065: footprint ato_sup:C_0805_2012Metric -> scci_rh_sup:C_0805_2012Metric; symbol ATO_SUP:C1065 -> SCCI_RH_SUP:C1065
- C51066: footprint ato_sup:C_0805_2012Metric -> scci_rh_sup:C_0805_2012Metric; symbol ATO_SUP:C1066 -> SCCI_RH_SUP:C1066
- C51067: footprint ato_sup:C_0805_2012Metric -> scci_rh_sup:C_0805_2012Metric; symbol ATO_SUP:C1067 -> SCCI_RH_SUP:C1067
- C51068: footprint ato_sup:C_0805_2012Metric -> scci_rh_sup:C_0805_2012Metric; symbol ATO_SUP:C1068 -> SCCI_RH_SUP:C1068
- C51069: footprint ato_sup:C_0805_2012Metric -> scci_rh_sup:C_0805_2012Metric; symbol ATO_SUP:C1069 -> SCCI_RH_SUP:C1069
- C51070: footprint ato_sup:C_0805_2012Metric -> scci_rh_sup:C_0805_2012Metric; symbol ATO_SUP:C1070 -> SCCI_RH_SUP:C1070
- C51097: footprint ato_sup:C_0805_2012Metric -> scci_rh_sup:C_0805_2012Metric; symbol ATO_SUP:C1097 -> SCCI_RH_SUP:C1097
- U50900: footprint ato_sup:VSSOP-8_2.3x2mm_P0.5mm -> scci_rh_sup:VSSOP-8_2.3x2mm_P0.5mm; symbol ATO_SUP:U900 -> SCCI_RH_SUP:U900
- U51060: footprint ato_sup:SOT-23-5 -> scci_rh_sup:SOT-23-5; symbol ATO_SUP:U1060 -> SCCI_RH_SUP:U1060
- U51061: footprint ato_sup:SOT-23-6 -> scci_rh_sup:SOT-23-6; symbol ATO_SUP:U1061 -> SCCI_RH_SUP:U1061
- U51062: footprint ato_sup:SOT-23-6 -> scci_rh_sup:SOT-23-6; symbol ATO_SUP:U1062 -> SCCI_RH_SUP:U1062
- U51063: footprint ato_sup:SOT-23-5 -> scci_rh_sup:SOT-23-5; symbol ATO_SUP:U1063 -> SCCI_RH_SUP:U1063
- U51064: footprint ato_sup:SOT-23-6 -> scci_rh_sup:SOT-23-6; symbol ATO_SUP:U1064 -> SCCI_RH_SUP:U1064
- U51065: footprint ato_sup:SOT-23-5 -> scci_rh_sup:SOT-23-5; symbol ATO_SUP:U1065 -> SCCI_RH_SUP:U1065
- U51066: footprint ato_sup:SOT-23-5 -> scci_rh_sup:SOT-23-5; symbol ATO_SUP:U1066 -> SCCI_RH_SUP:U1066
- U51067: footprint ato_sup:SOT-23-5 -> scci_rh_sup:SOT-23-5; symbol ATO_SUP:U1067 -> SCCI_RH_SUP:U1067
- U51068: footprint ato_sup:SOT-23-5 -> scci_rh_sup:SOT-23-5; symbol ATO_SUP:U1068 -> SCCI_RH_SUP:U1068
- U51069: footprint ato_sup:SOT-23-5 -> scci_rh_sup:SOT-23-5; symbol ATO_SUP:U1069 -> SCCI_RH_SUP:U1069
- U51070: footprint ato_sup:SOT-23-6 -> scci_rh_sup:SOT-23-6; symbol ATO_SUP:U1070 -> SCCI_RH_SUP:U1070
- U51097: footprint ato_sup:SOT-23-5 -> scci_rh_sup:SOT-23-5; symbol ATO_SUP:U1097 -> SCCI_RH_SUP:U1097
Other:
- company: Project ATO -> Project SCCI RH
- title: ATO S4 / Sticky permission and rearm / 2 -> Project SCCI RH S4 / Sticky permission and rearm / 2
