File: electronics/stage4/integrated-pcb/boards/supervision/host_rails.kicad_sch (KiCad schematic)
At the start: 21 parts, among them U50200 TPS3700DDCR, U50201 TPS3700DDCR, U50202 TPS3700DDCR

Commit message: Rename project to Project SCCI RH across research and engineering
Parts:
- C50200: footprint ato_sup:C_0805_2012Metric -> scci_rh_sup:C_0805_2012Metric; symbol ATO_SUP:C200 -> SCCI_RH_SUP:C200
- C50201: footprint ato_sup:C_0805_2012Metric -> scci_rh_sup:C_0805_2012Metric; symbol ATO_SUP:C201 -> SCCI_RH_SUP:C201
- C50202: footprint ato_sup:C_0805_2012Metric -> scci_rh_sup:C_0805_2012Metric; symbol ATO_SUP:C202 -> SCCI_RH_SUP:C202
- R52000: footprint ato_sup:R_0805_2012Metric -> scci_rh_sup:R_0805_2012Metric; symbol ATO_SUP:R2000 -> SCCI_RH_SUP:R2000
- R52001: footprint ato_sup:R_0805_2012Metric -> scci_rh_sup:R_0805_2012Metric; symbol ATO_SUP:R2001 -> SCCI_RH_SUP:R2001
- R52002: footprint ato_sup:R_0805_2012Metric -> scci_rh_sup:R_0805_2012Metric; symbol ATO_SUP:R2002 -> SCCI_RH_SUP:R2002
- R52003: footprint ato_sup:R_0805_2012Metric -> scci_rh_sup:R_0805_2012Metric; symbol ATO_SUP:R2003 -> SCCI_RH_SUP:R2003
- R52004: footprint ato_sup:R_0805_2012Metric -> scci_rh_sup:R_0805_2012Metric; symbol ATO_SUP:R2004 -> SCCI_RH_SUP:R2004
- R52010: footprint ato_sup:R_0805_2012Metric -> scci_rh_sup:R_0805_2012Metric; symbol ATO_SUP:R2010 -> SCCI_RH_SUP:R2010
- R52011: footprint ato_sup:R_0805_2012Metric -> scci_rh_sup:R_0805_2012Metric; symbol ATO_SUP:R2011 -> SCCI_RH_SUP:R2011
- R52012: footprint ato_sup:R_0805_2012Metric -> scci_rh_sup:R_0805_2012Metric; symbol ATO_SUP:R2012 -> SCCI_RH_SUP:R2012
- R52013: footprint ato_sup:R_0805_2012Metric -> scci_rh_sup:R_0805_2012Metric; symbol ATO_SUP:R2013 -> SCCI_RH_SUP:R2013
- R52014: footprint ato_sup:R_0805_2012Metric -> scci_rh_sup:R_0805_2012Metric; symbol ATO_SUP:R2014 -> SCCI_RH_SUP:R2014
- R52020: footprint ato_sup:R_0805_2012Metric -> scci_rh_sup:R_0805_2012Metric; symbol ATO_SUP:R2020 -> SCCI_RH_SUP:R2020
- R52021: footprint ato_sup:R_0805_2012Metric -> scci_rh_sup:R_0805_2012Metric; symbol ATO_SUP:R2021 -> SCCI_RH_SUP:R2021
- R52022: footprint ato_sup:R_0805_2012Metric -> scci_rh_sup:R_0805_2012Metric; symbol ATO_SUP:R2022 -> SCCI_RH_SUP:R2022
- R52023: footprint ato_sup:R_0805_2012Metric -> scci_rh_sup:R_0805_2012Metric; symbol ATO_SUP:R2023 -> SCCI_RH_SUP:R2023
- R52024: footprint ato_sup:R_0805_2012Metric -> scci_rh_sup:R_0805_2012Metric; symbol ATO_SUP:R2024 -> SCCI_RH_SUP:R2024
- U50200: footprint ato_sup:SOT-23-6 -> scci_rh_sup:SOT-23-6; symbol ATO_SUP:U200 -> SCCI_RH_SUP:U200
- U50201: footprint ato_sup:SOT-23-6 -> scci_rh_sup:SOT-23-6; symbol ATO_SUP:U201 -> SCCI_RH_SUP:U201
- U50202: footprint ato_sup:SOT-23-6 -> scci_rh_sup:SOT-23-6; symbol ATO_SUP:U202 -> SCCI_RH_SUP:U202
Other:
- company: Project ATO -> Project SCCI RH
- title: ATO S4 / Host supply windows -> Project SCCI RH S4 / Host supply windows
