File: electronics/stage4/integrated-pcb/boards/supervision/phase0.kicad_sch (KiCad schematic)
At the start: 28 parts, among them U50910 SN74LVC1G74DCUR, U51071 SN74LVC1G11DBVR, U51072 SN74LVC1G08DBVR, U51073 SN74LVC1G04DBVR, U51074 SN74LVC1G08DBVR, U51075 SN74LVC1G11DBVR, U51076 SN74LVC1G11DBVR, U51077 SN74LVC1G08DBVR, U51078 SN74LVC1G04DBVR, U51079 SN74LVC1G04DBVR, U51080 SN74LVC1G11DBVR, U51081 SN74LVC1G11DBVR, U51082 SN74LVC1G08DBVR, U51083 SN74LVC1G11DBVR

Commit message: Rename project to Project SCCI RH across research and engineering
Parts:
- C50910: footprint ato_sup:C_0805_2012Metric -> scci_rh_sup:C_0805_2012Metric; symbol ATO_SUP:C910 -> SCCI_RH_SUP:C910
- C51071: footprint ato_sup:C_0805_2012Metric -> scci_rh_sup:C_0805_2012Metric; symbol ATO_SUP:C1071 -> SCCI_RH_SUP:C1071
- C51072: footprint ato_sup:C_0805_2012Metric -> scci_rh_sup:C_0805_2012Metric; symbol ATO_SUP:C1072 -> SCCI_RH_SUP:C1072
- C51073: footprint ato_sup:C_0805_2012Metric -> scci_rh_sup:C_0805_2012Metric; symbol ATO_SUP:C1073 -> SCCI_RH_SUP:C1073
- C51074: footprint ato_sup:C_0805_2012Metric -> scci_rh_sup:C_0805_2012Metric; symbol ATO_SUP:C1074 -> SCCI_RH_SUP:C1074
- C51075: footprint ato_sup:C_0805_2012Metric -> scci_rh_sup:C_0805_2012Metric; symbol ATO_SUP:C1075 -> SCCI_RH_SUP:C1075
- C51076: footprint ato_sup:C_0805_2012Metric -> scci_rh_sup:C_0805_2012Metric; symbol ATO_SUP:C1076 -> SCCI_RH_SUP:C1076
- C51077: footprint ato_sup:C_0805_2012Metric -> scci_rh_sup:C_0805_2012Metric; symbol ATO_SUP:C1077 -> SCCI_RH_SUP:C1077
- C51078: footprint ato_sup:C_0805_2012Metric -> scci_rh_sup:C_0805_2012Metric; symbol ATO_SUP:C1078 -> SCCI_RH_SUP:C1078
- C51079: footprint ato_sup:C_0805_2012Metric -> scci_rh_sup:C_0805_2012Metric; symbol ATO_SUP:C1079 -> SCCI_RH_SUP:C1079
- C51080: footprint ato_sup:C_0805_2012Metric -> scci_rh_sup:C_0805_2012Metric; symbol ATO_SUP:C1080 -> SCCI_RH_SUP:C1080
- C51081: footprint ato_sup:C_0805_2012Metric -> scci_rh_sup:C_0805_2012Metric; symbol ATO_SUP:C1081 -> SCCI_RH_SUP:C1081
- C51082: footprint ato_sup:C_0805_2012Metric -> scci_rh_sup:C_0805_2012Metric; symbol ATO_SUP:C1082 -> SCCI_RH_SUP:C1082
- C51083: footprint ato_sup:C_0805_2012Metric -> scci_rh_sup:C_0805_2012Metric; symbol ATO_SUP:C1083 -> SCCI_RH_SUP:C1083
- U50910: footprint ato_sup:VSSOP-8_2.3x2mm_P0.5mm -> scci_rh_sup:VSSOP-8_2.3x2mm_P0.5mm; symbol ATO_SUP:U910 -> SCCI_RH_SUP:U910
- U51071: footprint ato_sup:SOT-23-6 -> scci_rh_sup:SOT-23-6; symbol ATO_SUP:U1071 -> SCCI_RH_SUP:U1071
- U51072: footprint ato_sup:SOT-23-5 -> scci_rh_sup:SOT-23-5; symbol ATO_SUP:U1072 -> SCCI_RH_SUP:U1072
- U51073: footprint ato_sup:SOT-23-5 -> scci_rh_sup:SOT-23-5; symbol ATO_SUP:U1073 -> SCCI_RH_SUP:U1073
- U51074: footprint ato_sup:SOT-23-5 -> scci_rh_sup:SOT-23-5; symbol ATO_SUP:U1074 -> SCCI_RH_SUP:U1074
- U51075: footprint ato_sup:SOT-23-6 -> scci_rh_sup:SOT-23-6; symbol ATO_SUP:U1075 -> SCCI_RH_SUP:U1075
- U51076: footprint ato_sup:SOT-23-6 -> scci_rh_sup:SOT-23-6; symbol ATO_SUP:U1076 -> SCCI_RH_SUP:U1076
- U51077: footprint ato_sup:SOT-23-5 -> scci_rh_sup:SOT-23-5; symbol ATO_SUP:U1077 -> SCCI_RH_SUP:U1077
- U51078: footprint ato_sup:SOT-23-5 -> scci_rh_sup:SOT-23-5; symbol ATO_SUP:U1078 -> SCCI_RH_SUP:U1078
- U51079: footprint ato_sup:SOT-23-5 -> scci_rh_sup:SOT-23-5; symbol ATO_SUP:U1079 -> SCCI_RH_SUP:U1079
- U51080: footprint ato_sup:SOT-23-6 -> scci_rh_sup:SOT-23-6; symbol ATO_SUP:U1080 -> SCCI_RH_SUP:U1080
- U51081: footprint ato_sup:SOT-23-6 -> scci_rh_sup:SOT-23-6; symbol ATO_SUP:U1081 -> SCCI_RH_SUP:U1081
- U51082: footprint ato_sup:SOT-23-5 -> scci_rh_sup:SOT-23-5; symbol ATO_SUP:U1082 -> SCCI_RH_SUP:U1082
- U51083: footprint ato_sup:SOT-23-6 -> scci_rh_sup:SOT-23-6; symbol ATO_SUP:U1083 -> SCCI_RH_SUP:U1083
Other:
- company: Project ATO -> Project SCCI RH
- title: ATO S4 / Source 0 phase permission -> Project SCCI RH S4 / Source 0 phase permission
