File: electronics/stage4/integrated-pcb/integration/master/current-driver/permission0.kicad_sch (KiCad schematic)
At the start: 53 parts, among them U20300 LTC6993HS6-1#TRPBF, U20301 SN74LVC1G86DBVR, U20302 SN74LVC1G11DBVR, U20303 SN74LVC1G11DBVR, U20304 SN74LVC1G08DBVR, U20305 SN74LVC1G04DBVR, U20306 SN74LVC1G04DBVR, U20307 SN74LVC1G08DBVR, U20308 SN74LVC1G04DBVR, U20309 SN74LVC1G08DBVR, U20310 SN74LVC1G11DBVR, U20311 SN74LVC1G11DBVR, U20312 SN74LVC1G04DBVR, U20313 SN74LVC1G74DCUR, U20314 SN74LVC1G32DBVR, U20315 SN74LVC1G74DCUR, U20316 SN74LVC1G74DCUR, U20317 SN74LVC1G11DBVR, U20318 SN74LVC1G11DBVR, U20319 SN74LVC1G08DBVR, U20320 SN74LVC1G08DBVR

Commit message: Rename project to Project SCCI RH across research and engineering
Parts:
- C20300: footprint ato_drv:C_0805_2012Metric -> scci_rh_drv:C_0805_2012Metric; symbol ATO_DRV:C300 -> SCCI_RH_DRV:C300
- C20301: footprint ato_drv:C_0805_2012Metric -> scci_rh_drv:C_0805_2012Metric; symbol ATO_DRV:C301 -> SCCI_RH_DRV:C301
- C20302: footprint ato_drv:C_0805_2012Metric -> scci_rh_drv:C_0805_2012Metric; symbol ATO_DRV:C302 -> SCCI_RH_DRV:C302
- C20303: footprint ato_drv:C_0805_2012Metric -> scci_rh_drv:C_0805_2012Metric; symbol ATO_DRV:C303 -> SCCI_RH_DRV:C303
- C20304: footprint ato_drv:C_0805_2012Metric -> scci_rh_drv:C_0805_2012Metric; symbol ATO_DRV:C304 -> SCCI_RH_DRV:C304
- C20305: footprint ato_drv:C_0805_2012Metric -> scci_rh_drv:C_0805_2012Metric; symbol ATO_DRV:C305 -> SCCI_RH_DRV:C305
- C20306: footprint ato_drv:C_0805_2012Metric -> scci_rh_drv:C_0805_2012Metric; symbol ATO_DRV:C306 -> SCCI_RH_DRV:C306
- C20307: footprint ato_drv:C_0805_2012Metric -> scci_rh_drv:C_0805_2012Metric; symbol ATO_DRV:C307 -> SCCI_RH_DRV:C307
- C20308: footprint ato_drv:C_0805_2012Metric -> scci_rh_drv:C_0805_2012Metric; symbol ATO_DRV:C308 -> SCCI_RH_DRV:C308
- C20309: footprint ato_drv:C_0805_2012Metric -> scci_rh_drv:C_0805_2012Metric; symbol ATO_DRV:C309 -> SCCI_RH_DRV:C309
- C20310: footprint ato_drv:C_0805_2012Metric -> scci_rh_drv:C_0805_2012Metric; symbol ATO_DRV:C310 -> SCCI_RH_DRV:C310
- C20311: footprint ato_drv:C_0805_2012Metric -> scci_rh_drv:C_0805_2012Metric; symbol ATO_DRV:C311 -> SCCI_RH_DRV:C311
- C20312: footprint ato_drv:C_0805_2012Metric -> scci_rh_drv:C_0805_2012Metric; symbol ATO_DRV:C312 -> SCCI_RH_DRV:C312
- C20313: footprint ato_drv:C_0805_2012Metric -> scci_rh_drv:C_0805_2012Metric; symbol ATO_DRV:C313 -> SCCI_RH_DRV:C313
- C20314: footprint ato_drv:C_0805_2012Metric -> scci_rh_drv:C_0805_2012Metric; symbol ATO_DRV:C314 -> SCCI_RH_DRV:C314
- C20315: footprint ato_drv:C_0805_2012Metric -> scci_rh_drv:C_0805_2012Metric; symbol ATO_DRV:C315 -> SCCI_RH_DRV:C315
- C20316: footprint ato_drv:C_0805_2012Metric -> scci_rh_drv:C_0805_2012Metric; symbol ATO_DRV:C316 -> SCCI_RH_DRV:C316
- C20317: footprint ato_drv:C_0805_2012Metric -> scci_rh_drv:C_0805_2012Metric; symbol ATO_DRV:C317 -> SCCI_RH_DRV:C317
- C20318: footprint ato_drv:C_0805_2012Metric -> scci_rh_drv:C_0805_2012Metric; symbol ATO_DRV:C318 -> SCCI_RH_DRV:C318
- C20319: footprint ato_drv:C_0805_2012Metric -> scci_rh_drv:C_0805_2012Metric; symbol ATO_DRV:C319 -> SCCI_RH_DRV:C319
- C20320: footprint ato_drv:C_0805_2012Metric -> scci_rh_drv:C_0805_2012Metric; symbol ATO_DRV:C320 -> SCCI_RH_DRV:C320
- R20300: footprint ato_drv:R_0805_2012Metric -> scci_rh_drv:R_0805_2012Metric; symbol ATO_DRV:R300 -> SCCI_RH_DRV:R300
- R20301: footprint ato_drv:R_0805_2012Metric -> scci_rh_drv:R_0805_2012Metric; symbol ATO_DRV:R301 -> SCCI_RH_DRV:R301
- R20302: footprint ato_drv:R_0805_2012Metric -> scci_rh_drv:R_0805_2012Metric; symbol ATO_DRV:R302 -> SCCI_RH_DRV:R302
- R20303: footprint ato_drv:R_0805_2012Metric -> scci_rh_drv:R_0805_2012Metric; symbol ATO_DRV:R303 -> SCCI_RH_DRV:R303
- R20304: footprint ato_drv:R_0805_2012Metric -> scci_rh_drv:R_0805_2012Metric; symbol ATO_DRV:R304 -> SCCI_RH_DRV:R304
- R20305: footprint ato_drv:R_0805_2012Metric -> scci_rh_drv:R_0805_2012Metric; symbol ATO_DRV:R305 -> SCCI_RH_DRV:R305
- R20306: footprint ato_drv:R_0805_2012Metric -> scci_rh_drv:R_0805_2012Metric; symbol ATO_DRV:R306 -> SCCI_RH_DRV:R306
- R20307: footprint ato_drv:R_0805_2012Metric -> scci_rh_drv:R_0805_2012Metric; symbol ATO_DRV:R307 -> SCCI_RH_DRV:R307
- R20308: footprint ato_drv:R_0805_2012Metric -> scci_rh_drv:R_0805_2012Metric; symbol ATO_DRV:R308 -> SCCI_RH_DRV:R308
- R20309: footprint ato_drv:R_0805_2012Metric -> scci_rh_drv:R_0805_2012Metric; symbol ATO_DRV:R309 -> SCCI_RH_DRV:R309
- R20310: footprint ato_drv:R_0805_2012Metric -> scci_rh_drv:R_0805_2012Metric; symbol ATO_DRV:R310 -> SCCI_RH_DRV:R310
- U20300: footprint ato_drv:TSOT-23-6 -> scci_rh_drv:TSOT-23-6; symbol ATO_DRV:U300 -> SCCI_RH_DRV:U300
- U20301: footprint ato_drv:SOT-23-5 -> scci_rh_drv:SOT-23-5; symbol ATO_DRV:U301 -> SCCI_RH_DRV:U301
- U20302: footprint ato_drv:SOT-23-6 -> scci_rh_drv:SOT-23-6; symbol ATO_DRV:U302 -> SCCI_RH_DRV:U302
- U20303: footprint ato_drv:SOT-23-6 -> scci_rh_drv:SOT-23-6; symbol ATO_DRV:U303 -> SCCI_RH_DRV:U303
- U20304: footprint ato_drv:SOT-23-5 -> scci_rh_drv:SOT-23-5; symbol ATO_DRV:U304 -> SCCI_RH_DRV:U304
- U20305: footprint ato_drv:SOT-23-5 -> scci_rh_drv:SOT-23-5; symbol ATO_DRV:U305 -> SCCI_RH_DRV:U305
- U20306: footprint ato_drv:SOT-23-5 -> scci_rh_drv:SOT-23-5; symbol ATO_DRV:U306 -> SCCI_RH_DRV:U306
- U20307: footprint ato_drv:SOT-23-5 -> scci_rh_drv:SOT-23-5; symbol ATO_DRV:U307 -> SCCI_RH_DRV:U307
- U20308: footprint ato_drv:SOT-23-5 -> scci_rh_drv:SOT-23-5; symbol ATO_DRV:U308 -> SCCI_RH_DRV:U308
- U20309: footprint ato_drv:SOT-23-5 -> scci_rh_drv:SOT-23-5; symbol ATO_DRV:U309 -> SCCI_RH_DRV:U309
- U20310: footprint ato_drv:SOT-23-6 -> scci_rh_drv:SOT-23-6; symbol ATO_DRV:U310 -> SCCI_RH_DRV:U310
- U20311: footprint ato_drv:SOT-23-6 -> scci_rh_drv:SOT-23-6; symbol ATO_DRV:U311 -> SCCI_RH_DRV:U311
- U20312: footprint ato_drv:SOT-23-5 -> scci_rh_drv:SOT-23-5; symbol ATO_DRV:U312 -> SCCI_RH_DRV:U312
- U20313: footprint ato_drv:VSSOP-8_2.3x2mm_P0.5mm -> scci_rh_drv:VSSOP-8_2.3x2mm_P0.5mm; symbol ATO_DRV:U313 -> SCCI_RH_DRV:U313
- U20314: footprint ato_drv:SOT-23-5 -> scci_rh_drv:SOT-23-5; symbol ATO_DRV:U314 -> SCCI_RH_DRV:U314
- U20315: footprint ato_drv:VSSOP-8_2.3x2mm_P0.5mm -> scci_rh_drv:VSSOP-8_2.3x2mm_P0.5mm; symbol ATO_DRV:U315 -> SCCI_RH_DRV:U315
- U20316: footprint ato_drv:VSSOP-8_2.3x2mm_P0.5mm -> scci_rh_drv:VSSOP-8_2.3x2mm_P0.5mm; symbol ATO_DRV:U316 -> SCCI_RH_DRV:U316
- U20317: footprint ato_drv:SOT-23-6 -> scci_rh_drv:SOT-23-6; symbol ATO_DRV:U317 -> SCCI_RH_DRV:U317
- U20318: footprint ato_drv:SOT-23-6 -> scci_rh_drv:SOT-23-6; symbol ATO_DRV:U318 -> SCCI_RH_DRV:U318
- U20319: footprint ato_drv:SOT-23-5 -> scci_rh_drv:SOT-23-5; symbol ATO_DRV:U319 -> SCCI_RH_DRV:U319
- U20320: footprint ato_drv:SOT-23-5 -> scci_rh_drv:SOT-23-5; symbol ATO_DRV:U320 -> SCCI_RH_DRV:U320
Other:
- company: Project ATO -> Project SCCI RH
- title: ATO S4 / Source 0: independent duration and sticky admission -> Project SCCI RH S4 / Source 0: independent duration and sticky admission
