File: electronics/stage4/integrated-pcb/integration/master/current-driver/permission1.kicad_sch (KiCad schematic)
At the start: 53 parts, among them U20400 LTC6993HS6-1#TRPBF, U20401 SN74LVC1G86DBVR, U20402 SN74LVC1G11DBVR, U20403 SN74LVC1G11DBVR, U20404 SN74LVC1G08DBVR, U20405 SN74LVC1G04DBVR, U20406 SN74LVC1G04DBVR, U20407 SN74LVC1G08DBVR, U20408 SN74LVC1G04DBVR, U20409 SN74LVC1G08DBVR, U20410 SN74LVC1G11DBVR, U20411 SN74LVC1G11DBVR, U20412 SN74LVC1G04DBVR, U20413 SN74LVC1G74DCUR, U20414 SN74LVC1G32DBVR, U20415 SN74LVC1G74DCUR, U20416 SN74LVC1G74DCUR, U20417 SN74LVC1G11DBVR, U20418 SN74LVC1G11DBVR, U20419 SN74LVC1G08DBVR, U20420 SN74LVC1G08DBVR

Commit message: Rename project to Project SCCI RH across research and engineering
Parts:
- C20400: footprint ato_drv:C_0805_2012Metric -> scci_rh_drv:C_0805_2012Metric; symbol ATO_DRV:C400 -> SCCI_RH_DRV:C400
- C20401: footprint ato_drv:C_0805_2012Metric -> scci_rh_drv:C_0805_2012Metric; symbol ATO_DRV:C401 -> SCCI_RH_DRV:C401
- C20402: footprint ato_drv:C_0805_2012Metric -> scci_rh_drv:C_0805_2012Metric; symbol ATO_DRV:C402 -> SCCI_RH_DRV:C402
- C20403: footprint ato_drv:C_0805_2012Metric -> scci_rh_drv:C_0805_2012Metric; symbol ATO_DRV:C403 -> SCCI_RH_DRV:C403
- C20404: footprint ato_drv:C_0805_2012Metric -> scci_rh_drv:C_0805_2012Metric; symbol ATO_DRV:C404 -> SCCI_RH_DRV:C404
- C20405: footprint ato_drv:C_0805_2012Metric -> scci_rh_drv:C_0805_2012Metric; symbol ATO_DRV:C405 -> SCCI_RH_DRV:C405
- C20406: footprint ato_drv:C_0805_2012Metric -> scci_rh_drv:C_0805_2012Metric; symbol ATO_DRV:C406 -> SCCI_RH_DRV:C406
- C20407: footprint ato_drv:C_0805_2012Metric -> scci_rh_drv:C_0805_2012Metric; symbol ATO_DRV:C407 -> SCCI_RH_DRV:C407
- C20408: footprint ato_drv:C_0805_2012Metric -> scci_rh_drv:C_0805_2012Metric; symbol ATO_DRV:C408 -> SCCI_RH_DRV:C408
- C20409: footprint ato_drv:C_0805_2012Metric -> scci_rh_drv:C_0805_2012Metric; symbol ATO_DRV:C409 -> SCCI_RH_DRV:C409
- C20410: footprint ato_drv:C_0805_2012Metric -> scci_rh_drv:C_0805_2012Metric; symbol ATO_DRV:C410 -> SCCI_RH_DRV:C410
- C20411: footprint ato_drv:C_0805_2012Metric -> scci_rh_drv:C_0805_2012Metric; symbol ATO_DRV:C411 -> SCCI_RH_DRV:C411
- C20412: footprint ato_drv:C_0805_2012Metric -> scci_rh_drv:C_0805_2012Metric; symbol ATO_DRV:C412 -> SCCI_RH_DRV:C412
- C20413: footprint ato_drv:C_0805_2012Metric -> scci_rh_drv:C_0805_2012Metric; symbol ATO_DRV:C413 -> SCCI_RH_DRV:C413
- C20414: footprint ato_drv:C_0805_2012Metric -> scci_rh_drv:C_0805_2012Metric; symbol ATO_DRV:C414 -> SCCI_RH_DRV:C414
- C20415: footprint ato_drv:C_0805_2012Metric -> scci_rh_drv:C_0805_2012Metric; symbol ATO_DRV:C415 -> SCCI_RH_DRV:C415
- C20416: footprint ato_drv:C_0805_2012Metric -> scci_rh_drv:C_0805_2012Metric; symbol ATO_DRV:C416 -> SCCI_RH_DRV:C416
- C20417: footprint ato_drv:C_0805_2012Metric -> scci_rh_drv:C_0805_2012Metric; symbol ATO_DRV:C417 -> SCCI_RH_DRV:C417
- C20418: footprint ato_drv:C_0805_2012Metric -> scci_rh_drv:C_0805_2012Metric; symbol ATO_DRV:C418 -> SCCI_RH_DRV:C418
- C20419: footprint ato_drv:C_0805_2012Metric -> scci_rh_drv:C_0805_2012Metric; symbol ATO_DRV:C419 -> SCCI_RH_DRV:C419
- C20420: footprint ato_drv:C_0805_2012Metric -> scci_rh_drv:C_0805_2012Metric; symbol ATO_DRV:C420 -> SCCI_RH_DRV:C420
- R20400: footprint ato_drv:R_0805_2012Metric -> scci_rh_drv:R_0805_2012Metric; symbol ATO_DRV:R400 -> SCCI_RH_DRV:R400
- R20401: footprint ato_drv:R_0805_2012Metric -> scci_rh_drv:R_0805_2012Metric; symbol ATO_DRV:R401 -> SCCI_RH_DRV:R401
- R20402: footprint ato_drv:R_0805_2012Metric -> scci_rh_drv:R_0805_2012Metric; symbol ATO_DRV:R402 -> SCCI_RH_DRV:R402
- R20403: footprint ato_drv:R_0805_2012Metric -> scci_rh_drv:R_0805_2012Metric; symbol ATO_DRV:R403 -> SCCI_RH_DRV:R403
- R20404: footprint ato_drv:R_0805_2012Metric -> scci_rh_drv:R_0805_2012Metric; symbol ATO_DRV:R404 -> SCCI_RH_DRV:R404
- R20405: footprint ato_drv:R_0805_2012Metric -> scci_rh_drv:R_0805_2012Metric; symbol ATO_DRV:R405 -> SCCI_RH_DRV:R405
- R20406: footprint ato_drv:R_0805_2012Metric -> scci_rh_drv:R_0805_2012Metric; symbol ATO_DRV:R406 -> SCCI_RH_DRV:R406
- R20407: footprint ato_drv:R_0805_2012Metric -> scci_rh_drv:R_0805_2012Metric; symbol ATO_DRV:R407 -> SCCI_RH_DRV:R407
- R20408: footprint ato_drv:R_0805_2012Metric -> scci_rh_drv:R_0805_2012Metric; symbol ATO_DRV:R408 -> SCCI_RH_DRV:R408
- R20409: footprint ato_drv:R_0805_2012Metric -> scci_rh_drv:R_0805_2012Metric; symbol ATO_DRV:R409 -> SCCI_RH_DRV:R409
- R20410: footprint ato_drv:R_0805_2012Metric -> scci_rh_drv:R_0805_2012Metric; symbol ATO_DRV:R410 -> SCCI_RH_DRV:R410
- U20400: footprint ato_drv:TSOT-23-6 -> scci_rh_drv:TSOT-23-6; symbol ATO_DRV:U400 -> SCCI_RH_DRV:U400
- U20401: footprint ato_drv:SOT-23-5 -> scci_rh_drv:SOT-23-5; symbol ATO_DRV:U401 -> SCCI_RH_DRV:U401
- U20402: footprint ato_drv:SOT-23-6 -> scci_rh_drv:SOT-23-6; symbol ATO_DRV:U402 -> SCCI_RH_DRV:U402
- U20403: footprint ato_drv:SOT-23-6 -> scci_rh_drv:SOT-23-6; symbol ATO_DRV:U403 -> SCCI_RH_DRV:U403
- U20404: footprint ato_drv:SOT-23-5 -> scci_rh_drv:SOT-23-5; symbol ATO_DRV:U404 -> SCCI_RH_DRV:U404
- U20405: footprint ato_drv:SOT-23-5 -> scci_rh_drv:SOT-23-5; symbol ATO_DRV:U405 -> SCCI_RH_DRV:U405
- U20406: footprint ato_drv:SOT-23-5 -> scci_rh_drv:SOT-23-5; symbol ATO_DRV:U406 -> SCCI_RH_DRV:U406
- U20407: footprint ato_drv:SOT-23-5 -> scci_rh_drv:SOT-23-5; symbol ATO_DRV:U407 -> SCCI_RH_DRV:U407
- U20408: footprint ato_drv:SOT-23-5 -> scci_rh_drv:SOT-23-5; symbol ATO_DRV:U408 -> SCCI_RH_DRV:U408
- U20409: footprint ato_drv:SOT-23-5 -> scci_rh_drv:SOT-23-5; symbol ATO_DRV:U409 -> SCCI_RH_DRV:U409
- U20410: footprint ato_drv:SOT-23-6 -> scci_rh_drv:SOT-23-6; symbol ATO_DRV:U410 -> SCCI_RH_DRV:U410
- U20411: footprint ato_drv:SOT-23-6 -> scci_rh_drv:SOT-23-6; symbol ATO_DRV:U411 -> SCCI_RH_DRV:U411
- U20412: footprint ato_drv:SOT-23-5 -> scci_rh_drv:SOT-23-5; symbol ATO_DRV:U412 -> SCCI_RH_DRV:U412
- U20413: footprint ato_drv:VSSOP-8_2.3x2mm_P0.5mm -> scci_rh_drv:VSSOP-8_2.3x2mm_P0.5mm; symbol ATO_DRV:U413 -> SCCI_RH_DRV:U413
- U20414: footprint ato_drv:SOT-23-5 -> scci_rh_drv:SOT-23-5; symbol ATO_DRV:U414 -> SCCI_RH_DRV:U414
- U20415: footprint ato_drv:VSSOP-8_2.3x2mm_P0.5mm -> scci_rh_drv:VSSOP-8_2.3x2mm_P0.5mm; symbol ATO_DRV:U415 -> SCCI_RH_DRV:U415
- U20416: footprint ato_drv:VSSOP-8_2.3x2mm_P0.5mm -> scci_rh_drv:VSSOP-8_2.3x2mm_P0.5mm; symbol ATO_DRV:U416 -> SCCI_RH_DRV:U416
- U20417: footprint ato_drv:SOT-23-6 -> scci_rh_drv:SOT-23-6; symbol ATO_DRV:U417 -> SCCI_RH_DRV:U417
- U20418: footprint ato_drv:SOT-23-6 -> scci_rh_drv:SOT-23-6; symbol ATO_DRV:U418 -> SCCI_RH_DRV:U418
- U20419: footprint ato_drv:SOT-23-5 -> scci_rh_drv:SOT-23-5; symbol ATO_DRV:U419 -> SCCI_RH_DRV:U419
- U20420: footprint ato_drv:SOT-23-5 -> scci_rh_drv:SOT-23-5; symbol ATO_DRV:U420 -> SCCI_RH_DRV:U420
Other:
- company: Project ATO -> Project SCCI RH
- title: ATO S4 / Source 1: independent duration and sticky admission -> Project SCCI RH S4 / Source 1: independent duration and sticky admission
