File: electronics/stage4/integrated-pcb/integration/master/current-driver/source1.kicad_sch (KiCad schematic)
At the start: 18 parts, among them J20200 EXTERNAL ROUTER / MONITOR, Q20200 BSP89H6327XTSA1, U20200 OPA192IDBVR, U20201 TMUX7212PWR, U20202 TMUX6219DGKR, U20203 TMUX6219DGKR

Commit message: Rename project to Project SCCI RH across research and engineering
Parts:
- C20200: footprint ato_drv:C_0805_2012Metric -> scci_rh_drv:C_0805_2012Metric; symbol ATO_DRV:C200 -> SCCI_RH_DRV:C200
- C20201: footprint ato_drv:C_0805_2012Metric -> scci_rh_drv:C_0805_2012Metric; symbol ATO_DRV:C201 -> SCCI_RH_DRV:C201
- C20202: footprint ato_drv:C_0805_2012Metric -> scci_rh_drv:C_0805_2012Metric; symbol ATO_DRV:C202 -> SCCI_RH_DRV:C202
- C20203: footprint ato_drv:C_0805_2012Metric -> scci_rh_drv:C_0805_2012Metric; symbol ATO_DRV:C203 -> SCCI_RH_DRV:C203
- C20204: footprint ato_drv:C_0805_2012Metric -> scci_rh_drv:C_0805_2012Metric; symbol ATO_DRV:C204 -> SCCI_RH_DRV:C204
- C20205: footprint ato_drv:C_0805_2012Metric -> scci_rh_drv:C_0805_2012Metric; symbol ATO_DRV:C205 -> SCCI_RH_DRV:C205
- J20200: footprint ato_drv:PinHeader_1x04_P2.54mm_Vertical -> scci_rh_drv:PinHeader_1x04_P2.54mm_Vertical; symbol ATO_DRV:J200 -> SCCI_RH_DRV:J200
- Q20200: footprint ato_drv:BSP89_PG-SOT223-4_DrainTab -> scci_rh_drv:BSP89_PG-SOT223-4_DrainTab; symbol ATO_DRV:Q200 -> SCCI_RH_DRV:Q200
- R20200: footprint ato_drv:R_0805_2012Metric -> scci_rh_drv:R_0805_2012Metric; symbol ATO_DRV:R200 -> SCCI_RH_DRV:R200
- R20201: footprint ato_drv:R_0805_2012Metric -> scci_rh_drv:R_0805_2012Metric; symbol ATO_DRV:R201 -> SCCI_RH_DRV:R201
- R20202: footprint ato_drv:R_0805_2012Metric -> scci_rh_drv:R_0805_2012Metric; symbol ATO_DRV:R202 -> SCCI_RH_DRV:R202
- R20203: footprint ato_drv:R_0805_2012Metric -> scci_rh_drv:R_0805_2012Metric; symbol ATO_DRV:R203 -> SCCI_RH_DRV:R203
- R20204: footprint ato_drv:R_0805_2012Metric -> scci_rh_drv:R_0805_2012Metric; symbol ATO_DRV:R204 -> SCCI_RH_DRV:R204
- R20205: footprint ato_drv:R_0805_2012Metric -> scci_rh_drv:R_0805_2012Metric; symbol ATO_DRV:R205 -> SCCI_RH_DRV:R205
- U20200: footprint ato_drv:SOT-23-5 -> scci_rh_drv:SOT-23-5; symbol ATO_DRV:U200 -> SCCI_RH_DRV:U200
- U20201: footprint ato_drv:TSSOP-16_4.4x5mm_P0.65mm -> scci_rh_drv:TSSOP-16_4.4x5mm_P0.65mm; symbol ATO_DRV:U201 -> SCCI_RH_DRV:U201
- U20202: footprint ato_drv:VSSOP-8_2.3x2mm_P0.5mm -> scci_rh_drv:VSSOP-8_2.3x2mm_P0.5mm; symbol ATO_DRV:U202 -> SCCI_RH_DRV:U202
- U20203: footprint ato_drv:VSSOP-8_2.3x2mm_P0.5mm -> scci_rh_drv:VSSOP-8_2.3x2mm_P0.5mm; symbol ATO_DRV:U203 -> SCCI_RH_DRV:U203
Other:
- company: Project ATO -> Project SCCI RH
- title: ATO S4 / Source 1: regulated sink and polarity bridge -> Project SCCI RH S4 / Source 1: regulated sink and polarity bridge
