File: electronics/stage4/integrated-pcb/integration/master/monitoring-cell/integration_taps.kicad_sch (KiCad schematic)
At the start: 1 part, among them J19901 HOST TAP HARNESS

Commit message: Rename project to Project SCCI RH across research and engineering
Parts:
- J19901: symbol ATO_INTEGRATION:J19901 -> SCCI_RH_INTEGRATION:J19901
Other:
- company: Project ATO -> Project SCCI RH
- title: ATO / monitoring-cell integration taps -> Project SCCI RH / monitoring-cell integration taps
