File: electronics/stage4/integrated-pcb/integration/master/monitoring-transport/monitoring_transport.kicad_sch (KiCad schematic)
At the start: 3 parts, among them J70001 HOST RAILS / RAW ADC, J70002 EXISTING ANALOG TAPS, J70003 DEDICATED RAW ADC BUS

Commit message: Rename project to Project SCCI RH across research and engineering
Parts:
- J70001: footprint ato_transport:PinHeader_1x03_P2.54mm_Vertical -> scci_rh_transport:PinHeader_1x03_P2.54mm_Vertical; symbol ATO_TRANSPORT:J1 -> SCCI_RH_TRANSPORT:J1
- J70002: footprint ato_transport:PinHeader_1x08_P2.54mm_Vertical -> scci_rh_transport:PinHeader_1x08_P2.54mm_Vertical; symbol ATO_TRANSPORT:J2 -> SCCI_RH_TRANSPORT:J2
- J70003: footprint ato_transport:PinHeader_1x06_P2.54mm_Vertical -> scci_rh_transport:PinHeader_1x06_P2.54mm_Vertical; symbol ATO_TRANSPORT:J3 -> SCCI_RH_TRANSPORT:J3
Other:
- company: Project ATO -> Project SCCI RH
- title: ATO S4 / Existing package and host endpoints -> Project SCCI RH S4 / Existing package and host endpoints
