File: electronics/stage4/integrated-pcb/integration/master/monitoring-transport/reference.kicad_sch (KiCad schematic)
At the start: 9 parts

Commit message: Rename project to Project SCCI RH across research and engineering
Parts:
- C70001: footprint ato_transport:C_1206_3216Metric -> scci_rh_transport:C_1206_3216Metric; symbol ATO_TRANSPORT:C1 -> SCCI_RH_TRANSPORT:C1
- C70002: footprint ato_transport:C_1206_3216Metric -> scci_rh_transport:C_1206_3216Metric; symbol ATO_TRANSPORT:C2 -> SCCI_RH_TRANSPORT:C2
- C70003: footprint ato_transport:C_1206_3216Metric -> scci_rh_transport:C_1206_3216Metric; symbol ATO_TRANSPORT:C3 -> SCCI_RH_TRANSPORT:C3
- C70004: footprint ato_transport:C_1206_3216Metric -> scci_rh_transport:C_1206_3216Metric; symbol ATO_TRANSPORT:C4 -> SCCI_RH_TRANSPORT:C4
- C70005: footprint ato_transport:C_1206_3216Metric -> scci_rh_transport:C_1206_3216Metric; symbol ATO_TRANSPORT:C5 -> SCCI_RH_TRANSPORT:C5
- C70006: footprint ato_transport:C_1206_3216Metric -> scci_rh_transport:C_1206_3216Metric; symbol ATO_TRANSPORT:C6 -> SCCI_RH_TRANSPORT:C6
- C70007: footprint ato_transport:C_1206_3216Metric -> scci_rh_transport:C_1206_3216Metric; symbol ATO_TRANSPORT:C7 -> SCCI_RH_TRANSPORT:C7
- C70008: footprint ato_transport:C_1206_3216Metric -> scci_rh_transport:C_1206_3216Metric; symbol ATO_TRANSPORT:C8 -> SCCI_RH_TRANSPORT:C8
- C70009: footprint ato_transport:C_1206_3216Metric -> scci_rh_transport:C_1206_3216Metric; symbol ATO_TRANSPORT:C9 -> SCCI_RH_TRANSPORT:C9
Other:
- company: Project ATO -> Project SCCI RH
- title: ATO S4 / Independent ADC reference and bypass -> Project SCCI RH S4 / Independent ADC reference and bypass
