File: electronics/stage4/integrated-pcb/integration/master/monitoring-transport/root_2.kicad_sch (KiCad schematic)
At the start: 3 parts, among them J70004 TWO EXISTING CHARGE ADCs, J70005 CHARGE CONTROL HANDOFF, J70006 READ-ONLY NATIVE HEALTH

Commit message: Rename project to Project SCCI RH across research and engineering
Parts:
- J70004: footprint ato_transport:PinHeader_1x08_P2.54mm_Vertical -> scci_rh_transport:PinHeader_1x08_P2.54mm_Vertical; symbol ATO_TRANSPORT:J4 -> SCCI_RH_TRANSPORT:J4
- J70005: footprint ato_transport:PinHeader_1x05_P2.54mm_Vertical -> scci_rh_transport:PinHeader_1x05_P2.54mm_Vertical; symbol ATO_TRANSPORT:J5 -> SCCI_RH_TRANSPORT:J5
- J70006: footprint ato_transport:PinHeader_1x10_P2.54mm_Vertical -> scci_rh_transport:PinHeader_1x10_P2.54mm_Vertical; symbol ATO_TRANSPORT:J6 -> SCCI_RH_TRANSPORT:J6
Other:
- company: Project ATO -> Project SCCI RH
- title: ATO S4 / Existing package and host endpoints / 2 -> Project SCCI RH S4 / Existing package and host endpoints / 2
