File: electronics/stage4/integrated-pcb/integration/master/power/boost15.kicad_sch (KiCad schematic)
At the start: 11 parts, among them U60300 LT8330ES6#TRPBF

Commit message: Rename project to Project SCCI RH across research and engineering
Parts:
- C63000: footprint ato_power:C_1206_3216Metric -> scci_rh_power:C_1206_3216Metric; symbol ATO_POWER:C3000 -> SCCI_RH_POWER:C3000
- C63001: footprint ato_power:C_1206_3216Metric -> scci_rh_power:C_1206_3216Metric; symbol ATO_POWER:C3001 -> SCCI_RH_POWER:C3001
- C63002: footprint ato_power:C_1206_3216Metric -> scci_rh_power:C_1206_3216Metric; symbol ATO_POWER:C3002 -> SCCI_RH_POWER:C3002
- C63003: footprint ato_power:C_1206_3216Metric -> scci_rh_power:C_1206_3216Metric; symbol ATO_POWER:C3003 -> SCCI_RH_POWER:C3003
- C63004: footprint ato_power:C_1206_3216Metric -> scci_rh_power:C_1206_3216Metric; symbol ATO_POWER:C3004 -> SCCI_RH_POWER:C3004
- D60300: footprint ato_power:D_SOD-323F -> scci_rh_power:D_SOD-323F; symbol ATO_POWER:D300 -> SCCI_RH_POWER:D300
- L60300: footprint ato_power:L_Bourns_SRP5030T -> scci_rh_power:L_Bourns_SRP5030T; symbol ATO_POWER:L300 -> SCCI_RH_POWER:L300
- R63000: footprint ato_power:R_0805_2012Metric -> scci_rh_power:R_0805_2012Metric; symbol ATO_POWER:R3000 -> SCCI_RH_POWER:R3000
- R63001: footprint ato_power:R_0805_2012Metric -> scci_rh_power:R_0805_2012Metric; symbol ATO_POWER:R3001 -> SCCI_RH_POWER:R3001
- R63002: footprint ato_power:R_0805_2012Metric -> scci_rh_power:R_0805_2012Metric; symbol ATO_POWER:R3002 -> SCCI_RH_POWER:R3002
- U60300: footprint ato_power:TSOT-23-6 -> scci_rh_power:TSOT-23-6; symbol ATO_POWER:U300 -> SCCI_RH_POWER:U300
Other:
- company: Project ATO -> Project SCCI RH
- title: ATO S4 / Host 15 V boost -> Project SCCI RH S4 / Host 15 V boost
