File: electronics/stage4/integrated-pcb/integration/master/power/boost24.kicad_sch (KiCad schematic)
At the start: 11 parts, among them U60301 LT8330ES6#TRPBF

Commit message: Rename project to Project SCCI RH across research and engineering
Parts:
- C63010: footprint ato_power:C_1206_3216Metric -> scci_rh_power:C_1206_3216Metric; symbol ATO_POWER:C3010 -> SCCI_RH_POWER:C3010
- C63011: footprint ato_power:C_1206_3216Metric -> scci_rh_power:C_1206_3216Metric; symbol ATO_POWER:C3011 -> SCCI_RH_POWER:C3011
- C63012: footprint ato_power:C_1206_3216Metric -> scci_rh_power:C_1206_3216Metric; symbol ATO_POWER:C3012 -> SCCI_RH_POWER:C3012
- C63013: footprint ato_power:C_1206_3216Metric -> scci_rh_power:C_1206_3216Metric; symbol ATO_POWER:C3013 -> SCCI_RH_POWER:C3013
- C63014: footprint ato_power:C_1206_3216Metric -> scci_rh_power:C_1206_3216Metric; symbol ATO_POWER:C3014 -> SCCI_RH_POWER:C3014
- D60301: footprint ato_power:D_SOD-323F -> scci_rh_power:D_SOD-323F; symbol ATO_POWER:D301 -> SCCI_RH_POWER:D301
- L60301: footprint ato_power:L_Bourns_SRP5030T -> scci_rh_power:L_Bourns_SRP5030T; symbol ATO_POWER:L301 -> SCCI_RH_POWER:L301
- R63010: footprint ato_power:R_0805_2012Metric -> scci_rh_power:R_0805_2012Metric; symbol ATO_POWER:R3010 -> SCCI_RH_POWER:R3010
- R63011: footprint ato_power:R_0805_2012Metric -> scci_rh_power:R_0805_2012Metric; symbol ATO_POWER:R3011 -> SCCI_RH_POWER:R3011
- R63012: footprint ato_power:R_0805_2012Metric -> scci_rh_power:R_0805_2012Metric; symbol ATO_POWER:R3012 -> SCCI_RH_POWER:R3012
- U60301: footprint ato_power:TSOT-23-6 -> scci_rh_power:TSOT-23-6; symbol ATO_POWER:U301 -> SCCI_RH_POWER:U301
Other:
- company: Project ATO -> Project SCCI RH
- title: ATO S4 / Stimulation 24 V boost -> Project SCCI RH S4 / Stimulation 24 V boost
