File: electronics/stage4/integrated-pcb/integration/master/power/host5.kicad_sch (KiCad schematic)
At the start: 10 parts, among them U60110 TPS62130ARGTR

Commit message: Rename project to Project SCCI RH across research and engineering
Parts:
- C61100: footprint ato_power:C_1206_3216Metric -> scci_rh_power:C_1206_3216Metric; symbol ATO_POWER:C1100 -> SCCI_RH_POWER:C1100
- C61101: footprint ato_power:C_1206_3216Metric -> scci_rh_power:C_1206_3216Metric; symbol ATO_POWER:C1101 -> SCCI_RH_POWER:C1101
- C61102: footprint ato_power:C_1206_3216Metric -> scci_rh_power:C_1206_3216Metric; symbol ATO_POWER:C1102 -> SCCI_RH_POWER:C1102
- C61103: footprint ato_power:C_1206_3216Metric -> scci_rh_power:C_1206_3216Metric; symbol ATO_POWER:C1103 -> SCCI_RH_POWER:C1103
- L60110: footprint ato_power:L_Bourns_SRP5030T -> scci_rh_power:L_Bourns_SRP5030T; symbol ATO_POWER:L110 -> SCCI_RH_POWER:L110
- R61100: footprint ato_power:R_0805_2012Metric -> scci_rh_power:R_0805_2012Metric; symbol ATO_POWER:R1100 -> SCCI_RH_POWER:R1100
- R61101: footprint ato_power:R_0805_2012Metric -> scci_rh_power:R_0805_2012Metric; symbol ATO_POWER:R1101 -> SCCI_RH_POWER:R1101
- R61102: footprint ato_power:R_0805_2012Metric -> scci_rh_power:R_0805_2012Metric; symbol ATO_POWER:R1102 -> SCCI_RH_POWER:R1102
- R61103: footprint ato_power:R_0805_2012Metric -> scci_rh_power:R_0805_2012Metric; symbol ATO_POWER:R1103 -> SCCI_RH_POWER:R1103
- U60110: footprint ato_power:VQFN-16-1EP_3x3mm_P0.5mm_EP1.68x1.68mm -> scci_rh_power:VQFN-16-1EP_3x3mm_P0.5mm_EP1.68x1.68mm; symbol ATO_POWER:U110 -> SCCI_RH_POWER:U110
Other:
- company: Project ATO -> Project SCCI RH
- title: ATO S4 / Host and module input 5 V -> Project SCCI RH S4 / Host and module input 5 V
