File: electronics/stage4/integrated-pcb/integration/master/power/sup3.kicad_sch (KiCad schematic)
At the start: 8 parts, among them U60100 TPS62160DGKR

Commit message: Rename project to Project SCCI RH across research and engineering
Parts:
- C61000: footprint ato_power:C_1206_3216Metric -> scci_rh_power:C_1206_3216Metric; symbol ATO_POWER:C1000 -> SCCI_RH_POWER:C1000
- C61001: footprint ato_power:C_1206_3216Metric -> scci_rh_power:C_1206_3216Metric; symbol ATO_POWER:C1001 -> SCCI_RH_POWER:C1001
- L60100: footprint ato_power:L_Bourns_SRP5030T -> scci_rh_power:L_Bourns_SRP5030T; symbol ATO_POWER:L100 -> SCCI_RH_POWER:L100
- R61000: footprint ato_power:R_0805_2012Metric -> scci_rh_power:R_0805_2012Metric; symbol ATO_POWER:R1000 -> SCCI_RH_POWER:R1000
- R61001: footprint ato_power:R_0805_2012Metric -> scci_rh_power:R_0805_2012Metric; symbol ATO_POWER:R1001 -> SCCI_RH_POWER:R1001
- R61002: footprint ato_power:R_0805_2012Metric -> scci_rh_power:R_0805_2012Metric; symbol ATO_POWER:R1002 -> SCCI_RH_POWER:R1002
- R61003: footprint ato_power:R_0805_2012Metric -> scci_rh_power:R_0805_2012Metric; symbol ATO_POWER:R1003 -> SCCI_RH_POWER:R1003
- U60100: footprint ato_power:VSSOP-8_3x3mm_P0.65mm -> scci_rh_power:VSSOP-8_3x3mm_P0.65mm; symbol ATO_POWER:U100 -> SCCI_RH_POWER:U100
Other:
- company: Project ATO -> Project SCCI RH
- title: ATO S4 / Always-on supervisor 3.3 V -> Project SCCI RH S4 / Always-on supervisor 3.3 V
