File: electronics/stage4/integrated-pcb/integration/master/recording-front-end/integration_taps.kicad_sch (KiCad schematic)
At the start: 2 parts, among them J39901 AFE TAP HARNESS, J39902 AFE TAP HARNESS

Commit message: Rename project to Project SCCI RH across research and engineering
Parts:
- J39901: symbol ATO_INTEGRATION:J39901 -> SCCI_RH_INTEGRATION:J39901
- J39902: symbol ATO_INTEGRATION:J39902 -> SCCI_RH_INTEGRATION:J39902
Other:
- company: Project ATO -> Project SCCI RH
- title: ATO / recording-front-end integration taps -> Project SCCI RH / recording-front-end integration taps
