File: electronics/stage4/integrated-pcb/integration/master/supervision/afe_rails.kicad_sch (KiCad schematic)
At the start: 16 parts, among them U50206 TPS3700DDCR, U50207 TPS3700DDCR, U50208 TPS3700DDCR

Commit message: Rename project to Project SCCI RH across research and engineering
Parts:
- C50206: footprint ato_sup:C_0805_2012Metric -> scci_rh_sup:C_0805_2012Metric; symbol ATO_SUP:C206 -> SCCI_RH_SUP:C206
- C50207: footprint ato_sup:C_0805_2012Metric -> scci_rh_sup:C_0805_2012Metric; symbol ATO_SUP:C207 -> SCCI_RH_SUP:C207
- R52060: footprint ato_sup:R_0805_2012Metric -> scci_rh_sup:R_0805_2012Metric; symbol ATO_SUP:R2060 -> SCCI_RH_SUP:R2060
- R52061: footprint ato_sup:R_0805_2012Metric -> scci_rh_sup:R_0805_2012Metric; symbol ATO_SUP:R2061 -> SCCI_RH_SUP:R2061
- R52062: footprint ato_sup:R_0805_2012Metric -> scci_rh_sup:R_0805_2012Metric; symbol ATO_SUP:R2062 -> SCCI_RH_SUP:R2062
- R52063: footprint ato_sup:R_0805_2012Metric -> scci_rh_sup:R_0805_2012Metric; symbol ATO_SUP:R2063 -> SCCI_RH_SUP:R2063
- R52064: footprint ato_sup:R_0805_2012Metric -> scci_rh_sup:R_0805_2012Metric; symbol ATO_SUP:R2064 -> SCCI_RH_SUP:R2064
- R52070: footprint ato_sup:R_0805_2012Metric -> scci_rh_sup:R_0805_2012Metric; symbol ATO_SUP:R2070 -> SCCI_RH_SUP:R2070
- R52071: footprint ato_sup:R_0805_2012Metric -> scci_rh_sup:R_0805_2012Metric; symbol ATO_SUP:R2071 -> SCCI_RH_SUP:R2071
- R52072: footprint ato_sup:R_0805_2012Metric -> scci_rh_sup:R_0805_2012Metric; symbol ATO_SUP:R2072 -> SCCI_RH_SUP:R2072
- R52073: footprint ato_sup:R_0805_2012Metric -> scci_rh_sup:R_0805_2012Metric; symbol ATO_SUP:R2073 -> SCCI_RH_SUP:R2073
- R52074: footprint ato_sup:R_0805_2012Metric -> scci_rh_sup:R_0805_2012Metric; symbol ATO_SUP:R2074 -> SCCI_RH_SUP:R2074
- R52080: footprint ato_sup:R_0805_2012Metric -> scci_rh_sup:R_0805_2012Metric; symbol ATO_SUP:R2080 -> SCCI_RH_SUP:R2080
- U50206: footprint ato_sup:SOT-23-6 -> scci_rh_sup:SOT-23-6; symbol ATO_SUP:U206 -> SCCI_RH_SUP:U206
- U50207: footprint ato_sup:SOT-23-6 -> scci_rh_sup:SOT-23-6; symbol ATO_SUP:U207 -> SCCI_RH_SUP:U207
- U50208: footprint ato_sup:SOT-23-6 -> scci_rh_sup:SOT-23-6; symbol ATO_SUP:U208 -> SCCI_RH_SUP:U208
Other:
- company: Project ATO -> Project SCCI RH
- title: ATO S4 / AFE supply windows -> Project SCCI RH S4 / AFE supply windows
