File: electronics/stage4/integrated-pcb/integration/master/supervision/defaults.kicad_sch (KiCad schematic)
At the start: 12 parts

Commit message: Rename project to Project SCCI RH across research and engineering
Parts:
- R50950: footprint ato_sup:R_0805_2012Metric -> scci_rh_sup:R_0805_2012Metric; symbol ATO_SUP:R950 -> SCCI_RH_SUP:R950
- R50951: footprint ato_sup:R_0805_2012Metric -> scci_rh_sup:R_0805_2012Metric; symbol ATO_SUP:R951 -> SCCI_RH_SUP:R951
- R50952: footprint ato_sup:R_0805_2012Metric -> scci_rh_sup:R_0805_2012Metric; symbol ATO_SUP:R952 -> SCCI_RH_SUP:R952
- R50953: footprint ato_sup:R_0805_2012Metric -> scci_rh_sup:R_0805_2012Metric; symbol ATO_SUP:R953 -> SCCI_RH_SUP:R953
- R50954: footprint ato_sup:R_0805_2012Metric -> scci_rh_sup:R_0805_2012Metric; symbol ATO_SUP:R954 -> SCCI_RH_SUP:R954
- R50955: footprint ato_sup:R_0805_2012Metric -> scci_rh_sup:R_0805_2012Metric; symbol ATO_SUP:R955 -> SCCI_RH_SUP:R955
- R50956: footprint ato_sup:R_0805_2012Metric -> scci_rh_sup:R_0805_2012Metric; symbol ATO_SUP:R956 -> SCCI_RH_SUP:R956
- R50957: footprint ato_sup:R_0805_2012Metric -> scci_rh_sup:R_0805_2012Metric; symbol ATO_SUP:R957 -> SCCI_RH_SUP:R957
- R50958: footprint ato_sup:R_0805_2012Metric -> scci_rh_sup:R_0805_2012Metric; symbol ATO_SUP:R958 -> SCCI_RH_SUP:R958
- R50959: footprint ato_sup:R_0805_2012Metric -> scci_rh_sup:R_0805_2012Metric; symbol ATO_SUP:R959 -> SCCI_RH_SUP:R959
- R50960: footprint ato_sup:R_0805_2012Metric -> scci_rh_sup:R_0805_2012Metric; symbol ATO_SUP:R960 -> SCCI_RH_SUP:R960
- R50961: footprint ato_sup:R_0805_2012Metric -> scci_rh_sup:R_0805_2012Metric; symbol ATO_SUP:R961 -> SCCI_RH_SUP:R961
Other:
- company: Project ATO -> Project SCCI RH
- title: ATO S4 / External defaults -> Project SCCI RH S4 / External defaults
