File: electronics/stage4/integrated-pcb/integration/master/supervision/duration.kicad_sch (KiCad schematic)
At the start: 22 parts, among them U50800 LTC6993HS6-1#TRPBF, U50801 LTC6993HS6-1#TRPBF, U50810 SN74LVC1G74DCUR, U50811 SN74LVC1G74DCUR, U51042 SN74LVC1G04DBVR, U51043 SN74LVC1G32DBVR, U51044 SN74LVC1G04DBVR, U51045 SN74LVC1G32DBVR

Commit message: Rename project to Project SCCI RH across research and engineering
Parts:
- C50800: footprint ato_sup:C_0805_2012Metric -> scci_rh_sup:C_0805_2012Metric; symbol ATO_SUP:C800 -> SCCI_RH_SUP:C800
- C50801: footprint ato_sup:C_0805_2012Metric -> scci_rh_sup:C_0805_2012Metric; symbol ATO_SUP:C801 -> SCCI_RH_SUP:C801
- C50810: footprint ato_sup:C_0805_2012Metric -> scci_rh_sup:C_0805_2012Metric; symbol ATO_SUP:C810 -> SCCI_RH_SUP:C810
- C50811: footprint ato_sup:C_0805_2012Metric -> scci_rh_sup:C_0805_2012Metric; symbol ATO_SUP:C811 -> SCCI_RH_SUP:C811
- C51042: footprint ato_sup:C_0805_2012Metric -> scci_rh_sup:C_0805_2012Metric; symbol ATO_SUP:C1042 -> SCCI_RH_SUP:C1042
- C51043: footprint ato_sup:C_0805_2012Metric -> scci_rh_sup:C_0805_2012Metric; symbol ATO_SUP:C1043 -> SCCI_RH_SUP:C1043
- C51044: footprint ato_sup:C_0805_2012Metric -> scci_rh_sup:C_0805_2012Metric; symbol ATO_SUP:C1044 -> SCCI_RH_SUP:C1044
- C51045: footprint ato_sup:C_0805_2012Metric -> scci_rh_sup:C_0805_2012Metric; symbol ATO_SUP:C1045 -> SCCI_RH_SUP:C1045
- R58000: footprint ato_sup:R_0805_2012Metric -> scci_rh_sup:R_0805_2012Metric; symbol ATO_SUP:R8000 -> SCCI_RH_SUP:R8000
- R58001: footprint ato_sup:R_0805_2012Metric -> scci_rh_sup:R_0805_2012Metric; symbol ATO_SUP:R8001 -> SCCI_RH_SUP:R8001
- R58002: footprint ato_sup:R_0805_2012Metric -> scci_rh_sup:R_0805_2012Metric; symbol ATO_SUP:R8002 -> SCCI_RH_SUP:R8002
- R58010: footprint ato_sup:R_0805_2012Metric -> scci_rh_sup:R_0805_2012Metric; symbol ATO_SUP:R8010 -> SCCI_RH_SUP:R8010
- R58011: footprint ato_sup:R_0805_2012Metric -> scci_rh_sup:R_0805_2012Metric; symbol ATO_SUP:R8011 -> SCCI_RH_SUP:R8011
- R58012: footprint ato_sup:R_0805_2012Metric -> scci_rh_sup:R_0805_2012Metric; symbol ATO_SUP:R8012 -> SCCI_RH_SUP:R8012
- U50800: footprint ato_sup:TSOT-23-6 -> scci_rh_sup:TSOT-23-6; symbol ATO_SUP:U800 -> SCCI_RH_SUP:U800
- U50801: footprint ato_sup:TSOT-23-6 -> scci_rh_sup:TSOT-23-6; symbol ATO_SUP:U801 -> SCCI_RH_SUP:U801
- U50810: footprint ato_sup:VSSOP-8_2.3x2mm_P0.5mm -> scci_rh_sup:VSSOP-8_2.3x2mm_P0.5mm; symbol ATO_SUP:U810 -> SCCI_RH_SUP:U810
- U50811: footprint ato_sup:VSSOP-8_2.3x2mm_P0.5mm -> scci_rh_sup:VSSOP-8_2.3x2mm_P0.5mm; symbol ATO_SUP:U811 -> SCCI_RH_SUP:U811
- U51042: footprint ato_sup:SOT-23-5 -> scci_rh_sup:SOT-23-5; symbol ATO_SUP:U1042 -> SCCI_RH_SUP:U1042
- U51043: footprint ato_sup:SOT-23-5 -> scci_rh_sup:SOT-23-5; symbol ATO_SUP:U1043 -> SCCI_RH_SUP:U1043
- U51044: footprint ato_sup:SOT-23-5 -> scci_rh_sup:SOT-23-5; symbol ATO_SUP:U1044 -> SCCI_RH_SUP:U1044
- U51045: footprint ato_sup:SOT-23-5 -> scci_rh_sup:SOT-23-5; symbol ATO_SUP:U1045 -> SCCI_RH_SUP:U1045
Other:
- company: Project ATO -> Project SCCI RH
- title: ATO S4 / Secondary phase duration -> Project SCCI RH S4 / Secondary phase duration
