File: electronics/stage4/integrated-pcb/integration/master/supervision/guards.kicad_sch (KiCad schematic)
At the start: 18 parts, among them J50100 CANONICAL ROUTER J7 / BEFORE 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, J50101 BODY-FACING ARTIFICIAL LOAD C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, U50100 TMUX7412FRRPR, U50101 TMUX7412FRRPR, U50102 TMUX7412FRRPR, U50103 TMUX7412FRRPR, U50104 TMUX7412FRRPR

Commit message: Rename project to Project SCCI RH across research and engineering
Parts:
- C50100: footprint ato_sup:C_0805_2012Metric -> scci_rh_sup:C_0805_2012Metric; symbol ATO_SUP:C100 -> SCCI_RH_SUP:C100
- C50101: footprint ato_sup:C_0805_2012Metric -> scci_rh_sup:C_0805_2012Metric; symbol ATO_SUP:C101 -> SCCI_RH_SUP:C101
- C50102: footprint ato_sup:C_0805_2012Metric -> scci_rh_sup:C_0805_2012Metric; symbol ATO_SUP:C102 -> SCCI_RH_SUP:C102
- C50103: footprint ato_sup:C_0805_2012Metric -> scci_rh_sup:C_0805_2012Metric; symbol ATO_SUP:C103 -> SCCI_RH_SUP:C103
- C50104: footprint ato_sup:C_0805_2012Metric -> scci_rh_sup:C_0805_2012Metric; symbol ATO_SUP:C104 -> SCCI_RH_SUP:C104
- J50100: footprint ato_sup:PinHeader_1x18_P2.54mm_Vertical -> scci_rh_sup:PinHeader_1x18_P2.54mm_Vertical; symbol ATO_SUP:J100 -> SCCI_RH_SUP:J100
- J50101: footprint ato_sup:PinHeader_1x18_P2.54mm_Vertical -> scci_rh_sup:PinHeader_1x18_P2.54mm_Vertical; symbol ATO_SUP:J101 -> SCCI_RH_SUP:J101
- R50100: footprint ato_sup:R_0805_2012Metric -> scci_rh_sup:R_0805_2012Metric; symbol ATO_SUP:R100 -> SCCI_RH_SUP:R100
- R50101: footprint ato_sup:R_0805_2012Metric -> scci_rh_sup:R_0805_2012Metric; symbol ATO_SUP:R101 -> SCCI_RH_SUP:R101
- R50102: footprint ato_sup:R_0805_2012Metric -> scci_rh_sup:R_0805_2012Metric; symbol ATO_SUP:R102 -> SCCI_RH_SUP:R102
- R50103: footprint ato_sup:R_0805_2012Metric -> scci_rh_sup:R_0805_2012Metric; symbol ATO_SUP:R103 -> SCCI_RH_SUP:R103
- R50104: footprint ato_sup:R_0805_2012Metric -> scci_rh_sup:R_0805_2012Metric; symbol ATO_SUP:R104 -> SCCI_RH_SUP:R104
- R50110: footprint ato_sup:R_0805_2012Metric -> scci_rh_sup:R_0805_2012Metric; symbol ATO_SUP:R110 -> SCCI_RH_SUP:R110
- U50100: footprint ato_sup:Texas_RRP0016A_WQFN16_4x4_P0.65_EP2.6 -> scci_rh_sup:Texas_RRP0016A_WQFN16_4x4_P0.65_EP2.6; symbol ATO_SUP:U100 -> SCCI_RH_SUP:U100
- U50101: footprint ato_sup:Texas_RRP0016A_WQFN16_4x4_P0.65_EP2.6 -> scci_rh_sup:Texas_RRP0016A_WQFN16_4x4_P0.65_EP2.6; symbol ATO_SUP:U101 -> SCCI_RH_SUP:U101
- U50102: footprint ato_sup:Texas_RRP0016A_WQFN16_4x4_P0.65_EP2.6 -> scci_rh_sup:Texas_RRP0016A_WQFN16_4x4_P0.65_EP2.6; symbol ATO_SUP:U102 -> SCCI_RH_SUP:U102
- U50103: footprint ato_sup:Texas_RRP0016A_WQFN16_4x4_P0.65_EP2.6 -> scci_rh_sup:Texas_RRP0016A_WQFN16_4x4_P0.65_EP2.6; symbol ATO_SUP:U103 -> SCCI_RH_SUP:U103
- U50104: footprint ato_sup:Texas_RRP0016A_WQFN16_4x4_P0.65_EP2.6 -> scci_rh_sup:Texas_RRP0016A_WQFN16_4x4_P0.65_EP2.6; symbol ATO_SUP:U104 -> SCCI_RH_SUP:U104
Other:
- company: Project ATO -> Project SCCI RH
- title: ATO S4 / 18 body-side terminal guards -> Project SCCI RH S4 / 18 body-side terminal guards
