File: electronics/stage4/integrated-pcb/integration/master/supervision/integration_taps.kicad_sch (KiCad schematic)
At the start: 1 part, among them J59901 HOST TAP HARNESS

Commit message: Rename project to Project SCCI RH across research and engineering
Parts:
- J59901: symbol ATO_INTEGRATION:J59901 -> SCCI_RH_INTEGRATION:J59901
Other:
- company: Project ATO -> Project SCCI RH
- title: ATO / supervision integration taps -> Project SCCI RH / supervision integration taps
