File: electronics/stage4/integrated-pcb/integration/master/supervision/watchdog.kicad_sch (KiCad schematic)
At the start: 27 parts, among them U50250 SN74LVC1G17DBVR, U50300 TPS3431SDRBR, U50301 SN74LVC1G74DCUR, U51000 SN74LVC1G11DBVR, U51001 SN74LVC1G11DBVR, U51002 SN74LVC1G11DBVR, U51005 SN74LVC1G04DBVR, U51006 SN74LVC1G08DBVR, U51007 SN74LVC1G11DBVR, U51008 SN74LVC1G08DBVR

Commit message: Rename project to Project SCCI RH across research and engineering
Parts:
- C50250: footprint ato_sup:C_0805_2012Metric -> scci_rh_sup:C_0805_2012Metric; symbol ATO_SUP:C250 -> SCCI_RH_SUP:C250
- C50251: footprint ato_sup:C_0805_2012Metric -> scci_rh_sup:C_0805_2012Metric; symbol ATO_SUP:C251 -> SCCI_RH_SUP:C251
- C50300: footprint ato_sup:C_0805_2012Metric -> scci_rh_sup:C_0805_2012Metric; symbol ATO_SUP:C300 -> SCCI_RH_SUP:C300
- C50301: footprint ato_sup:C_0805_2012Metric -> scci_rh_sup:C_0805_2012Metric; symbol ATO_SUP:C301 -> SCCI_RH_SUP:C301
- C51000: footprint ato_sup:C_0805_2012Metric -> scci_rh_sup:C_0805_2012Metric; symbol ATO_SUP:C1000 -> SCCI_RH_SUP:C1000
- C51001: footprint ato_sup:C_0805_2012Metric -> scci_rh_sup:C_0805_2012Metric; symbol ATO_SUP:C1001 -> SCCI_RH_SUP:C1001
- C51002: footprint ato_sup:C_0805_2012Metric -> scci_rh_sup:C_0805_2012Metric; symbol ATO_SUP:C1002 -> SCCI_RH_SUP:C1002
- C51005: footprint ato_sup:C_0805_2012Metric -> scci_rh_sup:C_0805_2012Metric; symbol ATO_SUP:C1005 -> SCCI_RH_SUP:C1005
- C51006: footprint ato_sup:C_0805_2012Metric -> scci_rh_sup:C_0805_2012Metric; symbol ATO_SUP:C1006 -> SCCI_RH_SUP:C1006
- C51007: footprint ato_sup:C_0805_2012Metric -> scci_rh_sup:C_0805_2012Metric; symbol ATO_SUP:C1007 -> SCCI_RH_SUP:C1007
- C51008: footprint ato_sup:C_0805_2012Metric -> scci_rh_sup:C_0805_2012Metric; symbol ATO_SUP:C1008 -> SCCI_RH_SUP:C1008
- D50250: footprint ato_sup:D_SOD-323 -> scci_rh_sup:D_SOD-323; symbol ATO_SUP:D250 -> SCCI_RH_SUP:D250
- R50250: footprint ato_sup:R_0805_2012Metric -> scci_rh_sup:R_0805_2012Metric; symbol ATO_SUP:R250 -> SCCI_RH_SUP:R250
- R50251: footprint ato_sup:R_0805_2012Metric -> scci_rh_sup:R_0805_2012Metric; symbol ATO_SUP:R251 -> SCCI_RH_SUP:R251
- R50300: footprint ato_sup:R_0805_2012Metric -> scci_rh_sup:R_0805_2012Metric; symbol ATO_SUP:R300 -> SCCI_RH_SUP:R300
- R50301: footprint ato_sup:R_0805_2012Metric -> scci_rh_sup:R_0805_2012Metric; symbol ATO_SUP:R301 -> SCCI_RH_SUP:R301
- R50302: footprint ato_sup:R_0805_2012Metric -> scci_rh_sup:R_0805_2012Metric; symbol ATO_SUP:R302 -> SCCI_RH_SUP:R302
- U50250: footprint ato_sup:SOT-23-5 -> scci_rh_sup:SOT-23-5; symbol ATO_SUP:U250 -> SCCI_RH_SUP:U250
- U50300: footprint ato_sup:Texas_DRB0008A_VSON8_3x3_P0.65_EP1.5x1.75 -> scci_rh_sup:Texas_DRB0008A_VSON8_3x3_P0.65_EP1.5x1.75; symbol ATO_SUP:U300 -> SCCI_RH_SUP:U300
- U50301: footprint ato_sup:VSSOP-8_2.3x2mm_P0.5mm -> scci_rh_sup:VSSOP-8_2.3x2mm_P0.5mm; symbol ATO_SUP:U301 -> SCCI_RH_SUP:U301
- U51000: footprint ato_sup:SOT-23-6 -> scci_rh_sup:SOT-23-6; symbol ATO_SUP:U1000 -> SCCI_RH_SUP:U1000
- U51001: footprint ato_sup:SOT-23-6 -> scci_rh_sup:SOT-23-6; symbol ATO_SUP:U1001 -> SCCI_RH_SUP:U1001
- U51002: footprint ato_sup:SOT-23-6 -> scci_rh_sup:SOT-23-6; symbol ATO_SUP:U1002 -> SCCI_RH_SUP:U1002
- U51005: footprint ato_sup:SOT-23-5 -> scci_rh_sup:SOT-23-5; symbol ATO_SUP:U1005 -> SCCI_RH_SUP:U1005
- U51006: footprint ato_sup:SOT-23-5 -> scci_rh_sup:SOT-23-5; symbol ATO_SUP:U1006 -> SCCI_RH_SUP:U1006
- U51007: footprint ato_sup:SOT-23-6 -> scci_rh_sup:SOT-23-6; symbol ATO_SUP:U1007 -> SCCI_RH_SUP:U1007
- U51008: footprint ato_sup:SOT-23-5 -> scci_rh_sup:SOT-23-5; symbol ATO_SUP:U1008 -> SCCI_RH_SUP:U1008
Other:
- company: Project ATO -> Project SCCI RH
- title: ATO S4 / Heartbeat and startup -> Project SCCI RH S4 / Heartbeat and startup
