File: electronics/stage4/monitoring-transport/companion.kicad_sch (KiCad schematic)
At the start: 13 parts, among them J7 HOST PROCESSED UART, J8 EXTERNAL COMPANION UART, U20 ISO6721BDR

Commit message: Rename project to Project SCCI RH across research and engineering
Parts:
- C20: footprint ato_transport:C_1206_3216Metric -> scci_rh_transport:C_1206_3216Metric; symbol ATO_TRANSPORT:C20 -> SCCI_RH_TRANSPORT:C20
- C21: footprint ato_transport:C_1206_3216Metric -> scci_rh_transport:C_1206_3216Metric; symbol ATO_TRANSPORT:C21 -> SCCI_RH_TRANSPORT:C21
- C22: footprint ato_transport:C_1206_3216Metric -> scci_rh_transport:C_1206_3216Metric; symbol ATO_TRANSPORT:C22 -> SCCI_RH_TRANSPORT:C22
- C23: footprint ato_transport:C_1206_3216Metric -> scci_rh_transport:C_1206_3216Metric; symbol ATO_TRANSPORT:C23 -> SCCI_RH_TRANSPORT:C23
- J7: footprint ato_transport:PinHeader_1x04_P2.54mm_Vertical -> scci_rh_transport:PinHeader_1x04_P2.54mm_Vertical; symbol ATO_TRANSPORT:J7 -> SCCI_RH_TRANSPORT:J7
- J8: footprint ato_transport:PinHeader_1x04_P2.54mm_Vertical -> scci_rh_transport:PinHeader_1x04_P2.54mm_Vertical; symbol ATO_TRANSPORT:J8 -> SCCI_RH_TRANSPORT:J8
- R20: footprint ato_transport:R_0805_2012Metric -> scci_rh_transport:R_0805_2012Metric; symbol ATO_TRANSPORT:R20 -> SCCI_RH_TRANSPORT:R20
- R21: footprint ato_transport:R_0805_2012Metric -> scci_rh_transport:R_0805_2012Metric; symbol ATO_TRANSPORT:R21 -> SCCI_RH_TRANSPORT:R21
- R22: footprint ato_transport:R_0805_2012Metric -> scci_rh_transport:R_0805_2012Metric; symbol ATO_TRANSPORT:R22 -> SCCI_RH_TRANSPORT:R22
- R23: footprint ato_transport:R_0805_2012Metric -> scci_rh_transport:R_0805_2012Metric; symbol ATO_TRANSPORT:R23 -> SCCI_RH_TRANSPORT:R23
- R24: footprint ato_transport:R_0805_2012Metric -> scci_rh_transport:R_0805_2012Metric; symbol ATO_TRANSPORT:R24 -> SCCI_RH_TRANSPORT:R24
- R25: footprint ato_transport:R_0805_2012Metric -> scci_rh_transport:R_0805_2012Metric; symbol ATO_TRANSPORT:R25 -> SCCI_RH_TRANSPORT:R25
- U20: footprint ato_transport:SOIC-8_3.9x4.9mm_P1.27mm -> scci_rh_transport:SOIC-8_3.9x4.9mm_P1.27mm; symbol ATO_TRANSPORT:U20 -> SCCI_RH_TRANSPORT:U20
Other:
- company: Project ATO -> Project SCCI RH
- title: ATO S4 / Isolated wired processed-feature companion -> Project SCCI RH S4 / Isolated wired processed-feature companion
