File: electronics/stage4/power/afe3.kicad_sch (KiCad schematic)
At the start: 9 parts, among them J410 QUIESCENT TRIM / TEST ONLY, U410 TPS7A4901DGNR

Commit message: Rename project to Project SCCI RH across research and engineering
Parts:
- C4100: footprint ato_power:C_1206_3216Metric -> scci_rh_power:C_1206_3216Metric; symbol ATO_POWER:C4100 -> SCCI_RH_POWER:C4100
- C4101: footprint ato_power:C_1206_3216Metric -> scci_rh_power:C_1206_3216Metric; symbol ATO_POWER:C4101 -> SCCI_RH_POWER:C4101
- C4102: footprint ato_power:C_1206_3216Metric -> scci_rh_power:C_1206_3216Metric; symbol ATO_POWER:C4102 -> SCCI_RH_POWER:C4102
- C4103: footprint ato_power:C_1206_3216Metric -> scci_rh_power:C_1206_3216Metric; symbol ATO_POWER:C4103 -> SCCI_RH_POWER:C4103
- J410: footprint ato_power:PinHeader_1x03_P2.54mm_Vertical -> scci_rh_power:PinHeader_1x03_P2.54mm_Vertical; symbol ATO_POWER:J410 -> SCCI_RH_POWER:J410
- R4100: footprint ato_power:R_0805_2012Metric -> scci_rh_power:R_0805_2012Metric; symbol ATO_POWER:R4100 -> SCCI_RH_POWER:R4100
- R4101: footprint ato_power:R_0805_2012Metric -> scci_rh_power:R_0805_2012Metric; symbol ATO_POWER:R4101 -> SCCI_RH_POWER:R4101
- R4102: footprint ato_power:R_0805_2012Metric -> scci_rh_power:R_0805_2012Metric; symbol ATO_POWER:R4102 -> SCCI_RH_POWER:R4102
- U410: footprint ato_power:Texas_DGN0008D_VSSOP-8-1EP_3x3mm_P0.65mm_EP2x2.94mm_Mask1.57x1.89mm -> scci_rh_power:Texas_DGN0008D_VSSOP-8-1EP_3x3mm_P0.65mm_EP2x2.94mm_Mask1.57x1.89mm; symbol ATO_POWER:U410 -> SCCI_RH_POWER:U410
Other:
- company: Project ATO -> Project SCCI RH
- title: ATO S4 / Floating AFE 3.45 V regulator -> Project SCCI RH S4 / Floating AFE 3.45 V regulator
