File: electronics/stage4/power/afep.kicad_sch (KiCad schematic)
At the start: 9 parts, among them J411 QUIESCENT TRIM / TEST ONLY, U411 TPS7A4901DGNR

Commit message: Rename project to Project SCCI RH across research and engineering
Parts:
- C4110: footprint ato_power:C_1206_3216Metric -> scci_rh_power:C_1206_3216Metric; symbol ATO_POWER:C4110 -> SCCI_RH_POWER:C4110
- C4111: footprint ato_power:C_1206_3216Metric -> scci_rh_power:C_1206_3216Metric; symbol ATO_POWER:C4111 -> SCCI_RH_POWER:C4111
- C4112: footprint ato_power:C_1206_3216Metric -> scci_rh_power:C_1206_3216Metric; symbol ATO_POWER:C4112 -> SCCI_RH_POWER:C4112
- C4113: footprint ato_power:C_1206_3216Metric -> scci_rh_power:C_1206_3216Metric; symbol ATO_POWER:C4113 -> SCCI_RH_POWER:C4113
- J411: footprint ato_power:PinHeader_1x03_P2.54mm_Vertical -> scci_rh_power:PinHeader_1x03_P2.54mm_Vertical; symbol ATO_POWER:J411 -> SCCI_RH_POWER:J411
- R4110: footprint ato_power:R_0805_2012Metric -> scci_rh_power:R_0805_2012Metric; symbol ATO_POWER:R4110 -> SCCI_RH_POWER:R4110
- R4111: footprint ato_power:R_0805_2012Metric -> scci_rh_power:R_0805_2012Metric; symbol ATO_POWER:R4111 -> SCCI_RH_POWER:R4111
- R4112: footprint ato_power:R_0805_2012Metric -> scci_rh_power:R_0805_2012Metric; symbol ATO_POWER:R4112 -> SCCI_RH_POWER:R4112
- U411: footprint ato_power:Texas_DGN0008D_VSSOP-8-1EP_3x3mm_P0.65mm_EP2x2.94mm_Mask1.57x1.89mm -> scci_rh_power:Texas_DGN0008D_VSSOP-8-1EP_3x3mm_P0.65mm_EP2x2.94mm_Mask1.57x1.89mm; symbol ATO_POWER:U411 -> SCCI_RH_POWER:U411
Other:
- company: Project ATO -> Project SCCI RH
- title: ATO S4 / Floating AFE +5.30 V regulator -> Project SCCI RH S4 / Floating AFE +5.30 V regulator
