File: electronics/stage4/power/host5.kicad_sch (KiCad schematic)
At the start: 10 parts, among them U110 TPS62130ARGTR

Commit message: Rename project to Project SCCI RH across research and engineering
Parts:
- C1100: footprint ato_power:C_1206_3216Metric -> scci_rh_power:C_1206_3216Metric; symbol ATO_POWER:C1100 -> SCCI_RH_POWER:C1100
- C1101: footprint ato_power:C_1206_3216Metric -> scci_rh_power:C_1206_3216Metric; symbol ATO_POWER:C1101 -> SCCI_RH_POWER:C1101
- C1102: footprint ato_power:C_1206_3216Metric -> scci_rh_power:C_1206_3216Metric; symbol ATO_POWER:C1102 -> SCCI_RH_POWER:C1102
- C1103: footprint ato_power:C_1206_3216Metric -> scci_rh_power:C_1206_3216Metric; symbol ATO_POWER:C1103 -> SCCI_RH_POWER:C1103
- L110: footprint ato_power:L_Bourns_SRP5030T -> scci_rh_power:L_Bourns_SRP5030T; symbol ATO_POWER:L110 -> SCCI_RH_POWER:L110
- R1100: footprint ato_power:R_0805_2012Metric -> scci_rh_power:R_0805_2012Metric; symbol ATO_POWER:R1100 -> SCCI_RH_POWER:R1100
- R1101: footprint ato_power:R_0805_2012Metric -> scci_rh_power:R_0805_2012Metric; symbol ATO_POWER:R1101 -> SCCI_RH_POWER:R1101
- R1102: footprint ato_power:R_0805_2012Metric -> scci_rh_power:R_0805_2012Metric; symbol ATO_POWER:R1102 -> SCCI_RH_POWER:R1102
- R1103: footprint ato_power:R_0805_2012Metric -> scci_rh_power:R_0805_2012Metric; symbol ATO_POWER:R1103 -> SCCI_RH_POWER:R1103
- U110: footprint ato_power:VQFN-16-1EP_3x3mm_P0.5mm_EP1.68x1.68mm -> scci_rh_power:VQFN-16-1EP_3x3mm_P0.5mm_EP1.68x1.68mm; symbol ATO_POWER:U110 -> SCCI_RH_POWER:U110
Other:
- company: Project ATO -> Project SCCI RH
- title: ATO S4 / Host and module input 5 V -> Project SCCI RH S4 / Host and module input 5 V
