File: electronics/stage4/power/power.kicad_sch (KiCad schematic)
At the start: 6 parts, among them J1 AT31004 PROTECTED 2S PACK / 6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, J2 POWER REQUEST / STATUS, J3 HOST AND SUPERVISOR RAILS, J4 FLOATING RECORDING RAILS, J5 CONVERTER TEST POINTS, J6 EXISTING MONITOR REFERENCES

Commit message: Rename project to Project SCCI RH across research and engineering
Parts:
- J1: footprint ato_power:PinHeader_1x02_P2.54mm_Vertical -> scci_rh_power:PinHeader_1x02_P2.54mm_Vertical; symbol ATO_POWER:J1 -> SCCI_RH_POWER:J1
- J2: footprint ato_power:PinHeader_1x12_P2.54mm_Vertical -> scci_rh_power:PinHeader_1x12_P2.54mm_Vertical; symbol ATO_POWER:J2 -> SCCI_RH_POWER:J2
- J3: footprint ato_power:PinHeader_1x07_P2.54mm_Vertical -> scci_rh_power:PinHeader_1x07_P2.54mm_Vertical; symbol ATO_POWER:J3 -> SCCI_RH_POWER:J3
- J4: footprint ato_power:PinHeader_1x04_P2.54mm_Vertical -> scci_rh_power:PinHeader_1x04_P2.54mm_Vertical; symbol ATO_POWER:J4 -> SCCI_RH_POWER:J4
- J5: footprint ato_power:PinHeader_1x05_P2.54mm_Vertical -> scci_rh_power:PinHeader_1x05_P2.54mm_Vertical; symbol ATO_POWER:J5 -> SCCI_RH_POWER:J5
- J6: footprint ato_power:PinHeader_1x03_P2.54mm_Vertical -> scci_rh_power:PinHeader_1x03_P2.54mm_Vertical; symbol ATO_POWER:J6 -> SCCI_RH_POWER:J6
Other:
- company: Project ATO -> Project SCCI RH
- title: ATO S4 / Interfaces and rail handoff -> Project SCCI RH S4 / Interfaces and rail handoff
