File: electronics/stage4/supervision/afe_bank0.kicad_sch (KiCad schematic)
At the start: 28 parts, among them J600 REC00 ACTUAL RHD-SIDE TAP, J601 REC01 ACTUAL RHD-SIDE TAP, J602 REC02 ACTUAL RHD-SIDE TAP, J603 REC03 ACTUAL RHD-SIDE TAP, U1013 SN74LVC1G08DBVR, U1014 SN74LVC1G08DBVR, U1015 SN74LVC1G08DBVR, U1016 SN74LVC1G08DBVR, U600 TLV3202DGKR, U601 TLV3202DGKR, U602 TLV3202DGKR, U603 TLV3202DGKR

Commit message: Rename project to Project SCCI RH across research and engineering
Parts:
- C1013: footprint ato_sup:C_0805_2012Metric -> scci_rh_sup:C_0805_2012Metric; symbol ATO_SUP:C1013 -> SCCI_RH_SUP:C1013
- C1014: footprint ato_sup:C_0805_2012Metric -> scci_rh_sup:C_0805_2012Metric; symbol ATO_SUP:C1014 -> SCCI_RH_SUP:C1014
- C1015: footprint ato_sup:C_0805_2012Metric -> scci_rh_sup:C_0805_2012Metric; symbol ATO_SUP:C1015 -> SCCI_RH_SUP:C1015
- C1016: footprint ato_sup:C_0805_2012Metric -> scci_rh_sup:C_0805_2012Metric; symbol ATO_SUP:C1016 -> SCCI_RH_SUP:C1016
- C600: footprint ato_sup:C_0805_2012Metric -> scci_rh_sup:C_0805_2012Metric; symbol ATO_SUP:C600 -> SCCI_RH_SUP:C600
- C601: footprint ato_sup:C_0805_2012Metric -> scci_rh_sup:C_0805_2012Metric; symbol ATO_SUP:C601 -> SCCI_RH_SUP:C601
- C602: footprint ato_sup:C_0805_2012Metric -> scci_rh_sup:C_0805_2012Metric; symbol ATO_SUP:C602 -> SCCI_RH_SUP:C602
- C603: footprint ato_sup:C_0805_2012Metric -> scci_rh_sup:C_0805_2012Metric; symbol ATO_SUP:C603 -> SCCI_RH_SUP:C603
- J600: footprint ato_sup:PinHeader_1x02_P2.54mm_Vertical -> scci_rh_sup:PinHeader_1x02_P2.54mm_Vertical; symbol ATO_SUP:J600 -> SCCI_RH_SUP:J600
- J601: footprint ato_sup:PinHeader_1x02_P2.54mm_Vertical -> scci_rh_sup:PinHeader_1x02_P2.54mm_Vertical; symbol ATO_SUP:J601 -> SCCI_RH_SUP:J601
- J602: footprint ato_sup:PinHeader_1x02_P2.54mm_Vertical -> scci_rh_sup:PinHeader_1x02_P2.54mm_Vertical; symbol ATO_SUP:J602 -> SCCI_RH_SUP:J602
- J603: footprint ato_sup:PinHeader_1x02_P2.54mm_Vertical -> scci_rh_sup:PinHeader_1x02_P2.54mm_Vertical; symbol ATO_SUP:J603 -> SCCI_RH_SUP:J603
- R6000: footprint ato_sup:R_0805_2012Metric -> scci_rh_sup:R_0805_2012Metric; symbol ATO_SUP:R6000 -> SCCI_RH_SUP:R6000
- R6001: footprint ato_sup:R_0805_2012Metric -> scci_rh_sup:R_0805_2012Metric; symbol ATO_SUP:R6001 -> SCCI_RH_SUP:R6001
- R6010: footprint ato_sup:R_0805_2012Metric -> scci_rh_sup:R_0805_2012Metric; symbol ATO_SUP:R6010 -> SCCI_RH_SUP:R6010
- R6011: footprint ato_sup:R_0805_2012Metric -> scci_rh_sup:R_0805_2012Metric; symbol ATO_SUP:R6011 -> SCCI_RH_SUP:R6011
- R6020: footprint ato_sup:R_0805_2012Metric -> scci_rh_sup:R_0805_2012Metric; symbol ATO_SUP:R6020 -> SCCI_RH_SUP:R6020
- R6021: footprint ato_sup:R_0805_2012Metric -> scci_rh_sup:R_0805_2012Metric; symbol ATO_SUP:R6021 -> SCCI_RH_SUP:R6021
- R6030: footprint ato_sup:R_0805_2012Metric -> scci_rh_sup:R_0805_2012Metric; symbol ATO_SUP:R6030 -> SCCI_RH_SUP:R6030
- R6031: footprint ato_sup:R_0805_2012Metric -> scci_rh_sup:R_0805_2012Metric; symbol ATO_SUP:R6031 -> SCCI_RH_SUP:R6031
- U1013: footprint ato_sup:SOT-23-5 -> scci_rh_sup:SOT-23-5; symbol ATO_SUP:U1013 -> SCCI_RH_SUP:U1013
- U1014: footprint ato_sup:SOT-23-5 -> scci_rh_sup:SOT-23-5; symbol ATO_SUP:U1014 -> SCCI_RH_SUP:U1014
- U1015: footprint ato_sup:SOT-23-5 -> scci_rh_sup:SOT-23-5; symbol ATO_SUP:U1015 -> SCCI_RH_SUP:U1015
- U1016: footprint ato_sup:SOT-23-5 -> scci_rh_sup:SOT-23-5; symbol ATO_SUP:U1016 -> SCCI_RH_SUP:U1016
- U600: footprint ato_sup:VSSOP-8_2.3x2mm_P0.5mm -> scci_rh_sup:VSSOP-8_2.3x2mm_P0.5mm; symbol ATO_SUP:U600 -> SCCI_RH_SUP:U600
- U601: footprint ato_sup:VSSOP-8_2.3x2mm_P0.5mm -> scci_rh_sup:VSSOP-8_2.3x2mm_P0.5mm; symbol ATO_SUP:U601 -> SCCI_RH_SUP:U601
- U602: footprint ato_sup:VSSOP-8_2.3x2mm_P0.5mm -> scci_rh_sup:VSSOP-8_2.3x2mm_P0.5mm; symbol ATO_SUP:U602 -> SCCI_RH_SUP:U602
- U603: footprint ato_sup:VSSOP-8_2.3x2mm_P0.5mm -> scci_rh_sup:VSSOP-8_2.3x2mm_P0.5mm; symbol ATO_SUP:U603 -> SCCI_RH_SUP:U603
Other:
- company: Project ATO -> Project SCCI RH
- title: ATO S4 / RHD input windows 0 -> Project SCCI RH S4 / RHD input windows 0
