File: electronics/stage4/supervision/afe_bank1.kicad_sch (KiCad schematic)
At the start: 28 parts, among them J604 REC04 ACTUAL RHD-SIDE TAP, J605 REC05 ACTUAL RHD-SIDE TAP, J606 REC06 ACTUAL RHD-SIDE TAP, J607 REC07 ACTUAL RHD-SIDE TAP, U1017 SN74LVC1G08DBVR, U1018 SN74LVC1G08DBVR, U1019 SN74LVC1G08DBVR, U1020 SN74LVC1G08DBVR, U604 TLV3202DGKR, U605 TLV3202DGKR, U606 TLV3202DGKR, U607 TLV3202DGKR

Commit message: Rename project to Project SCCI RH across research and engineering
Parts:
- C1017: footprint ato_sup:C_0805_2012Metric -> scci_rh_sup:C_0805_2012Metric; symbol ATO_SUP:C1017 -> SCCI_RH_SUP:C1017
- C1018: footprint ato_sup:C_0805_2012Metric -> scci_rh_sup:C_0805_2012Metric; symbol ATO_SUP:C1018 -> SCCI_RH_SUP:C1018
- C1019: footprint ato_sup:C_0805_2012Metric -> scci_rh_sup:C_0805_2012Metric; symbol ATO_SUP:C1019 -> SCCI_RH_SUP:C1019
- C1020: footprint ato_sup:C_0805_2012Metric -> scci_rh_sup:C_0805_2012Metric; symbol ATO_SUP:C1020 -> SCCI_RH_SUP:C1020
- C604: footprint ato_sup:C_0805_2012Metric -> scci_rh_sup:C_0805_2012Metric; symbol ATO_SUP:C604 -> SCCI_RH_SUP:C604
- C605: footprint ato_sup:C_0805_2012Metric -> scci_rh_sup:C_0805_2012Metric; symbol ATO_SUP:C605 -> SCCI_RH_SUP:C605
- C606: footprint ato_sup:C_0805_2012Metric -> scci_rh_sup:C_0805_2012Metric; symbol ATO_SUP:C606 -> SCCI_RH_SUP:C606
- C607: footprint ato_sup:C_0805_2012Metric -> scci_rh_sup:C_0805_2012Metric; symbol ATO_SUP:C607 -> SCCI_RH_SUP:C607
- J604: footprint ato_sup:PinHeader_1x02_P2.54mm_Vertical -> scci_rh_sup:PinHeader_1x02_P2.54mm_Vertical; symbol ATO_SUP:J604 -> SCCI_RH_SUP:J604
- J605: footprint ato_sup:PinHeader_1x02_P2.54mm_Vertical -> scci_rh_sup:PinHeader_1x02_P2.54mm_Vertical; symbol ATO_SUP:J605 -> SCCI_RH_SUP:J605
- J606: footprint ato_sup:PinHeader_1x02_P2.54mm_Vertical -> scci_rh_sup:PinHeader_1x02_P2.54mm_Vertical; symbol ATO_SUP:J606 -> SCCI_RH_SUP:J606
- J607: footprint ato_sup:PinHeader_1x02_P2.54mm_Vertical -> scci_rh_sup:PinHeader_1x02_P2.54mm_Vertical; symbol ATO_SUP:J607 -> SCCI_RH_SUP:J607
- R6040: footprint ato_sup:R_0805_2012Metric -> scci_rh_sup:R_0805_2012Metric; symbol ATO_SUP:R6040 -> SCCI_RH_SUP:R6040
- R6041: footprint ato_sup:R_0805_2012Metric -> scci_rh_sup:R_0805_2012Metric; symbol ATO_SUP:R6041 -> SCCI_RH_SUP:R6041
- R6050: footprint ato_sup:R_0805_2012Metric -> scci_rh_sup:R_0805_2012Metric; symbol ATO_SUP:R6050 -> SCCI_RH_SUP:R6050
- R6051: footprint ato_sup:R_0805_2012Metric -> scci_rh_sup:R_0805_2012Metric; symbol ATO_SUP:R6051 -> SCCI_RH_SUP:R6051
- R6060: footprint ato_sup:R_0805_2012Metric -> scci_rh_sup:R_0805_2012Metric; symbol ATO_SUP:R6060 -> SCCI_RH_SUP:R6060
- R6061: footprint ato_sup:R_0805_2012Metric -> scci_rh_sup:R_0805_2012Metric; symbol ATO_SUP:R6061 -> SCCI_RH_SUP:R6061
- R6070: footprint ato_sup:R_0805_2012Metric -> scci_rh_sup:R_0805_2012Metric; symbol ATO_SUP:R6070 -> SCCI_RH_SUP:R6070
- R6071: footprint ato_sup:R_0805_2012Metric -> scci_rh_sup:R_0805_2012Metric; symbol ATO_SUP:R6071 -> SCCI_RH_SUP:R6071
- U1017: footprint ato_sup:SOT-23-5 -> scci_rh_sup:SOT-23-5; symbol ATO_SUP:U1017 -> SCCI_RH_SUP:U1017
- U1018: footprint ato_sup:SOT-23-5 -> scci_rh_sup:SOT-23-5; symbol ATO_SUP:U1018 -> SCCI_RH_SUP:U1018
- U1019: footprint ato_sup:SOT-23-5 -> scci_rh_sup:SOT-23-5; symbol ATO_SUP:U1019 -> SCCI_RH_SUP:U1019
- U1020: footprint ato_sup:SOT-23-5 -> scci_rh_sup:SOT-23-5; symbol ATO_SUP:U1020 -> SCCI_RH_SUP:U1020
- U604: footprint ato_sup:VSSOP-8_2.3x2mm_P0.5mm -> scci_rh_sup:VSSOP-8_2.3x2mm_P0.5mm; symbol ATO_SUP:U604 -> SCCI_RH_SUP:U604
- U605: footprint ato_sup:VSSOP-8_2.3x2mm_P0.5mm -> scci_rh_sup:VSSOP-8_2.3x2mm_P0.5mm; symbol ATO_SUP:U605 -> SCCI_RH_SUP:U605
- U606: footprint ato_sup:VSSOP-8_2.3x2mm_P0.5mm -> scci_rh_sup:VSSOP-8_2.3x2mm_P0.5mm; symbol ATO_SUP:U606 -> SCCI_RH_SUP:U606
- U607: footprint ato_sup:VSSOP-8_2.3x2mm_P0.5mm -> scci_rh_sup:VSSOP-8_2.3x2mm_P0.5mm; symbol ATO_SUP:U607 -> SCCI_RH_SUP:U607
Other:
- company: Project ATO -> Project SCCI RH
- title: ATO S4 / RHD input windows 1 -> Project SCCI RH S4 / RHD input windows 1
