File: electronics/stage4/supervision/afe_bank2.kicad_sch (KiCad schematic)
At the start: 28 parts, among them J608 REC08 ACTUAL RHD-SIDE TAP, J609 REC09 ACTUAL RHD-SIDE TAP, J610 REC10 ACTUAL RHD-SIDE TAP, J611 REC11 ACTUAL RHD-SIDE TAP, U1021 SN74LVC1G08DBVR, U1022 SN74LVC1G08DBVR, U1023 SN74LVC1G08DBVR, U1024 SN74LVC1G08DBVR, U608 TLV3202DGKR, U609 TLV3202DGKR, U610 TLV3202DGKR, U611 TLV3202DGKR

Commit message: Rename project to Project SCCI RH across research and engineering
Parts:
- C1021: footprint ato_sup:C_0805_2012Metric -> scci_rh_sup:C_0805_2012Metric; symbol ATO_SUP:C1021 -> SCCI_RH_SUP:C1021
- C1022: footprint ato_sup:C_0805_2012Metric -> scci_rh_sup:C_0805_2012Metric; symbol ATO_SUP:C1022 -> SCCI_RH_SUP:C1022
- C1023: footprint ato_sup:C_0805_2012Metric -> scci_rh_sup:C_0805_2012Metric; symbol ATO_SUP:C1023 -> SCCI_RH_SUP:C1023
- C1024: footprint ato_sup:C_0805_2012Metric -> scci_rh_sup:C_0805_2012Metric; symbol ATO_SUP:C1024 -> SCCI_RH_SUP:C1024
- C608: footprint ato_sup:C_0805_2012Metric -> scci_rh_sup:C_0805_2012Metric; symbol ATO_SUP:C608 -> SCCI_RH_SUP:C608
- C609: footprint ato_sup:C_0805_2012Metric -> scci_rh_sup:C_0805_2012Metric; symbol ATO_SUP:C609 -> SCCI_RH_SUP:C609
- C610: footprint ato_sup:C_0805_2012Metric -> scci_rh_sup:C_0805_2012Metric; symbol ATO_SUP:C610 -> SCCI_RH_SUP:C610
- C611: footprint ato_sup:C_0805_2012Metric -> scci_rh_sup:C_0805_2012Metric; symbol ATO_SUP:C611 -> SCCI_RH_SUP:C611
- J608: footprint ato_sup:PinHeader_1x02_P2.54mm_Vertical -> scci_rh_sup:PinHeader_1x02_P2.54mm_Vertical; symbol ATO_SUP:J608 -> SCCI_RH_SUP:J608
- J609: footprint ato_sup:PinHeader_1x02_P2.54mm_Vertical -> scci_rh_sup:PinHeader_1x02_P2.54mm_Vertical; symbol ATO_SUP:J609 -> SCCI_RH_SUP:J609
- J610: footprint ato_sup:PinHeader_1x02_P2.54mm_Vertical -> scci_rh_sup:PinHeader_1x02_P2.54mm_Vertical; symbol ATO_SUP:J610 -> SCCI_RH_SUP:J610
- J611: footprint ato_sup:PinHeader_1x02_P2.54mm_Vertical -> scci_rh_sup:PinHeader_1x02_P2.54mm_Vertical; symbol ATO_SUP:J611 -> SCCI_RH_SUP:J611
- R6080: footprint ato_sup:R_0805_2012Metric -> scci_rh_sup:R_0805_2012Metric; symbol ATO_SUP:R6080 -> SCCI_RH_SUP:R6080
- R6081: footprint ato_sup:R_0805_2012Metric -> scci_rh_sup:R_0805_2012Metric; symbol ATO_SUP:R6081 -> SCCI_RH_SUP:R6081
- R6090: footprint ato_sup:R_0805_2012Metric -> scci_rh_sup:R_0805_2012Metric; symbol ATO_SUP:R6090 -> SCCI_RH_SUP:R6090
- R6091: footprint ato_sup:R_0805_2012Metric -> scci_rh_sup:R_0805_2012Metric; symbol ATO_SUP:R6091 -> SCCI_RH_SUP:R6091
- R6100: footprint ato_sup:R_0805_2012Metric -> scci_rh_sup:R_0805_2012Metric; symbol ATO_SUP:R6100 -> SCCI_RH_SUP:R6100
- R6101: footprint ato_sup:R_0805_2012Metric -> scci_rh_sup:R_0805_2012Metric; symbol ATO_SUP:R6101 -> SCCI_RH_SUP:R6101
- R6110: footprint ato_sup:R_0805_2012Metric -> scci_rh_sup:R_0805_2012Metric; symbol ATO_SUP:R6110 -> SCCI_RH_SUP:R6110
- R6111: footprint ato_sup:R_0805_2012Metric -> scci_rh_sup:R_0805_2012Metric; symbol ATO_SUP:R6111 -> SCCI_RH_SUP:R6111
- U1021: footprint ato_sup:SOT-23-5 -> scci_rh_sup:SOT-23-5; symbol ATO_SUP:U1021 -> SCCI_RH_SUP:U1021
- U1022: footprint ato_sup:SOT-23-5 -> scci_rh_sup:SOT-23-5; symbol ATO_SUP:U1022 -> SCCI_RH_SUP:U1022
- U1023: footprint ato_sup:SOT-23-5 -> scci_rh_sup:SOT-23-5; symbol ATO_SUP:U1023 -> SCCI_RH_SUP:U1023
- U1024: footprint ato_sup:SOT-23-5 -> scci_rh_sup:SOT-23-5; symbol ATO_SUP:U1024 -> SCCI_RH_SUP:U1024
- U608: footprint ato_sup:VSSOP-8_2.3x2mm_P0.5mm -> scci_rh_sup:VSSOP-8_2.3x2mm_P0.5mm; symbol ATO_SUP:U608 -> SCCI_RH_SUP:U608
- U609: footprint ato_sup:VSSOP-8_2.3x2mm_P0.5mm -> scci_rh_sup:VSSOP-8_2.3x2mm_P0.5mm; symbol ATO_SUP:U609 -> SCCI_RH_SUP:U609
- U610: footprint ato_sup:VSSOP-8_2.3x2mm_P0.5mm -> scci_rh_sup:VSSOP-8_2.3x2mm_P0.5mm; symbol ATO_SUP:U610 -> SCCI_RH_SUP:U610
- U611: footprint ato_sup:VSSOP-8_2.3x2mm_P0.5mm -> scci_rh_sup:VSSOP-8_2.3x2mm_P0.5mm; symbol ATO_SUP:U611 -> SCCI_RH_SUP:U611
Other:
- company: Project ATO -> Project SCCI RH
- title: ATO S4 / RHD input windows 2 -> Project SCCI RH S4 / RHD input windows 2
