File: electronics/stage4/supervision/afe_bank3.kicad_sch (KiCad schematic)
At the start: 28 parts, among them J612 REC12 ACTUAL RHD-SIDE TAP, J613 REC13 ACTUAL RHD-SIDE TAP, J614 REC14 ACTUAL RHD-SIDE TAP, J615 REC15 ACTUAL RHD-SIDE TAP, U1025 SN74LVC1G08DBVR, U1026 SN74LVC1G08DBVR, U1027 SN74LVC1G08DBVR, U1028 SN74LVC1G08DBVR, U612 TLV3202DGKR, U613 TLV3202DGKR, U614 TLV3202DGKR, U615 TLV3202DGKR

Commit message: Rename project to Project SCCI RH across research and engineering
Parts:
- C1025: footprint ato_sup:C_0805_2012Metric -> scci_rh_sup:C_0805_2012Metric; symbol ATO_SUP:C1025 -> SCCI_RH_SUP:C1025
- C1026: footprint ato_sup:C_0805_2012Metric -> scci_rh_sup:C_0805_2012Metric; symbol ATO_SUP:C1026 -> SCCI_RH_SUP:C1026
- C1027: footprint ato_sup:C_0805_2012Metric -> scci_rh_sup:C_0805_2012Metric; symbol ATO_SUP:C1027 -> SCCI_RH_SUP:C1027
- C1028: footprint ato_sup:C_0805_2012Metric -> scci_rh_sup:C_0805_2012Metric; symbol ATO_SUP:C1028 -> SCCI_RH_SUP:C1028
- C612: footprint ato_sup:C_0805_2012Metric -> scci_rh_sup:C_0805_2012Metric; symbol ATO_SUP:C612 -> SCCI_RH_SUP:C612
- C613: footprint ato_sup:C_0805_2012Metric -> scci_rh_sup:C_0805_2012Metric; symbol ATO_SUP:C613 -> SCCI_RH_SUP:C613
- C614: footprint ato_sup:C_0805_2012Metric -> scci_rh_sup:C_0805_2012Metric; symbol ATO_SUP:C614 -> SCCI_RH_SUP:C614
- C615: footprint ato_sup:C_0805_2012Metric -> scci_rh_sup:C_0805_2012Metric; symbol ATO_SUP:C615 -> SCCI_RH_SUP:C615
- J612: footprint ato_sup:PinHeader_1x02_P2.54mm_Vertical -> scci_rh_sup:PinHeader_1x02_P2.54mm_Vertical; symbol ATO_SUP:J612 -> SCCI_RH_SUP:J612
- J613: footprint ato_sup:PinHeader_1x02_P2.54mm_Vertical -> scci_rh_sup:PinHeader_1x02_P2.54mm_Vertical; symbol ATO_SUP:J613 -> SCCI_RH_SUP:J613
- J614: footprint ato_sup:PinHeader_1x02_P2.54mm_Vertical -> scci_rh_sup:PinHeader_1x02_P2.54mm_Vertical; symbol ATO_SUP:J614 -> SCCI_RH_SUP:J614
- J615: footprint ato_sup:PinHeader_1x02_P2.54mm_Vertical -> scci_rh_sup:PinHeader_1x02_P2.54mm_Vertical; symbol ATO_SUP:J615 -> SCCI_RH_SUP:J615
- R6120: footprint ato_sup:R_0805_2012Metric -> scci_rh_sup:R_0805_2012Metric; symbol ATO_SUP:R6120 -> SCCI_RH_SUP:R6120
- R6121: footprint ato_sup:R_0805_2012Metric -> scci_rh_sup:R_0805_2012Metric; symbol ATO_SUP:R6121 -> SCCI_RH_SUP:R6121
- R6130: footprint ato_sup:R_0805_2012Metric -> scci_rh_sup:R_0805_2012Metric; symbol ATO_SUP:R6130 -> SCCI_RH_SUP:R6130
- R6131: footprint ato_sup:R_0805_2012Metric -> scci_rh_sup:R_0805_2012Metric; symbol ATO_SUP:R6131 -> SCCI_RH_SUP:R6131
- R6140: footprint ato_sup:R_0805_2012Metric -> scci_rh_sup:R_0805_2012Metric; symbol ATO_SUP:R6140 -> SCCI_RH_SUP:R6140
- R6141: footprint ato_sup:R_0805_2012Metric -> scci_rh_sup:R_0805_2012Metric; symbol ATO_SUP:R6141 -> SCCI_RH_SUP:R6141
- R6150: footprint ato_sup:R_0805_2012Metric -> scci_rh_sup:R_0805_2012Metric; symbol ATO_SUP:R6150 -> SCCI_RH_SUP:R6150
- R6151: footprint ato_sup:R_0805_2012Metric -> scci_rh_sup:R_0805_2012Metric; symbol ATO_SUP:R6151 -> SCCI_RH_SUP:R6151
- U1025: footprint ato_sup:SOT-23-5 -> scci_rh_sup:SOT-23-5; symbol ATO_SUP:U1025 -> SCCI_RH_SUP:U1025
- U1026: footprint ato_sup:SOT-23-5 -> scci_rh_sup:SOT-23-5; symbol ATO_SUP:U1026 -> SCCI_RH_SUP:U1026
- U1027: footprint ato_sup:SOT-23-5 -> scci_rh_sup:SOT-23-5; symbol ATO_SUP:U1027 -> SCCI_RH_SUP:U1027
- U1028: footprint ato_sup:SOT-23-5 -> scci_rh_sup:SOT-23-5; symbol ATO_SUP:U1028 -> SCCI_RH_SUP:U1028
- U612: footprint ato_sup:VSSOP-8_2.3x2mm_P0.5mm -> scci_rh_sup:VSSOP-8_2.3x2mm_P0.5mm; symbol ATO_SUP:U612 -> SCCI_RH_SUP:U612
- U613: footprint ato_sup:VSSOP-8_2.3x2mm_P0.5mm -> scci_rh_sup:VSSOP-8_2.3x2mm_P0.5mm; symbol ATO_SUP:U613 -> SCCI_RH_SUP:U613
- U614: footprint ato_sup:VSSOP-8_2.3x2mm_P0.5mm -> scci_rh_sup:VSSOP-8_2.3x2mm_P0.5mm; symbol ATO_SUP:U614 -> SCCI_RH_SUP:U614
- U615: footprint ato_sup:VSSOP-8_2.3x2mm_P0.5mm -> scci_rh_sup:VSSOP-8_2.3x2mm_P0.5mm; symbol ATO_SUP:U615 -> SCCI_RH_SUP:U615
Other:
- company: Project ATO -> Project SCCI RH
- title: ATO S4 / RHD input windows 3 -> Project SCCI RH S4 / RHD input windows 3
