File: electronics/stage4/supervision/afe_bank4.kicad_sch (KiCad schematic)
At the start: 7 parts, among them J616 REF ACTUAL RHD-SIDE TAP, U1029 SN74LVC1G08DBVR, U616 TLV3202DGKR

Commit message: Rename project to Project SCCI RH across research and engineering
Parts:
- C1029: footprint ato_sup:C_0805_2012Metric -> scci_rh_sup:C_0805_2012Metric; symbol ATO_SUP:C1029 -> SCCI_RH_SUP:C1029
- C616: footprint ato_sup:C_0805_2012Metric -> scci_rh_sup:C_0805_2012Metric; symbol ATO_SUP:C616 -> SCCI_RH_SUP:C616
- J616: footprint ato_sup:PinHeader_1x02_P2.54mm_Vertical -> scci_rh_sup:PinHeader_1x02_P2.54mm_Vertical; symbol ATO_SUP:J616 -> SCCI_RH_SUP:J616
- R6160: footprint ato_sup:R_0805_2012Metric -> scci_rh_sup:R_0805_2012Metric; symbol ATO_SUP:R6160 -> SCCI_RH_SUP:R6160
- R6161: footprint ato_sup:R_0805_2012Metric -> scci_rh_sup:R_0805_2012Metric; symbol ATO_SUP:R6161 -> SCCI_RH_SUP:R6161
- U1029: footprint ato_sup:SOT-23-5 -> scci_rh_sup:SOT-23-5; symbol ATO_SUP:U1029 -> SCCI_RH_SUP:U1029
- U616: footprint ato_sup:VSSOP-8_2.3x2mm_P0.5mm -> scci_rh_sup:VSSOP-8_2.3x2mm_P0.5mm; symbol ATO_SUP:U616 -> SCCI_RH_SUP:U616
Other:
- company: Project ATO -> Project SCCI RH
- title: ATO S4 / RHD input windows 4 -> Project SCCI RH S4 / RHD input windows 4
