File: electronics/stage4/supervision/afe_rails.kicad_sch (KiCad schematic)
At the start: 16 parts, among them U206 TPS3700DDCR, U207 TPS3700DDCR, U208 TPS3700DDCR

Commit message: Rename project to Project SCCI RH across research and engineering
Parts:
- C206: footprint ato_sup:C_0805_2012Metric -> scci_rh_sup:C_0805_2012Metric; symbol ATO_SUP:C206 -> SCCI_RH_SUP:C206
- C207: footprint ato_sup:C_0805_2012Metric -> scci_rh_sup:C_0805_2012Metric; symbol ATO_SUP:C207 -> SCCI_RH_SUP:C207
- R2060: footprint ato_sup:R_0805_2012Metric -> scci_rh_sup:R_0805_2012Metric; symbol ATO_SUP:R2060 -> SCCI_RH_SUP:R2060
- R2061: footprint ato_sup:R_0805_2012Metric -> scci_rh_sup:R_0805_2012Metric; symbol ATO_SUP:R2061 -> SCCI_RH_SUP:R2061
- R2062: footprint ato_sup:R_0805_2012Metric -> scci_rh_sup:R_0805_2012Metric; symbol ATO_SUP:R2062 -> SCCI_RH_SUP:R2062
- R2063: footprint ato_sup:R_0805_2012Metric -> scci_rh_sup:R_0805_2012Metric; symbol ATO_SUP:R2063 -> SCCI_RH_SUP:R2063
- R2064: footprint ato_sup:R_0805_2012Metric -> scci_rh_sup:R_0805_2012Metric; symbol ATO_SUP:R2064 -> SCCI_RH_SUP:R2064
- R2070: footprint ato_sup:R_0805_2012Metric -> scci_rh_sup:R_0805_2012Metric; symbol ATO_SUP:R2070 -> SCCI_RH_SUP:R2070
- R2071: footprint ato_sup:R_0805_2012Metric -> scci_rh_sup:R_0805_2012Metric; symbol ATO_SUP:R2071 -> SCCI_RH_SUP:R2071
- R2072: footprint ato_sup:R_0805_2012Metric -> scci_rh_sup:R_0805_2012Metric; symbol ATO_SUP:R2072 -> SCCI_RH_SUP:R2072
- R2073: footprint ato_sup:R_0805_2012Metric -> scci_rh_sup:R_0805_2012Metric; symbol ATO_SUP:R2073 -> SCCI_RH_SUP:R2073
- R2074: footprint ato_sup:R_0805_2012Metric -> scci_rh_sup:R_0805_2012Metric; symbol ATO_SUP:R2074 -> SCCI_RH_SUP:R2074
- R2080: footprint ato_sup:R_0805_2012Metric -> scci_rh_sup:R_0805_2012Metric; symbol ATO_SUP:R2080 -> SCCI_RH_SUP:R2080
- U206: footprint ato_sup:SOT-23-6 -> scci_rh_sup:SOT-23-6; symbol ATO_SUP:U206 -> SCCI_RH_SUP:U206
- U207: footprint ato_sup:SOT-23-6 -> scci_rh_sup:SOT-23-6; symbol ATO_SUP:U207 -> SCCI_RH_SUP:U207
- U208: footprint ato_sup:SOT-23-6 -> scci_rh_sup:SOT-23-6; symbol ATO_SUP:U208 -> SCCI_RH_SUP:U208
Other:
- company: Project ATO -> Project SCCI RH
- title: ATO S4 / AFE supply windows -> Project SCCI RH S4 / AFE supply windows
