File: electronics/stage4/supervision/guards.kicad_sch (KiCad schematic)
At the start: 18 parts, among them J100 CANONICAL ROUTER J7 / BEFORE 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, J101 BODY-FACING ARTIFICIAL LOAD C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, U100 TMUX7412FRRPR, U101 TMUX7412FRRPR, U102 TMUX7412FRRPR, U103 TMUX7412FRRPR, U104 TMUX7412FRRPR

Commit message: Rename project to Project SCCI RH across research and engineering
Parts:
- C100: footprint ato_sup:C_0805_2012Metric -> scci_rh_sup:C_0805_2012Metric; symbol ATO_SUP:C100 -> SCCI_RH_SUP:C100
- C101: footprint ato_sup:C_0805_2012Metric -> scci_rh_sup:C_0805_2012Metric; symbol ATO_SUP:C101 -> SCCI_RH_SUP:C101
- C102: footprint ato_sup:C_0805_2012Metric -> scci_rh_sup:C_0805_2012Metric; symbol ATO_SUP:C102 -> SCCI_RH_SUP:C102
- C103: footprint ato_sup:C_0805_2012Metric -> scci_rh_sup:C_0805_2012Metric; symbol ATO_SUP:C103 -> SCCI_RH_SUP:C103
- C104: footprint ato_sup:C_0805_2012Metric -> scci_rh_sup:C_0805_2012Metric; symbol ATO_SUP:C104 -> SCCI_RH_SUP:C104
- J100: footprint ato_sup:PinHeader_1x18_P2.54mm_Vertical -> scci_rh_sup:PinHeader_1x18_P2.54mm_Vertical; symbol ATO_SUP:J100 -> SCCI_RH_SUP:J100
- J101: footprint ato_sup:PinHeader_1x18_P2.54mm_Vertical -> scci_rh_sup:PinHeader_1x18_P2.54mm_Vertical; symbol ATO_SUP:J101 -> SCCI_RH_SUP:J101
- R100: footprint ato_sup:R_0805_2012Metric -> scci_rh_sup:R_0805_2012Metric; symbol ATO_SUP:R100 -> SCCI_RH_SUP:R100
- R101: footprint ato_sup:R_0805_2012Metric -> scci_rh_sup:R_0805_2012Metric; symbol ATO_SUP:R101 -> SCCI_RH_SUP:R101
- R102: footprint ato_sup:R_0805_2012Metric -> scci_rh_sup:R_0805_2012Metric; symbol ATO_SUP:R102 -> SCCI_RH_SUP:R102
- R103: footprint ato_sup:R_0805_2012Metric -> scci_rh_sup:R_0805_2012Metric; symbol ATO_SUP:R103 -> SCCI_RH_SUP:R103
- R104: footprint ato_sup:R_0805_2012Metric -> scci_rh_sup:R_0805_2012Metric; symbol ATO_SUP:R104 -> SCCI_RH_SUP:R104
- R110: footprint ato_sup:R_0805_2012Metric -> scci_rh_sup:R_0805_2012Metric; symbol ATO_SUP:R110 -> SCCI_RH_SUP:R110
- U100: footprint ato_sup:Texas_RRP0016A_WQFN16_4x4_P0.65_EP2.6 -> scci_rh_sup:Texas_RRP0016A_WQFN16_4x4_P0.65_EP2.6; symbol ATO_SUP:U100 -> SCCI_RH_SUP:U100
- U101: footprint ato_sup:Texas_RRP0016A_WQFN16_4x4_P0.65_EP2.6 -> scci_rh_sup:Texas_RRP0016A_WQFN16_4x4_P0.65_EP2.6; symbol ATO_SUP:U101 -> SCCI_RH_SUP:U101
- U102: footprint ato_sup:Texas_RRP0016A_WQFN16_4x4_P0.65_EP2.6 -> scci_rh_sup:Texas_RRP0016A_WQFN16_4x4_P0.65_EP2.6; symbol ATO_SUP:U102 -> SCCI_RH_SUP:U102
- U103: footprint ato_sup:Texas_RRP0016A_WQFN16_4x4_P0.65_EP2.6 -> scci_rh_sup:Texas_RRP0016A_WQFN16_4x4_P0.65_EP2.6; symbol ATO_SUP:U103 -> SCCI_RH_SUP:U103
- U104: footprint ato_sup:Texas_RRP0016A_WQFN16_4x4_P0.65_EP2.6 -> scci_rh_sup:Texas_RRP0016A_WQFN16_4x4_P0.65_EP2.6; symbol ATO_SUP:U104 -> SCCI_RH_SUP:U104
Other:
- company: Project ATO -> Project SCCI RH
- title: ATO S4 / 18 body-side terminal guards -> Project SCCI RH S4 / 18 body-side terminal guards
