File: electronics/stage4/supervision/host_rails_2.kicad_sch (KiCad schematic)
At the start: 21 parts, among them U203 TPS3700DDCR, U204 TPS3700DDCR, U205 TPS3700DDCR

Commit message: Rename project to Project SCCI RH across research and engineering
Parts:
- C203: footprint ato_sup:C_0805_2012Metric -> scci_rh_sup:C_0805_2012Metric; symbol ATO_SUP:C203 -> SCCI_RH_SUP:C203
- C204: footprint ato_sup:C_0805_2012Metric -> scci_rh_sup:C_0805_2012Metric; symbol ATO_SUP:C204 -> SCCI_RH_SUP:C204
- C205: footprint ato_sup:C_0805_2012Metric -> scci_rh_sup:C_0805_2012Metric; symbol ATO_SUP:C205 -> SCCI_RH_SUP:C205
- R2030: footprint ato_sup:R_0805_2012Metric -> scci_rh_sup:R_0805_2012Metric; symbol ATO_SUP:R2030 -> SCCI_RH_SUP:R2030
- R2031: footprint ato_sup:R_0805_2012Metric -> scci_rh_sup:R_0805_2012Metric; symbol ATO_SUP:R2031 -> SCCI_RH_SUP:R2031
- R2032: footprint ato_sup:R_0805_2012Metric -> scci_rh_sup:R_0805_2012Metric; symbol ATO_SUP:R2032 -> SCCI_RH_SUP:R2032
- R2033: footprint ato_sup:R_0805_2012Metric -> scci_rh_sup:R_0805_2012Metric; symbol ATO_SUP:R2033 -> SCCI_RH_SUP:R2033
- R2034: footprint ato_sup:R_0805_2012Metric -> scci_rh_sup:R_0805_2012Metric; symbol ATO_SUP:R2034 -> SCCI_RH_SUP:R2034
- R2040: footprint ato_sup:R_0805_2012Metric -> scci_rh_sup:R_0805_2012Metric; symbol ATO_SUP:R2040 -> SCCI_RH_SUP:R2040
- R2041: footprint ato_sup:R_0805_2012Metric -> scci_rh_sup:R_0805_2012Metric; symbol ATO_SUP:R2041 -> SCCI_RH_SUP:R2041
- R2042: footprint ato_sup:R_0805_2012Metric -> scci_rh_sup:R_0805_2012Metric; symbol ATO_SUP:R2042 -> SCCI_RH_SUP:R2042
- R2043: footprint ato_sup:R_0805_2012Metric -> scci_rh_sup:R_0805_2012Metric; symbol ATO_SUP:R2043 -> SCCI_RH_SUP:R2043
- R2044: footprint ato_sup:R_0805_2012Metric -> scci_rh_sup:R_0805_2012Metric; symbol ATO_SUP:R2044 -> SCCI_RH_SUP:R2044
- R2050: footprint ato_sup:R_0805_2012Metric -> scci_rh_sup:R_0805_2012Metric; symbol ATO_SUP:R2050 -> SCCI_RH_SUP:R2050
- R2051: footprint ato_sup:R_0805_2012Metric -> scci_rh_sup:R_0805_2012Metric; symbol ATO_SUP:R2051 -> SCCI_RH_SUP:R2051
- R2052: footprint ato_sup:R_0805_2012Metric -> scci_rh_sup:R_0805_2012Metric; symbol ATO_SUP:R2052 -> SCCI_RH_SUP:R2052
- R2053: footprint ato_sup:R_0805_2012Metric -> scci_rh_sup:R_0805_2012Metric; symbol ATO_SUP:R2053 -> SCCI_RH_SUP:R2053
- R2054: footprint ato_sup:R_0805_2012Metric -> scci_rh_sup:R_0805_2012Metric; symbol ATO_SUP:R2054 -> SCCI_RH_SUP:R2054
- U203: footprint ato_sup:SOT-23-6 -> scci_rh_sup:SOT-23-6; symbol ATO_SUP:U203 -> SCCI_RH_SUP:U203
- U204: footprint ato_sup:SOT-23-6 -> scci_rh_sup:SOT-23-6; symbol ATO_SUP:U204 -> SCCI_RH_SUP:U204
- U205: footprint ato_sup:SOT-23-6 -> scci_rh_sup:SOT-23-6; symbol ATO_SUP:U205 -> SCCI_RH_SUP:U205
Other:
- company: Project ATO -> Project SCCI RH
- title: ATO S4 / Host supply windows / 2 -> Project SCCI RH S4 / Host supply windows / 2
