File: electronics/stage4/supervision/phase1.kicad_sch (KiCad schematic)
At the start: 28 parts, among them U1084 SN74LVC1G11DBVR, U1085 SN74LVC1G08DBVR, U1086 SN74LVC1G04DBVR, U1087 SN74LVC1G08DBVR, U1088 SN74LVC1G11DBVR, U1089 SN74LVC1G11DBVR, U1090 SN74LVC1G08DBVR, U1091 SN74LVC1G04DBVR, U1092 SN74LVC1G04DBVR, U1093 SN74LVC1G11DBVR, U1094 SN74LVC1G11DBVR, U1095 SN74LVC1G08DBVR, U1096 SN74LVC1G11DBVR, U911 SN74LVC1G74DCUR

Commit message: Rename project to Project SCCI RH across research and engineering
Parts:
- C1084: footprint ato_sup:C_0805_2012Metric -> scci_rh_sup:C_0805_2012Metric; symbol ATO_SUP:C1084 -> SCCI_RH_SUP:C1084
- C1085: footprint ato_sup:C_0805_2012Metric -> scci_rh_sup:C_0805_2012Metric; symbol ATO_SUP:C1085 -> SCCI_RH_SUP:C1085
- C1086: footprint ato_sup:C_0805_2012Metric -> scci_rh_sup:C_0805_2012Metric; symbol ATO_SUP:C1086 -> SCCI_RH_SUP:C1086
- C1087: footprint ato_sup:C_0805_2012Metric -> scci_rh_sup:C_0805_2012Metric; symbol ATO_SUP:C1087 -> SCCI_RH_SUP:C1087
- C1088: footprint ato_sup:C_0805_2012Metric -> scci_rh_sup:C_0805_2012Metric; symbol ATO_SUP:C1088 -> SCCI_RH_SUP:C1088
- C1089: footprint ato_sup:C_0805_2012Metric -> scci_rh_sup:C_0805_2012Metric; symbol ATO_SUP:C1089 -> SCCI_RH_SUP:C1089
- C1090: footprint ato_sup:C_0805_2012Metric -> scci_rh_sup:C_0805_2012Metric; symbol ATO_SUP:C1090 -> SCCI_RH_SUP:C1090
- C1091: footprint ato_sup:C_0805_2012Metric -> scci_rh_sup:C_0805_2012Metric; symbol ATO_SUP:C1091 -> SCCI_RH_SUP:C1091
- C1092: footprint ato_sup:C_0805_2012Metric -> scci_rh_sup:C_0805_2012Metric; symbol ATO_SUP:C1092 -> SCCI_RH_SUP:C1092
- C1093: footprint ato_sup:C_0805_2012Metric -> scci_rh_sup:C_0805_2012Metric; symbol ATO_SUP:C1093 -> SCCI_RH_SUP:C1093
- C1094: footprint ato_sup:C_0805_2012Metric -> scci_rh_sup:C_0805_2012Metric; symbol ATO_SUP:C1094 -> SCCI_RH_SUP:C1094
- C1095: footprint ato_sup:C_0805_2012Metric -> scci_rh_sup:C_0805_2012Metric; symbol ATO_SUP:C1095 -> SCCI_RH_SUP:C1095
- C1096: footprint ato_sup:C_0805_2012Metric -> scci_rh_sup:C_0805_2012Metric; symbol ATO_SUP:C1096 -> SCCI_RH_SUP:C1096
- C911: footprint ato_sup:C_0805_2012Metric -> scci_rh_sup:C_0805_2012Metric; symbol ATO_SUP:C911 -> SCCI_RH_SUP:C911
- U1084: footprint ato_sup:SOT-23-6 -> scci_rh_sup:SOT-23-6; symbol ATO_SUP:U1084 -> SCCI_RH_SUP:U1084
- U1085: footprint ato_sup:SOT-23-5 -> scci_rh_sup:SOT-23-5; symbol ATO_SUP:U1085 -> SCCI_RH_SUP:U1085
- U1086: footprint ato_sup:SOT-23-5 -> scci_rh_sup:SOT-23-5; symbol ATO_SUP:U1086 -> SCCI_RH_SUP:U1086
- U1087: footprint ato_sup:SOT-23-5 -> scci_rh_sup:SOT-23-5; symbol ATO_SUP:U1087 -> SCCI_RH_SUP:U1087
- U1088: footprint ato_sup:SOT-23-6 -> scci_rh_sup:SOT-23-6; symbol ATO_SUP:U1088 -> SCCI_RH_SUP:U1088
- U1089: footprint ato_sup:SOT-23-6 -> scci_rh_sup:SOT-23-6; symbol ATO_SUP:U1089 -> SCCI_RH_SUP:U1089
- U1090: footprint ato_sup:SOT-23-5 -> scci_rh_sup:SOT-23-5; symbol ATO_SUP:U1090 -> SCCI_RH_SUP:U1090
- U1091: footprint ato_sup:SOT-23-5 -> scci_rh_sup:SOT-23-5; symbol ATO_SUP:U1091 -> SCCI_RH_SUP:U1091
- U1092: footprint ato_sup:SOT-23-5 -> scci_rh_sup:SOT-23-5; symbol ATO_SUP:U1092 -> SCCI_RH_SUP:U1092
- U1093: footprint ato_sup:SOT-23-6 -> scci_rh_sup:SOT-23-6; symbol ATO_SUP:U1093 -> SCCI_RH_SUP:U1093
- U1094: footprint ato_sup:SOT-23-6 -> scci_rh_sup:SOT-23-6; symbol ATO_SUP:U1094 -> SCCI_RH_SUP:U1094
- U1095: footprint ato_sup:SOT-23-5 -> scci_rh_sup:SOT-23-5; symbol ATO_SUP:U1095 -> SCCI_RH_SUP:U1095
- U1096: footprint ato_sup:SOT-23-6 -> scci_rh_sup:SOT-23-6; symbol ATO_SUP:U1096 -> SCCI_RH_SUP:U1096
- U911: footprint ato_sup:VSSOP-8_2.3x2mm_P0.5mm -> scci_rh_sup:VSSOP-8_2.3x2mm_P0.5mm; symbol ATO_SUP:U911 -> SCCI_RH_SUP:U911
Other:
- company: Project ATO -> Project SCCI RH
- title: ATO S4 / Source 1 phase permission -> Project SCCI RH S4 / Source 1 phase permission
