File: electronics/stage4/supervision/supervision.kicad_sch (KiCad schematic)
At the start: 6 parts, among them J1 EXTERNAL SUPERVISOR AND HOST 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, J2 FLOATING AFE RAILS AND OBSERV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, J3 RAW CONTROL / STATUS, J4 EXISTING MONITOR OBSERVATIONS, J5 EXPORTED NATIVE HEALTH / PERM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, J6 DRIVER INTERNAL DIFFERENTIAL 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

Commit message: Rename project to Project SCCI RH across research and engineering
Parts:
- J1: footprint ato_sup:PinHeader_1x07_P2.54mm_Vertical -> scci_rh_sup:PinHeader_1x07_P2.54mm_Vertical; symbol ATO_SUP:J1 -> SCCI_RH_SUP:J1
- J2: footprint ato_sup:PinHeader_1x06_P2.54mm_Vertical -> scci_rh_sup:PinHeader_1x06_P2.54mm_Vertical; symbol ATO_SUP:J2 -> SCCI_RH_SUP:J2
- J3: footprint ato_sup:PinHeader_1x12_P2.54mm_Vertical -> scci_rh_sup:PinHeader_1x12_P2.54mm_Vertical; symbol ATO_SUP:J3 -> SCCI_RH_SUP:J3
- J4: footprint ato_sup:PinHeader_1x09_P2.54mm_Vertical -> scci_rh_sup:PinHeader_1x09_P2.54mm_Vertical; symbol ATO_SUP:J4 -> SCCI_RH_SUP:J4
- J5: footprint ato_sup:PinHeader_1x13_P2.54mm_Vertical -> scci_rh_sup:PinHeader_1x13_P2.54mm_Vertical; symbol ATO_SUP:J5 -> SCCI_RH_SUP:J5
- J6: footprint ato_sup:PinHeader_1x05_P2.54mm_Vertical -> scci_rh_sup:PinHeader_1x05_P2.54mm_Vertical; symbol ATO_SUP:J6 -> SCCI_RH_SUP:J6
Other:
- company: Project ATO -> Project SCCI RH
- title: ATO S4 / Interfaces and handoff -> Project SCCI RH S4 / Interfaces and handoff
